Commit message: commit

File: body.urdf (robot description, URDF)
Before this commit: robot robot, 30 links, 29 joints
Links:
- removed link 22
- removed link 23
- removed link 24
- removed link 25
- removed link 26
- removed link 27
- removed link 28
- removed link 29
- link 0: geometry collision box size=0.005244274653084302 0.8226080823699238 0.19467511196622322; visual box size=0.005244274653084302 0.8226080823699238 0.19467511196622322
- link 1: geometry collision box size=0.9122767895336106 0.3122622312726785 0.005631053959663346; visual box size=0.9122767895336106 0.3122622312726785 0.005631053959663346
- link 10: geometry collision box size=0.40276276758908025 0.7162003919973214 0.8340320007583978; visual box size=0.40276276758908025 0.7162003919973214 0.8340320007583978
- link 11: geometry collision box size=0.11141302994328595 0.11607964616457378 0.2941708685667266; visual box size=0.11141302994328595 0.11607964616457378 0.2941708685667266
- link 12: geometry collision box size=0.6228423497145011 0.5207200162487802 0.616803327174415; visual box size=0.6228423497145011 0.5207200162487802 0.616803327174415
- link 13: geometry collision box size=0.12995794897402557 0.8598289825889011 0.9830197629178058; visual box size=0.12995794897402557 0.8598289825889011 0.9830197629178058
- link 14: geometry collision box size=0.37693902030828275 0.8290522262573269 0.3196342536005451; visual box size=0.37693902030828275 0.8290522262573269 0.3196342536005451
- link 15: geometry collision box size=0.687222177442973 0.18865421848377062 0.8942624392254513; visual box size=0.687222177442973 0.18865421848377062 0.8942624392254513
- link 16: geometry collision box size=0.8779207279190931 0.04622271993416638 0.635555917453163; visual box size=0.8779207279190931 0.04622271993416638 0.635555917453163
- link 17: geometry collision box size=0.6904119983055426 0.31320371856655904 0.5939566847685087; visual box size=0.6904119983055426 0.31320371856655904 0.5939566847685087
- link 18: geometry collision box size=0.9701529497143704 0.5147601507271262 0.951962863421401; visual box size=0.9701529497143704 0.5147601507271262 0.951962863421401
- link 19: geometry collision box size=0.6815699902866723 0.1608824740445456 0.9677904079601489; visual box size=0.6815699902866723 0.1608824740445456 0.9677904079601489
- link 2: geometry collision box size=0.8410294012002504 0.7368235786639841 0.6699454524356928; visual box size=0.8410294012002504 0.7368235786639841 0.6699454524356928
- link 20: geometry collision box size=0.18962314563565352 0.26627043206239975 0.6749067091255374; visual box size=0.18962314563565352 0.26627043206239975 0.6749067091255374
- link 21: geometry collision box size=0.6426069428245889 0.4644236221899406 0.11748007762395629; visual box size=0.6426069428245889 0.4644236221899406 0.11748007762395629
- link 3: geometry collision box size=0.8148245701293075 0.11736278624040142 0.32306954823576506; visual box size=0.8148245701293075 0.11736278624040142 0.32306954823576506
- link 4: geometry collision box size=0.056167770504606085 0.5205606359270737 0.2426628331829317; visual box size=0.056167770504606085 0.5205606359270737 0.2426628331829317
- link 5: geometry collision box size=0.26427949599189327 0.7296820151044697 0.687247728228293; visual box size=0.26427949599189327 0.7296820151044697 0.687247728228293
- link 6: geometry collision box size=0.5494416787210893 0.12462041601905538 0.9595838871203926; visual box size=0.5494416787210893 0.12462041601905538 0.9595838871203926
- link 7: geometry collision box size=0.7845833275216404 0.514027015904515 0.9196424534213085; visual box size=0.7845833275216404 0.514027015904515 0.9196424534213085
- link 8: geometry collision box size=0.4893250477731339 0.1726285868809193 0.21714337926065264; visual box size=0.4893250477731339 0.1726285868809193 0.21714337926065264
- link 9: geometry collision box size=0.8988883112505559 0.8108909251512177 0.7294797723134089; visual box size=0.8988883112505559 0.8108909251512177 0.7294797723134089
Joints:
- removed joint 11_12
- removed joint 16_17
- removed joint 1_16
- removed joint 1_23
- removed joint 1_9
- removed joint 21_22
- removed joint 23_24
- removed joint 24_25
- removed joint 25_26
- removed joint 26_27
- removed joint 27_28
- removed joint 28_29
- removed joint 6_7
- added joint 15_16: type revolute, parent 15, child 16, origin xyz=0 -0.18865421848377062 0 rpy=0 0 0, axis 1 0 0, limit lower=-3.14159 upper=3.14159 effort=0.0 velocity=0.0
- added joint 1_12: type revolute, parent 1, child 12, origin xyz=0 -0.15613111563633925 0 rpy=0 0 0, axis 1 0 0, limit lower=-3.14159 upper=3.14159 effort=0.0 velocity=0.0
- added joint 1_17: type revolute, parent 1, child 17, origin xyz=0 0.15613111563633925 0 rpy=0 0 0, axis 1 0 0, limit lower=-3.14159 upper=3.14159 effort=0.0 velocity=0.0
- added joint 1_7: type revolute, parent 1, child 7, origin xyz=0.4561383947668053 0 0 rpy=0 0 0, axis 0 1 0, limit lower=-3.14159 upper=3.14159 effort=0.0 velocity=0.0
- added joint 8_9: type revolute, parent 8, child 9, origin xyz=0.4893250477731339 0 0 rpy=0 0 0, axis 0 1 0, limit lower=-3.14159 upper=3.14159 effort=0.0 velocity=0.0
- joint 0_1: origin xyz=0 0 0.7105919188561834 rpy=0 0 0 -> xyz=0 0 0.19467511196622322 rpy=0 0 0
- joint 10_11: origin xyz=0.7071861840649788 0 0 rpy=0 0 0 -> xyz=0.40276276758908025 0 0 rpy=0 0 0
- joint 12_13: axis 0 1 0 -> 1 0 0; origin xyz=0.9196571976824377 0 0 rpy=0 0 0 -> xyz=0 -0.5207200162487802 0 rpy=0 0 0
- joint 13_14: axis 0 1 0 -> 1 0 0; origin xyz=0.4922349663734352 0 0 rpy=0 0 0 -> xyz=0 -0.8598289825889011 0 rpy=0 0 0
- joint 14_15: axis 0 1 0 -> 1 0 0; origin xyz=0.5104874849399225 0 0 rpy=0 0 0 -> xyz=0 -0.8290522262573269 0 rpy=0 0 0
- joint 17_18: origin xyz=0 -0.6771743925958059 0 rpy=0 0 0 -> xyz=0 0.31320371856655904 0 rpy=0 0 0
- joint 18_19: origin xyz=0 -0.9109955621327389 0 rpy=0 0 0 -> xyz=0 0.5147601507271262 0 rpy=0 0 0
- joint 19_20: origin xyz=0 -0.7680019056594278 0 rpy=0 0 0 -> xyz=0 0.1608824740445456 0 rpy=0 0 0
- joint 1_2: origin xyz=-0.421382269444644 0 0 rpy=0 0 0 -> xyz=-0.4561383947668053 0 0 rpy=0 0 0
- joint 20_21: origin xyz=0 -0.16831502906814866 0 rpy=0 0 0 -> xyz=0 0.26627043206239975 0 rpy=0 0 0
- joint 2_3: origin xyz=-0.8134976787654494 0 0 rpy=0 0 0 -> xyz=-0.8410294012002504 0 0 rpy=0 0 0
- joint 3_4: origin xyz=-0.709926816870258 0 0 rpy=0 0 0 -> xyz=-0.8148245701293075 0 0 rpy=0 0 0
- joint 4_5: origin xyz=-0.9629561340392867 0 0 rpy=0 0 0 -> xyz=-0.056167770504606085 0 0 rpy=0 0 0
- joint 5_6: origin xyz=-0.3871942437204503 0 0 rpy=0 0 0 -> xyz=-0.26427949599189327 0 0 rpy=0 0 0
- joint 7_8: origin xyz=-0.30424092407817216 0 0 rpy=0 0 0 -> xyz=0.7845833275216404 0 0 rpy=0 0 0
- joint 9_10: origin xyz=0.47532148543576647 0 0 rpy=0 0 0 -> xyz=0.8988883112505559 0 0 rpy=0 0 0

Commit message: commit

File: body.urdf (robot description, URDF)
Before this commit: robot robot, 22 links, 21 joints
Links:
- added link 22, mass 1; collision box size=1.2079261061107076 0.5167735699331193 1.0628215892302557; visual box size=1.2079261061107076 0.5167735699331193 1.0628215892302557
- added link 23, mass 1; collision box size=0.5078678594291194 0.9283672302573892 0.6026901189324503; visual box size=0.5078678594291194 0.9283672302573892 0.6026901189324503
- added link 24, mass 1; collision box size=1.0829449225668526 0.9165676564516637 1.083947845908103; visual box size=1.0829449225668526 0.9165676564516637 1.083947845908103
- added link 25, mass 1; collision box size=1.2801462521571376 1.279855832593107 1.116237131328702; visual box size=1.2801462521571376 1.279855832593107 1.116237131328702
- link 0: geometry collision box size=1.2627566359170785 1.2961242100682833 0.6485001319658493; visual box size=1.2627566359170785 1.2961242100682833 0.6485001319658493
- link 1: geometry collision box size=0.6590990674730851 0.9294944514419887 1.1392419269137668; visual box size=0.6590990674730851 0.9294944514419887 1.1392419269137668
- link 10: geometry collision box size=1.1652614119718296 0.5921064724983778 1.0111066707995695; visual box size=1.1652614119718296 0.5921064724983778 1.0111066707995695
- link 11: geometry collision box size=0.7257910509952685 0.8918526341710729 0.9639424672995165; visual box size=0.7257910509952685 0.8918526341710729 0.9639424672995165
- link 12: geometry collision box size=1.2903928209129916 1.4841686273435282 1.4072044571488282; visual box size=1.2903928209129916 1.4841686273435282 1.4072044571488282
- link 13: geometry collision box size=1.2996815301224407 1.0179436554831975 1.2496621517768847; visual box size=1.2996815301224407 1.0179436554831975 1.2496621517768847
- link 14: geometry collision box size=1.4617822170188706 0.7520095411194454 0.6150554695862274; visual box size=1.4617822170188706 0.7520095411194454 0.6150554695862274
- link 15: geometry collision box size=0.7189477157817482 0.6570660113612115 1.3308458109450627; visual box size=0.7189477157817482 0.6570660113612115 1.3308458109450627
- link 16: geometry collision box size=1.279997264115927 0.984296790701333 0.8782683275325326; visual box size=1.279997264115927 0.984296790701333 0.8782683275325326
- link 17: geometry collision box size=0.8223089265385084 0.7906416780416502 1.221166967163319; visual box size=0.8223089265385084 0.7906416780416502 1.221166967163319
- link 18: geometry collision box size=1.029999447725717 1.2981311974185483 0.5598119189816206; visual box size=1.029999447725717 1.2981311974185483 0.5598119189816206
- link 19: geometry collision box size=0.7520689903426899 1.1689798385760726 1.4467224750229302; visual box size=0.7520689903426899 1.1689798385760726 1.4467224750229302
- link 2: geometry collision box size=1.4743783164672537 1.0052614870989545 0.6252761937478193; visual box size=1.4743783164672537 1.0052614870989545 0.6252761937478193
- link 20: geometry collision box size=1.2713981087649562 1.374041853769826 1.1442840078405545; visual box size=1.2713981087649562 1.374041853769826 1.1442840078405545
- link 21: geometry collision box size=0.9737971454513603 0.8642984563430406 0.8024761969296237; visual box size=0.9737971454513603 0.8642984563430406 0.8024761969296237
- link 3: geometry collision box size=0.9204475680991742 0.9635915531424264 0.8829391545866059; visual box size=0.9204475680991742 0.9635915531424264 0.8829391545866059
- link 4: geometry collision box size=0.5145870679693659 1.1891049881431903 0.8453951417807416; visual box size=0.5145870679693659 1.1891049881431903 0.8453951417807416
- link 5: geometry collision box size=0.8606013984458336 0.9851465492398848 1.3639349040801925; visual box size=0.8606013984458336 0.9851465492398848 1.3639349040801925
- link 6: geometry collision box size=0.7852162461437203 1.214116784691261 0.5370164413812284; visual box size=0.7852162461437203 1.214116784691261 0.5370164413812284
- link 7: geometry collision box size=1.1773432431003106 1.3188665367607504 1.0191136688148477; visual box size=1.1773432431003106 1.3188665367607504 1.0191136688148477
- link 8: geometry collision box size=1.1520574370760541 0.9186844309585493 0.7625799988978774; visual box size=1.1520574370760541 0.9186844309585493 0.7625799988978774
- link 9: geometry collision box size=0.5000824420419352 0.9416564132025538 0.5235083082741483; visual box size=0.5000824420419352 0.9416564132025538 0.5235083082741483
Joints:
- removed joint 13_14
- removed joint 19_20
- removed joint 1_12
- removed joint 1_17
- removed joint 1_7
- removed joint 7_8
- added joint 11_12: type revolute, parent 11, child 12, origin xyz=0.7257910509952685 0 0 rpy=0 0 0, axis 0 1 0, limit lower=-3.14159 upper=3.14159 effort=0.0 velocity=0.0
- added joint 16_17: type revolute, parent 16, child 17, origin xyz=0 -0.984296790701333 0 rpy=0 0 0, axis 1 0 0, limit lower=-3.14159 upper=3.14159 effort=0.0 velocity=0.0
- added joint 1_14: type revolute, parent 1, child 14, origin xyz=0 -0.46474722572099436 0 rpy=0 0 0, axis 1 0 0, limit lower=-3.14159 upper=3.14159 effort=0.0 velocity=0.0
- added joint 1_20: type revolute, parent 1, child 20, origin xyz=0 0.46474722572099436 0 rpy=0 0 0, axis 1 0 0, limit lower=-3.14159 upper=3.14159 effort=0.0 velocity=0.0
- added joint 1_8: type revolute, parent 1, child 8, origin xyz=0.32954953373654255 0 0 rpy=0 0 0, axis 0 1 0, limit lower=-3.14159 upper=3.14159 effort=0.0 velocity=0.0
- added joint 21_22: type revolute, parent 21, child 22, origin xyz=0 0.8642984563430406 0 rpy=0 0 0, axis 1 0 0, limit lower=-3.14159 upper=3.14159 effort=0.0 velocity=0.0
- added joint 22_23: type revolute, parent 22, child 23, origin xyz=0 0.5167735699331193 0 rpy=0 0 0, axis 1 0 0, limit lower=-3.14159 upper=3.14159 effort=0.0 velocity=0.0
- added joint 23_24: type revolute, parent 23, child 24, origin xyz=0 0.9283672302573892 0 rpy=0 0 0, axis 1 0 0, limit lower=-3.14159 upper=3.14159 effort=0.0 velocity=0.0
- added joint 24_25: type revolute, parent 24, child 25, origin xyz=0 0.9165676564516637 0 rpy=0 0 0, axis 1 0 0, limit lower=-3.14159 upper=3.14159 effort=0.0 velocity=0.0
- added joint 6_7: type revolute, parent 6, child 7, origin xyz=-0.7852162461437203 0 0 rpy=0 0 0, axis 0 1 0, limit lower=-3.14159 upper=3.14159 effort=0.0 velocity=0.0
- joint 0_1: origin xyz=0 0 0.19467511196622322 rpy=0 0 0 -> xyz=0 0 0.6485001319658493 rpy=0 0 0
- joint 10_11: origin xyz=0.40276276758908025 0 0 rpy=0 0 0 -> xyz=1.1652614119718296 0 0 rpy=0 0 0
- joint 12_13: axis 1 0 0 -> 0 1 0; origin xyz=0 -0.5207200162487802 0 rpy=0 0 0 -> xyz=1.2903928209129916 0 0 rpy=0 0 0
- joint 14_15: origin xyz=0 -0.8290522262573269 0 rpy=0 0 0 -> xyz=0 -0.7520095411194454 0 rpy=0 0 0
- joint 15_16: origin xyz=0 -0.18865421848377062 0 rpy=0 0 0 -> xyz=0 -0.6570660113612115 0 rpy=0 0 0
- joint 17_18: origin xyz=0 0.31320371856655904 0 rpy=0 0 0 -> xyz=0 -0.7906416780416502 0 rpy=0 0 0
- joint 18_19: origin xyz=0 0.5147601507271262 0 rpy=0 0 0 -> xyz=0 -1.2981311974185483 0 rpy=0 0 0
- joint 1_2: origin xyz=-0.4561383947668053 0 0 rpy=0 0 0 -> xyz=-0.32954953373654255 0 0 rpy=0 0 0
- joint 20_21: origin xyz=0 0.26627043206239975 0 rpy=0 0 0 -> xyz=0 1.374041853769826 0 rpy=0 0 0
- joint 2_3: origin xyz=-0.8410294012002504 0 0 rpy=0 0 0 -> xyz=-1.4743783164672537 0 0 rpy=0 0 0
- joint 3_4: origin xyz=-0.8148245701293075 0 0 rpy=0 0 0 -> xyz=-0.9204475680991742 0 0 rpy=0 0 0
- joint 4_5: origin xyz=-0.056167770504606085 0 0 rpy=0 0 0 -> xyz=-0.5145870679693659 0 0 rpy=0 0 0
- joint 5_6: origin xyz=-0.26427949599189327 0 0 rpy=0 0 0 -> xyz=-0.8606013984458336 0 0 rpy=0 0 0
- joint 8_9: origin xyz=0.4893250477731339 0 0 rpy=0 0 0 -> xyz=1.1520574370760541 0 0 rpy=0 0 0
- joint 9_10: origin xyz=0.8988883112505559 0 0 rpy=0 0 0 -> xyz=0.5000824420419352 0 0 rpy=0 0 0
