Commit message: commit

File: body.urdf (robot description, URDF)
Before this commit: robot robot, 26 links, 25 joints
Links:
- added link 26, mass 1; collision box size=1.182651623118462 0.9697200587474879 1.2300319811622105; visual box size=1.182651623118462 0.9697200587474879 1.2300319811622105
- added link 27, mass 1; collision box size=1.2495962439109154 0.9717308058936879 0.748364865209505; visual box size=1.2495962439109154 0.9717308058936879 0.748364865209505
- added link 28, mass 1; collision box size=1.0337643186019192 0.5197212597187995 0.8702291991251845; visual box size=1.0337643186019192 0.5197212597187995 0.8702291991251845
- added link 29, mass 1; collision box size=1.4583089188639076 0.8412454219440353 1.0678643879364673; visual box size=1.4583089188639076 0.8412454219440353 1.0678643879364673
- link 0: geometry collision box size=0.8746202316741509 1.3622074626411367 0.5790046736399407; visual box size=0.8746202316741509 1.3622074626411367 0.5790046736399407
- link 1: geometry collision box size=1.4897177289208372 1.4398741057968372 0.98369275734712; visual box size=1.4897177289208372 1.4398741057968372 0.98369275734712
- link 10: geometry collision box size=1.038367807708777 0.9346084155129871 1.1470421557890775; visual box size=1.038367807708777 0.9346084155129871 1.1470421557890775
- link 11: geometry collision box size=0.5918594429245907 0.8715871795335866 0.8050535803663055; visual box size=0.5918594429245907 0.8715871795335866 0.8050535803663055
- link 12: geometry collision box size=1.094281473167582 0.7701176791003863 1.323486710219953; visual box size=1.094281473167582 0.7701176791003863 1.323486710219953
- link 13: geometry collision box size=0.7480414220258839 1.4659657402092792 1.1146167764156316; visual box size=0.7480414220258839 1.4659657402092792 1.1146167764156316
- link 14: geometry collision box size=1.2072118740758417 1.2132514214840102 0.921708121126595; visual box size=1.2072118740758417 1.2132514214840102 0.921708121126595
- link 15: geometry collision box size=1.28612339717762 0.5047711883267749 0.7135904743735425; visual box size=1.28612339717762 0.5047711883267749 0.7135904743735425
- link 16: geometry collision box size=0.9276886205633367 1.3267246639475487 0.5369953368509427; visual box size=0.9276886205633367 1.3267246639475487 0.5369953368509427
- link 17: geometry collision box size=0.6389093150776591 1.2064207260023943 1.2862836492588636; visual box size=0.6389093150776591 1.2064207260023943 1.2862836492588636
- link 18: geometry collision box size=0.8815507788068854 0.8764382312028642 0.5947395714556597; visual box size=0.8815507788068854 0.8764382312028642 0.5947395714556597
- link 19: geometry collision box size=0.6978030397802202 1.2245650790350997 0.6199094664378165; visual box size=0.6978030397802202 1.2245650790350997 0.6199094664378165
- link 2: geometry collision box size=1.217398045582362 1.0718342861032721 1.277855476216156; visual box size=1.217398045582362 1.0718342861032721 1.277855476216156
- link 20: geometry collision box size=1.013277340864016 0.9813170217703513 0.5973014796389583; visual box size=1.013277340864016 0.9813170217703513 0.5973014796389583
- link 21: geometry collision box size=0.9706264442220659 0.9725067478526005 0.5527055883139228; visual box size=0.9706264442220659 0.9725067478526005 0.5527055883139228
- link 22: geometry collision box size=1.4787060404861645 1.3683533801472179 1.389478002634841; visual box size=1.4787060404861645 1.3683533801472179 1.389478002634841
- link 23: geometry collision box size=0.7277213479093918 1.1142586394475222 0.9280626637730692; visual box size=0.7277213479093918 1.1142586394475222 0.9280626637730692
- link 24: geometry collision box size=1.1719331543154643 0.6079714533601787 1.0884744234249897; visual box size=1.1719331543154643 0.6079714533601787 1.0884744234249897
- link 25: geometry collision box size=1.3065884129076972 0.8346374386064294 1.2548693992341204; visual box size=1.3065884129076972 0.8346374386064294 1.2548693992341204
- link 3: geometry collision box size=0.8177488962389357 1.1817320034933525 1.4909159984372669; visual box size=0.8177488962389357 1.1817320034933525 1.4909159984372669
- link 4: geometry collision box size=0.7496276789051287 1.3204784589511191 1.1191143993577177; visual box size=0.7496276789051287 1.3204784589511191 1.1191143993577177
- link 5: geometry collision box size=0.7596317999505052 0.9046904326940284 0.5292898080427996; visual box size=0.7596317999505052 0.9046904326940284 0.5292898080427996
- link 6: geometry collision box size=0.5678932575674358 1.2149610354268048 0.9187515249875843; visual box size=0.5678932575674358 1.2149610354268048 0.9187515249875843
- link 7: geometry collision box size=1.3382278101012555 0.960166643751687 1.3868073483861005; visual box size=1.3382278101012555 0.960166643751687 1.3868073483861005
- link 8: geometry collision box size=0.5128598536432615 1.3622119606183016 1.1103777743245573; visual box size=0.5128598536432615 1.3622119606183016 1.1103777743245573
- link 9: geometry collision box size=1.4468511204196597 0.6249332550321411 1.2099073400534395; visual box size=1.4468511204196597 0.6249332550321411 1.2099073400534395
Joints:
- removed joint 15_16
- removed joint 1_14
- removed joint 1_20
- removed joint 1_8
- removed joint 22_23
- removed joint 8_9
- added joint 13_14: type revolute, parent 13, child 14, origin xyz=0.7480414220258839 0 0 rpy=0 0 0, axis 0 1 1, limit lower=-3.14159 upper=3.14159 effort=0.0 velocity=0.0
- added joint 19_20: type revolute, parent 19, child 20, origin xyz=0 -1.2245650790350997 0 rpy=0 0 0, axis 0 1 1, limit lower=-3.14159 upper=3.14159 effort=0.0 velocity=0.0
- added joint 1_16: type revolute, parent 1, child 16, origin xyz=0 -0.7199370528984186 0 rpy=0 0 0, axis 0 1 0, limit lower=-3.14159 upper=3.14159 effort=0.0 velocity=0.0
- added joint 1_23: type revolute, parent 1, child 23, origin xyz=0 0.7199370528984186 0 rpy=0 0 0, axis 1 0 0, limit lower=-3.14159 upper=3.14159 effort=0.0 velocity=0.0
- added joint 1_9: type revolute, parent 1, child 9, origin xyz=0.7448588644604186 0 0 rpy=0 0 0, axis 1 1 0, limit lower=-3.14159 upper=3.14159 effort=0.0 velocity=0.0
- added joint 25_26: type revolute, parent 25, child 26, origin xyz=0 0.8346374386064294 0 rpy=0 0 0, axis 1 1 1, limit lower=-3.14159 upper=3.14159 effort=0.0 velocity=0.0
- added joint 26_27: type revolute, parent 26, child 27, origin xyz=0 0.9697200587474879 0 rpy=0 0 0, axis 0 1 0, limit lower=-3.14159 upper=3.14159 effort=0.0 velocity=0.0
- added joint 27_28: type revolute, parent 27, child 28, origin xyz=0 0.9717308058936879 0 rpy=0 0 0, axis 0 0 1, limit lower=-3.14159 upper=3.14159 effort=0.0 velocity=0.0
- added joint 28_29: type revolute, parent 28, child 29, origin xyz=0 0.5197212597187995 0 rpy=0 0 0, axis 1 1 0, limit lower=-3.14159 upper=3.14159 effort=0.0 velocity=0.0
- added joint 7_8: type revolute, parent 7, child 8, origin xyz=-1.3382278101012555 0 0 rpy=0 0 0, axis 1 1 0, limit lower=-3.14159 upper=3.14159 effort=0.0 velocity=0.0
- joint 0_1: axis 1 1 1 -> 0 1 1; origin xyz=0 0 0.6485001319658493 rpy=0 0 0 -> xyz=0 0 0.5790046736399407 rpy=0 0 0
- joint 10_11: axis 0 1 0 -> 1 1 1; origin xyz=1.1652614119718296 0 0 rpy=0 0 0 -> xyz=1.038367807708777 0 0 rpy=0 0 0
- joint 11_12: axis 0 1 0 -> 0 0 1; origin xyz=0.7257910509952685 0 0 rpy=0 0 0 -> xyz=0.5918594429245907 0 0 rpy=0 0 0
- joint 12_13: axis 0 1 0 -> 0 0 1; origin xyz=1.2903928209129916 0 0 rpy=0 0 0 -> xyz=1.094281473167582 0 0 rpy=0 0 0
- joint 14_15: axis 1 0 0 -> 0 0 1; origin xyz=0 -0.7520095411194454 0 rpy=0 0 0 -> xyz=1.2072118740758417 0 0 rpy=0 0 0
- joint 16_17: axis 1 0 0 -> 1 1 1; origin xyz=0 -0.984296790701333 0 rpy=0 0 0 -> xyz=0 -1.3267246639475487 0 rpy=0 0 0
- joint 17_18: axis 1 0 0 -> 1 1 0; origin xyz=0 -0.7906416780416502 0 rpy=0 0 0 -> xyz=0 -1.2064207260023943 0 rpy=0 0 0
- joint 18_19: axis 1 0 0 -> 0 1 0; origin xyz=0 -1.2981311974185483 0 rpy=0 0 0 -> xyz=0 -0.8764382312028642 0 rpy=0 0 0
- joint 1_2: axis 0 1 0 -> 0 0 1; origin xyz=-0.32954953373654255 0 0 rpy=0 0 0 -> xyz=-0.7448588644604186 0 0 rpy=0 0 0
- joint 20_21: axis 1 0 0 -> 1 0 1; origin xyz=0 1.374041853769826 0 rpy=0 0 0 -> xyz=0 -0.9813170217703513 0 rpy=0 0 0
- joint 21_22: axis 1 0 0 -> 1 1 0; origin xyz=0 0.8642984563430406 0 rpy=0 0 0 -> xyz=0 -0.9725067478526005 0 rpy=0 0 0
- joint 23_24: axis 1 0 0 -> 0 0 1; origin xyz=0 0.9283672302573892 0 rpy=0 0 0 -> xyz=0 1.1142586394475222 0 rpy=0 0 0
- joint 24_25: axis 1 0 0 -> 1 1 0; origin xyz=0 0.9165676564516637 0 rpy=0 0 0 -> xyz=0 0.6079714533601787 0 rpy=0 0 0
- joint 2_3: axis 0 1 0 -> 1 1 0; origin xyz=-1.4743783164672537 0 0 rpy=0 0 0 -> xyz=-1.217398045582362 0 0 rpy=0 0 0
- joint 3_4: axis 0 1 0 -> 1 0 0; origin xyz=-0.9204475680991742 0 0 rpy=0 0 0 -> xyz=-0.8177488962389357 0 0 rpy=0 0 0
- joint 4_5: axis 0 1 0 -> 1 1 0; origin xyz=-0.5145870679693659 0 0 rpy=0 0 0 -> xyz=-0.7496276789051287 0 0 rpy=0 0 0
- joint 5_6: axis 0 1 0 -> 1 0 1; origin xyz=-0.8606013984458336 0 0 rpy=0 0 0 -> xyz=-0.7596317999505052 0 0 rpy=0 0 0
- joint 6_7: axis 0 1 0 -> 1 0 0; origin xyz=-0.7852162461437203 0 0 rpy=0 0 0 -> xyz=-0.5678932575674358 0 0 rpy=0 0 0
- joint 9_10: axis 0 1 0 -> 1 1 0; origin xyz=0.5000824420419352 0 0 rpy=0 0 0 -> xyz=1.4468511204196597 0 0 rpy=0 0 0
