Commit message: commit

File: body8.urdf (robot description, URDF)
Before this commit: robot robot, 26 links, 25 joints
Links:
- link 0: geometry collision box size=0.9351831948565327 0.6863295193631712 0.5189113132658583; visual box size=0.9351831948565327 0.6863295193631712 0.5189113132658583
- link 1: geometry collision box size=0.6588538405696044 1.032807774393872 0.734486704715667; visual box size=0.6588538405696044 1.032807774393872 0.734486704715667
- link 10: geometry collision box size=1.0944192830004047 0.6166471001808986 0.9542927911067252; visual box size=1.0944192830004047 0.6166471001808986 0.9542927911067252
- link 11: geometry collision box size=1.0737006551421828 0.9787355857861331 1.1287079521217025; visual box size=1.0737006551421828 0.9787355857861331 1.1287079521217025
- link 12: geometry collision box size=0.895143240970111 0.9879236470737907 1.4499111218945249; visual box size=0.895143240970111 0.9879236470737907 1.4499111218945249
- link 13: geometry collision box size=0.8259502592893584 1.3580220474456284 1.2422217848344217; visual box size=0.8259502592893584 1.3580220474456284 1.2422217848344217
- link 14: geometry collision box size=1.2487023266711768 1.4733372560572922 0.5440619303180794; visual box size=1.2487023266711768 1.4733372560572922 0.5440619303180794
- link 15: geometry collision box size=0.6846704118248477 0.9467031612315469 1.4180594481362436; visual box size=0.6846704118248477 0.9467031612315469 1.4180594481362436
- link 16: geometry collision box size=0.9154696249972087 1.0319667042132994 1.0529773535102938; visual box size=0.9154696249972087 1.0319667042132994 1.0529773535102938
- link 17: geometry collision box size=1.0064212922344966 1.3950167926695412 0.7594054480355552; visual box size=1.0064212922344966 1.3950167926695412 0.7594054480355552
- link 18: geometry collision box size=0.5765294080234404 0.5756079880593035 0.7517989885131344; visual box size=0.5765294080234404 0.5756079880593035 0.7517989885131344
- link 19: geometry collision box size=0.7021617346085206 1.2873289815015043 0.5256347552241695; visual box size=0.7021617346085206 1.2873289815015043 0.5256347552241695
- link 2: geometry collision box size=1.427297634983474 1.2013530226401243 1.4037270927465793; visual box size=1.427297634983474 1.2013530226401243 1.4037270927465793
- link 20: geometry collision box size=0.5362490309849505 1.0453187850577357 1.0624017808868134; visual box size=0.5362490309849505 1.0453187850577357 1.0624017808868134
- link 21: geometry collision box size=0.9755849096437765 1.3861232536105026 0.8245207172640135; visual box size=0.9755849096437765 1.3861232536105026 0.8245207172640135
- link 22: geometry collision box size=0.5340763490527783 1.1577808714000333 0.8886887166876852; visual box size=0.5340763490527783 1.1577808714000333 0.8886887166876852
- link 23: geometry collision box size=1.1551246088038467 1.1540784260148267 0.6048831177681389; visual box size=1.1551246088038467 1.1540784260148267 0.6048831177681389
- link 24: geometry collision box size=1.3815134474531168 0.8606459403518184 1.2438645793525225; visual box size=1.3815134474531168 0.8606459403518184 1.2438645793525225
- link 25: geometry collision box size=1.1827610244857776 0.5583967853880966 1.247445902110221; visual box size=1.1827610244857776 0.5583967853880966 1.247445902110221
- link 3: geometry collision box size=1.0768783987380166 1.4970609985063095 1.211062804557624; visual box size=1.0768783987380166 1.4970609985063095 1.211062804557624
- link 4: geometry collision box size=1.0304710264057029 1.2143778940930186 1.1869040290140562; visual box size=1.0304710264057029 1.2143778940930186 1.1869040290140562
- link 5: geometry collision box size=1.115628330569768 0.6852979300866507 1.1725260448800456; visual box size=1.115628330569768 0.6852979300866507 1.1725260448800456
- link 6: geometry collision box size=0.7597096202495328 1.2654523829550057 0.6370087259797488; visual box size=0.7597096202495328 1.2654523829550057 0.6370087259797488
- link 7: geometry collision box size=1.143221228891338 1.34517566763612 0.7475309969698671; visual box size=1.143221228891338 1.34517566763612 0.7475309969698671
- link 8: geometry collision box size=1.300311240060878 1.0620340466685356 0.6655902775428125; visual box size=1.300311240060878 1.0620340466685356 0.6655902775428125
- link 9: geometry collision box size=0.7675662846110222 1.1425009918654028 0.8861568737007743; visual box size=0.7675662846110222 1.1425009918654028 0.8861568737007743
Joints:
- joint 0_1: axis 0 1 1 -> 1 1 1; origin xyz=0 0 1.1088774505390555 rpy=0 0 0 -> xyz=0 0 0.5189113132658583 rpy=0 0 0
- joint 10_11: axis 1 1 1 -> 0 1 1; origin xyz=1.1531816267434374 0 0 rpy=0 0 0 -> xyz=1.0944192830004047 0 0 rpy=0 0 0
- joint 11_12: origin xyz=0.8432146919433464 0 0 rpy=0 0 0 -> xyz=1.0737006551421828 0 0 rpy=0 0 0
- joint 12_13: axis 1 1 1 -> 0 1 1; origin xyz=0.804743590207092 0 0 rpy=0 0 0 -> xyz=0.895143240970111 0 0 rpy=0 0 0
- joint 14_15: axis 1 1 1 -> 1 1 0; origin xyz=0 -0.8714020395959037 0 rpy=0 0 0 -> xyz=0 -1.4733372560572922 0 rpy=0 0 0
- joint 15_16: axis 0 1 0 -> 0 0 1; origin xyz=0 -0.8711672804434076 0 rpy=0 0 0 -> xyz=0 -0.9467031612315469 0 rpy=0 0 0
- joint 16_17: axis 1 1 0 -> 1 0 0; origin xyz=0 -1.0149722870240572 0 rpy=0 0 0 -> xyz=0 -1.0319667042132994 0 rpy=0 0 0
- joint 17_18: axis 1 1 0 -> 1 0 0; origin xyz=0 -1.0477021996224758 0 rpy=0 0 0 -> xyz=0 -1.3950167926695412 0 rpy=0 0 0
- joint 18_19: axis 1 0 1 -> 1 0 0; origin xyz=0 -0.702286827424538 0 rpy=0 0 0 -> xyz=0 -0.5756079880593035 0 rpy=0 0 0
- joint 1_14: axis 1 1 1 -> 1 1 0; origin xyz=0 -0.49938939283172495 0 rpy=0 0 0 -> xyz=0 -0.516403887196936 0 rpy=0 0 0
- joint 1_2: axis 1 0 1 -> 0 1 1; origin xyz=-0.6916197365357452 0 0 rpy=0 0 0 -> xyz=-0.3294269202848022 0 0 rpy=0 0 0
- joint 1_20: axis 1 1 0 -> 0 0 1; origin xyz=0 0.49938939283172495 0 rpy=0 0 0 -> xyz=0 0.516403887196936 0 rpy=0 0 0
- joint 1_8: axis 0 1 1 -> 1 1 0; origin xyz=0.6916197365357452 0 0 rpy=0 0 0 -> xyz=0.3294269202848022 0 0 rpy=0 0 0
- joint 20_21: axis 0 1 0 -> 0 0 1; origin xyz=0 0.5454765216200347 0 rpy=0 0 0 -> xyz=0 1.0453187850577357 0 rpy=0 0 0
- joint 21_22: axis 1 1 0 -> 0 0 1; origin xyz=0 0.765878022693122 0 rpy=0 0 0 -> xyz=0 1.3861232536105026 0 rpy=0 0 0
- joint 22_23: axis 1 1 1 -> 0 0 1; origin xyz=0 0.5993230666127954 0 rpy=0 0 0 -> xyz=0 1.1577808714000333 0 rpy=0 0 0
- joint 23_24: axis 0 0 1 -> 0 1 1; origin xyz=0 1.4722674959905344 0 rpy=0 0 0 -> xyz=0 1.1540784260148267 0 rpy=0 0 0
- joint 24_25: axis 1 1 0 -> 0 0 1; origin xyz=0 1.3058575389062101 0 rpy=0 0 0 -> xyz=0 0.8606459403518184 0 rpy=0 0 0
- joint 2_3: axis 1 0 0 -> 0 1 0; origin xyz=-1.405281650226796 0 0 rpy=0 0 0 -> xyz=-1.427297634983474 0 0 rpy=0 0 0
- joint 3_4: axis 0 1 1 -> 0 1 0; origin xyz=-0.8929928358687664 0 0 rpy=0 0 0 -> xyz=-1.0768783987380166 0 0 rpy=0 0 0
- joint 4_5: axis 1 1 0 -> 1 0 1; origin xyz=-0.6385567790346584 0 0 rpy=0 0 0 -> xyz=-1.0304710264057029 0 0 rpy=0 0 0
- joint 5_6: axis 1 0 0 -> 0 1 1; origin xyz=-1.1841964361392323 0 0 rpy=0 0 0 -> xyz=-1.115628330569768 0 0 rpy=0 0 0
- joint 6_7: axis 0 1 1 -> 1 1 0; origin xyz=-0.6218434345403399 0 0 rpy=0 0 0 -> xyz=-0.7597096202495328 0 0 rpy=0 0 0
- joint 8_9: axis 1 0 1 -> 1 1 1; origin xyz=0.7773028878045448 0 0 rpy=0 0 0 -> xyz=1.300311240060878 0 0 rpy=0 0 0
- joint 9_10: origin xyz=0.7808296374438785 0 0 rpy=0 0 0 -> xyz=0.7675662846110222 0 0 rpy=0 0 0
