Commit message: commit

File: body0.urdf (robot description, URDF)
Before this commit: robot robot, 41 links, 40 joints
Links:
- removed link 17
- removed link 18
- removed link 19
- removed link 20
- removed link 21
- removed link 22
- removed link 23
- removed link 24
- removed link 25
- removed link 26
- removed link 27
- removed link 28
- removed link 29
- removed link 30
- removed link 31
- removed link 32
- removed link 33
- removed link 34
- removed link 35
- removed link 36
- removed link 37
- removed link 38
- removed link 39
- removed link 40
- link 0: geometry collision box size=1.5 1.5 0.8; visual box size=1.5 1.5 0.8
- link 1: geometry collision box size=0.6702345426989633 0.21287209693449805 0.37159576182471377; visual box size=0.6702345426989633 0.21287209693449805 0.37159576182471377
- link 10: geometry collision box size=0.46879324816473966 0.2597146778920525 1.197705955447554; visual box size=0.46879324816473966 0.2597146778920525 1.197705955447554
- link 11: geometry collision box size=0.4662353596470955 0.7955502272599311 0.2710188445761256; visual box size=0.4662353596470955 0.7955502272599311 0.2710188445761256
- link 12: geometry collision box size=0.07642053723271125 0.5006620783473082 0.13127519997632053; visual box size=0.07642053723271125 0.5006620783473082 0.13127519997632053
- link 13: geometry collision box size=0.5024662383423795 0.3780543288283582 0.6728061909327361; visual box size=0.5024662383423795 0.3780543288283582 0.6728061909327361
- link 14: geometry collision box size=0.5932290619888556 0.31454518925058506 1.275105207340246; visual box size=0.5932290619888556 0.31454518925058506 1.275105207340246
- link 15: geometry collision box size=0.23833191774039897 0.7042817960903667 0.2493924332519192; visual box size=0.23833191774039897 0.7042817960903667 0.2493924332519192
- link 16: geometry collision box size=0.06842433539386872 0.7112248843641235 0.07550235940783487; visual box size=0.06842433539386872 0.7112248843641235 0.07550235940783487
- link 2: geometry collision box size=0.8989833854012441 0.6091583059084927 0.6845951070633703; visual box size=0.8989833854012441 0.6091583059084927 0.6845951070633703
- link 3: geometry collision box size=0.8584767690814185 0.42609111552644063 0.05157313386257725; visual box size=0.8584767690814185 0.42609111552644063 0.05157313386257725
- link 4: geometry collision box size=0.9765802679423216 0.903851121819558 0.8638317590740525; visual box size=0.9765802679423216 0.903851121819558 0.8638317590740525
- link 5: geometry collision box size=0.011959510140161389 0.9040537748160613 0.8252821159519917; visual box size=0.011959510140161389 0.9040537748160613 0.8252821159519917
- link 6: geometry collision box size=0.7009180718395827 0.07313384807432288 0.4674553661300461; visual box size=0.7009180718395827 0.07313384807432288 0.4674553661300461
- link 7: geometry collision box size=0.9820940913361346 0.39034657585124033 0.21551419053083565; visual box size=0.9820940913361346 0.39034657585124033 0.21551419053083565
- link 8: geometry collision box size=0.4386293816665944 0.32567144046738017 0.9170304433391184; visual box size=0.4386293816665944 0.32567144046738017 0.9170304433391184
- link 9: geometry collision box size=0.9318344076992425 0.7019440096288151 0.30822533083970827; visual box size=0.9318344076992425 0.7019440096288151 0.30822533083970827
Joints:
- removed joint 0_11
- removed joint 0_21
- removed joint 0_31
- removed joint 12_13
- removed joint 16_17
- removed joint 17_18
- removed joint 18_19
- removed joint 19_20
- removed joint 21_22
- removed joint 22_23
- removed joint 23_24
- removed joint 24_25
- removed joint 25_26
- removed joint 26_27
- removed joint 27_28
- removed joint 28_29
- removed joint 29_30
- removed joint 31_32
- removed joint 32_33
- removed joint 33_34
- removed joint 34_35
- removed joint 35_36
- removed joint 36_37
- removed joint 37_38
- removed joint 38_39
- removed joint 39_40
- removed joint 4_5
- removed joint 8_9
- added joint 0_13: type revolute, parent 0, child 13, origin xyz=0 0.75 2 rpy=0 0 0, axis 0 1 0, limit lower=-3.14159 upper=3.14159 effort=0.0 velocity=0.0
- added joint 0_5: type revolute, parent 0, child 5, origin xyz=0.75 0 2 rpy=0 0 0, axis 0 1 1, limit lower=-3.14159 upper=3.14159 effort=0.0 velocity=0.0
- added joint 0_9: type revolute, parent 0, child 9, origin xyz=0 -0.75 2 rpy=0 0 0, axis 0 1 0, limit lower=-3.14159 upper=3.14159 effort=0.0 velocity=0.0
- added joint 10_11: type revolute, parent 10, child 11, origin xyz=0 0 -1.197705955447554 rpy=0 0 0, axis 1 0 1, limit lower=-3.14159 upper=3.14159 effort=0.0 velocity=0.0
- joint 0_1: axis 1 0 0 -> 1 1 0; origin xyz=-0.4008816538630179 0 4 rpy=0 0 0 -> xyz=-0.75 0 2 rpy=0 0 0
- joint 11_12: axis 1 0 1 -> 0 0 1; origin xyz=0.5569123051303049 0 0 rpy=0 0 0 -> xyz=0 0 -0.2710188445761256 rpy=0 0 0
- joint 13_14: axis 1 0 0 -> 0 1 0; origin xyz=1.4241550221860866 0 0 rpy=0 0 0 -> xyz=0 0.1890271644141791 -0.33640309546636804 rpy=0 0 0
- joint 14_15: axis 0 1 0 -> 1 1 0; origin xyz=1.3125101086905333 0 0 rpy=0 0 0 -> xyz=0 0 -1.275105207340246 rpy=0 0 0
- joint 15_16: axis 1 0 1 -> 1 1 0; origin xyz=0.6573445162833567 0 0 rpy=0 0 0 -> xyz=0 0 -0.2493924332519192 rpy=0 0 0
- joint 1_2: axis 1 0 0 -> 0 1 0; origin xyz=-0.5217629097272315 0 0 rpy=0 0 0 -> xyz=-0.33511727134948166 0 -0.18579788091235688 rpy=0 0 0
- joint 2_3: origin xyz=-1.351861460581996 0 0 rpy=0 0 0 -> xyz=0 0 -0.6845951070633703 rpy=0 0 0
- joint 3_4: axis 1 0 1 -> 0 1 0; origin xyz=-0.6643527714711773 0 0 rpy=0 0 0 -> xyz=0 0 -0.05157313386257725 rpy=0 0 0
- joint 5_6: axis 1 0 0 -> 1 1 0; origin xyz=-1.1905912906462432 0 0 rpy=0 0 0 -> xyz=0.0059797550700806945 0 -0.4126410579759959 rpy=0 0 0
- joint 6_7: axis 0 0 1 -> 1 1 0; origin xyz=-1.234049107638493 0 0 rpy=0 0 0 -> xyz=0 0 -0.4674553661300461 rpy=0 0 0
- joint 7_8: origin xyz=-0.5953675322894127 0 -0.45663801285028977 rpy=0 0 0 -> xyz=0 0 -0.21551419053083565 rpy=0 0 0
- joint 9_10: origin xyz=0 0 -1.2622944437097354 rpy=0 0 0 -> xyz=0 -0.35097200481440755 -0.15411266541985413 rpy=0 0 0

File: body1.urdf (robot description, URDF)
Before this commit: robot robot, 33 links, 32 joints
Links:
- removed link 29
- removed link 30
- removed link 31
- removed link 32
- link 0: geometry collision box size=1.5 1.5 0.8; visual box size=1.5 1.5 0.8
- link 1: geometry collision box size=0.5126919324777913 0.7250848360421205 0.6766733458425387; visual box size=0.5126919324777913 0.7250848360421205 0.6766733458425387
- link 10: geometry collision box size=0.5676691240743692 0.5837109934343283 0.38486369148582156; visual box size=0.5676691240743692 0.5837109934343283 0.38486369148582156
- link 11: geometry collision box size=0.3011352872397415 0.0392068794767767 0.1720421449356887; visual box size=0.3011352872397415 0.0392068794767767 0.1720421449356887
- link 12: geometry collision box size=0.7067909068291881 0.40114093418263363 0.28302003313781904; visual box size=0.7067909068291881 0.40114093418263363 0.28302003313781904
- link 13: geometry collision box size=0.11547933711655733 0.2640037584646495 1.159030535521866; visual box size=0.11547933711655733 0.2640037584646495 1.159030535521866
- link 14: geometry collision box size=0.9070504564632319 0.993336897168533 0.15794943134031514; visual box size=0.9070504564632319 0.993336897168533 0.15794943134031514
- link 15: geometry collision box size=0.6622726260350417 0.6772169183529062 0.14585411885173627; visual box size=0.6622726260350417 0.6772169183529062 0.14585411885173627
- link 16: geometry collision box size=0.8366007721626993 0.4269871454216021 0.4067008534918739; visual box size=0.8366007721626993 0.4269871454216021 0.4067008534918739
- link 17: geometry collision box size=0.7098465212767554 0.8305211523512608 0.006355232711636072; visual box size=0.7098465212767554 0.8305211523512608 0.006355232711636072
- link 18: geometry collision box size=0.7872751519827784 0.49615788342725275 0.1451367674689985; visual box size=0.7872751519827784 0.49615788342725275 0.1451367674689985
- link 19: geometry collision box size=0.5199661668432042 0.6266582951084588 1.4277303665203707; visual box size=0.5199661668432042 0.6266582951084588 1.4277303665203707
- link 2: geometry collision box size=0.26643980550734525 0.6056395960002187 0.8429219739471231; visual box size=0.26643980550734525 0.6056395960002187 0.8429219739471231
- link 20: geometry collision box size=0.6172644269979802 0.6590512564067744 0.08703985776590724; visual box size=0.6172644269979802 0.6590512564067744 0.08703985776590724
- link 21: geometry collision box size=0.8576849083477198 0.691832546171722 0.08522977571372219; visual box size=0.8576849083477198 0.691832546171722 0.08522977571372219
- link 22: geometry collision box size=0.45214459164414367 0.6359521381373019 0.46169478193927416; visual box size=0.45214459164414367 0.6359521381373019 0.46169478193927416
- link 23: geometry collision box size=0.8872114184635592 0.6084636674703443 0.1638347728830657; visual box size=0.8872114184635592 0.6084636674703443 0.1638347728830657
- link 24: geometry collision box size=0.32168729304931554 0.6049892320501622 0.5187321613744026; visual box size=0.32168729304931554 0.6049892320501622 0.5187321613744026
- link 25: geometry collision box size=0.5133776798653343 0.7025180963276974 0.08975757152889519; visual box size=0.5133776798653343 0.7025180963276974 0.08975757152889519
- link 26: geometry collision box size=0.8209785906551847 0.1539099406362504 1.5262864467383297; visual box size=0.8209785906551847 0.1539099406362504 1.5262864467383297
- link 27: geometry collision box size=0.8842619639665266 0.9505686631599713 0.05910438275453276; visual box size=0.8842619639665266 0.9505686631599713 0.05910438275453276
- link 28: geometry collision box size=0.6189010058554533 0.07218414474188206 0.014609170507137635; visual box size=0.6189010058554533 0.07218414474188206 0.014609170507137635
- link 3: geometry collision box size=0.7385440566924593 0.04486902995547781 0.5631316447009382; visual box size=0.7385440566924593 0.04486902995547781 0.5631316447009382
- link 4: geometry collision box size=0.985353577516576 0.12164266320213613 0.5024067309299646; visual box size=0.985353577516576 0.12164266320213613 0.5024067309299646
- link 5: geometry collision box size=0.8340961985163321 0.517068305912865 0.33122092922989044; visual box size=0.8340961985163321 0.517068305912865 0.33122092922989044
- link 6: geometry collision box size=0.6410204634145508 0.8087951894904831 0.9622351898784216; visual box size=0.6410204634145508 0.8087951894904831 0.9622351898784216
- link 7: geometry collision box size=0.14061779712318845 0.8013829556516872 0.30654388089168805; visual box size=0.14061779712318845 0.8013829556516872 0.30654388089168805
- link 8: geometry collision box size=0.9049937149172881 0.01828122990373382 0.9228063026115582; visual box size=0.9049937149172881 0.01828122990373382 0.9228063026115582
- link 9: geometry collision box size=0.751879339325681 0.026706143992640596 0.4744201685651175; visual box size=0.751879339325681 0.026706143992640596 0.4744201685651175
Joints:
- removed joint 0_17
- removed joint 0_25
- removed joint 0_9
- removed joint 14_15
- removed joint 21_22
- removed joint 28_29
- removed joint 29_30
- removed joint 30_31
- removed joint 31_32
- removed joint 7_8
- added joint 0_15: type revolute, parent 0, child 15, origin xyz=0 -0.75 2 rpy=0 0 0, axis 0 0 1, limit lower=-3.14159 upper=3.14159 effort=0.0 velocity=0.0
- added joint 0_22: type revolute, parent 0, child 22, origin xyz=0 0.75 2 rpy=0 0 0, axis 0 0 1, limit lower=-3.14159 upper=3.14159 effort=0.0 velocity=0.0
- added joint 0_8: type revolute, parent 0, child 8, origin xyz=0.75 0 2 rpy=0 0 0, axis 0 1 0, limit lower=-3.14159 upper=3.14159 effort=0.0 velocity=0.0
- added joint 16_17: type revolute, parent 16, child 17, origin xyz=0 -0.4269871454216021 0 rpy=0 0 0, axis 1 0 0, limit lower=-3.14159 upper=3.14159 effort=0.0 velocity=0.0
- added joint 24_25: type revolute, parent 24, child 25, origin xyz=0 0.6049892320501622 0 rpy=0 0 0, axis 0 0 1, limit lower=-3.14159 upper=3.14159 effort=0.0 velocity=0.0
- added joint 8_9: type revolute, parent 8, child 9, origin xyz=0.9049937149172881 0 0 rpy=0 0 0, axis 0 1 0, limit lower=-3.14159 upper=3.14159 effort=0.0 velocity=0.0
- joint 0_1: axis 0 0 1 -> 1 1 0; origin xyz=-0.4409059417523364 0 4 rpy=0 0 0 -> xyz=-0.75 0 2 rpy=0 0 0
- joint 10_11: axis 1 1 0 -> 1 0 0; origin xyz=0.5210289899762637 0 0 rpy=0 0 0 -> xyz=0.5676691240743692 0 0 rpy=0 0 0
- joint 11_12: axis 0 0 1 -> 1 0 0; origin xyz=1.3056761688912237 0 0 rpy=0 0 0 -> xyz=0.15056764361987074 0 -0.08602107246784435 rpy=0 0 0
- joint 12_13: axis 1 0 1 -> 1 0 0; origin xyz=0.7632051336208211 0 0 rpy=0 0 0 -> xyz=0 0 -0.28302003313781904 rpy=0 0 0
- joint 13_14: axis 1 1 1 -> 0 1 0; origin xyz=0.6736187866683107 0 -0.3902027771574174 rpy=0 0 0 -> xyz=0 0 -1.159030535521866 rpy=0 0 0
- joint 15_16: axis 0 0 1 -> 1 0 1; origin xyz=0 0 -0.2722842383379379 rpy=0 0 0 -> xyz=0 -0.6772169183529062 0 rpy=0 0 0
- joint 17_18: axis 1 1 1 -> 1 0 0; origin xyz=0 -0.5558097307557481 0 rpy=0 0 0 -> xyz=0 -0.8305211523512608 0 rpy=0 0 0
- joint 18_19: axis 1 0 1 -> 1 0 0; origin xyz=0 -0.926607874783237 0 rpy=0 0 0 -> xyz=0 -0.24807894171362638 -0.07256838373449925 rpy=0 0 0
- joint 19_20: axis 0 1 0 -> 1 1 0; origin xyz=0 -0.8731979453417321 0 rpy=0 0 0 -> xyz=0 0 -1.4277303665203707 rpy=0 0 0
- joint 1_2: axis 0 1 0 -> 1 1 1; origin xyz=-1.0803652337860519 0 0 rpy=0 0 0 -> xyz=-0.5126919324777913 0 0 rpy=0 0 0
- joint 20_21: axis 0 1 0 -> 1 0 0; origin xyz=0 -1.4816644037524593 0 rpy=0 0 0 -> xyz=0 0 -0.08703985776590724 rpy=0 0 0
- joint 22_23: axis 1 0 0 -> 1 0 1; origin xyz=0 0 -2.7737875428246808 rpy=0 0 0 -> xyz=0 0.6359521381373019 0 rpy=0 0 0
- joint 23_24: axis 0 1 1 -> 1 0 1; origin xyz=0 0 -0.2754737246596185 rpy=0 0 0 -> xyz=0 0.6084636674703443 0 rpy=0 0 0
- joint 25_26: axis 1 0 0 -> 1 0 1; origin xyz=0 0.779002826021134 0 rpy=0 0 0 -> xyz=0 0.3512590481638487 -0.04487878576444759 rpy=0 0 0
- joint 26_27: axis 0 0 1 -> 1 0 1; origin xyz=0 1.4719335000233407 0 rpy=0 0 0 -> xyz=0 0 -1.5262864467383297 rpy=0 0 0
- joint 27_28: axis 0 1 0 -> 1 0 1; origin xyz=0 1.4033096482833392 0 rpy=0 0 0 -> xyz=0 0 -0.05910438275453276 rpy=0 0 0
- joint 2_3: axis 1 0 1 -> 0 0 1; origin xyz=-0.8648230755338585 0 0 rpy=0 0 0 -> xyz=-0.26643980550734525 0 0 rpy=0 0 0
- joint 3_4: axis 0 1 0 -> 1 1 1; origin xyz=-0.7890238396428964 0 0 rpy=0 0 0 -> xyz=-0.7385440566924593 0 0 rpy=0 0 0
- joint 4_5: axis 1 1 1 -> 0 1 0; origin xyz=-0.599589396708943 0 0 rpy=0 0 0 -> xyz=-0.492676788758288 0 -0.2512033654649823 rpy=0 0 0
- joint 5_6: axis 1 1 1 -> 0 1 1; origin xyz=-0.5285800787729784 0 -0.5957495236075203 rpy=0 0 0 -> xyz=0 0 -0.33122092922989044 rpy=0 0 0
- joint 6_7: axis 1 0 0 -> 1 1 0; origin xyz=0 0 -1.8372445085430886 rpy=0 0 0 -> xyz=0 0 -0.9622351898784216 rpy=0 0 0
- joint 9_10: axis 1 1 1 -> 1 0 1; origin xyz=1.2496144706419725 0 0 rpy=0 0 0 -> xyz=0.751879339325681 0 0 rpy=0 0 0

File: body2.urdf (robot description, URDF)
Before this commit: robot robot, 33 links, 32 joints
Links:
- removed link 17
- removed link 18
- removed link 19
- removed link 20
- removed link 21
- removed link 22
- removed link 23
- removed link 24
- removed link 25
- removed link 26
- removed link 27
- removed link 28
- removed link 29
- removed link 30
- removed link 31
- removed link 32
- link 0: geometry collision box size=1.5 1.5 0.8; visual box size=1.5 1.5 0.8
- link 1: geometry collision box size=0.9030762260385637 0.20517425253158905 0.8330806028345026; visual box size=0.9030762260385637 0.20517425253158905 0.8330806028345026
- link 10: geometry collision box size=0.37349353794806484 0.863717117491277 0.010179508229267498; visual box size=0.37349353794806484 0.863717117491277 0.010179508229267498
- link 11: geometry collision box size=0.6417276301103257 0.2924296284594907 1.5168762766021917; visual box size=0.6417276301103257 0.2924296284594907 1.5168762766021917
- link 12: geometry collision box size=0.6522115054883146 0.6743761836458936 0.07294421516854088; visual box size=0.6522115054883146 0.6743761836458936 0.07294421516854088
- link 13: geometry collision box size=0.9514197919805734 0.43617830035769733 0.3293468218797; visual box size=0.9514197919805734 0.43617830035769733 0.3293468218797
- link 14: geometry collision box size=0.7532692362111783 0.28254001864148315 0.1671641089637273; visual box size=0.7532692362111783 0.28254001864148315 0.1671641089637273
- link 15: geometry collision box size=0.40661978033690405 0.014146890684940239 0.7154577019836661; visual box size=0.40661978033690405 0.014146890684940239 0.7154577019836661
- link 16: geometry collision box size=0.7224860995059165 0.8855017909520231 0.7173781890526068; visual box size=0.7224860995059165 0.8855017909520231 0.7173781890526068
- link 2: geometry collision box size=0.2036520670117472 0.36634164080411824 0.9711447529790068; visual box size=0.2036520670117472 0.36634164080411824 0.9711447529790068
- link 3: geometry collision box size=0.8754101210999268 0.7104793416614378 0.37664274529537023; visual box size=0.8754101210999268 0.7104793416614378 0.37664274529537023
- link 4: geometry collision box size=0.4521959486945568 0.8509237039125549 0.25221250172562304; visual box size=0.4521959486945568 0.8509237039125549 0.25221250172562304
- link 5: geometry collision box size=0.5855378179212705 0.04680711699677431 0.8614572040206672; visual box size=0.5855378179212705 0.04680711699677431 0.8614572040206672
- link 6: geometry collision box size=0.3420986493715984 0.5411848959174158 0.2452807970919887; visual box size=0.3420986493715984 0.5411848959174158 0.2452807970919887
- link 7: geometry collision box size=0.9624917945093213 0.4331248656192297 1.0666585869148995; visual box size=0.9624917945093213 0.4331248656192297 1.0666585869148995
- link 8: geometry collision box size=0.9243886959557672 0.3021779348427739 0.28806061599311206; visual box size=0.9243886959557672 0.3021779348427739 0.28806061599311206
- link 9: geometry collision box size=0.276563173168608 0.4722051308485823 0.5470121677340033; visual box size=0.276563173168608 0.4722051308485823 0.5470121677340033
Joints:
- removed joint 0_17
- removed joint 0_25
- removed joint 12_13
- removed joint 17_18
- removed joint 18_19
- removed joint 19_20
- removed joint 20_21
- removed joint 21_22
- removed joint 22_23
- removed joint 23_24
- removed joint 25_26
- removed joint 26_27
- removed joint 27_28
- removed joint 28_29
- removed joint 29_30
- removed joint 30_31
- removed joint 31_32
- removed joint 4_5
- added joint 0_13: type revolute, parent 0, child 13, origin xyz=0 0.75 2 rpy=0 0 0, axis 0 1 0, limit lower=-3.14159 upper=3.14159 effort=0.0 velocity=0.0
- added joint 0_5: type revolute, parent 0, child 5, origin xyz=0.75 0 2 rpy=0 0 0, axis 0 1 1, limit lower=-3.14159 upper=3.14159 effort=0.0 velocity=0.0
- joint 0_1: axis 0 1 0 -> 0 0 1; origin xyz=-0.257655522084081 0 4 rpy=0 0 0 -> xyz=-0.75 0 2 rpy=0 0 0
- joint 0_9: origin xyz=0.257655522084081 0 4 rpy=0 0 0 -> xyz=0 -0.75 2 rpy=0 0 0
- joint 10_11: origin xyz=1.1693160965981977 0 0 rpy=0 0 0 -> xyz=0 0 -0.010179508229267498 rpy=0 0 0
- joint 11_12: axis 1 1 0 -> 0 1 0; origin xyz=1.0774838223758034 0 0 rpy=0 0 0 -> xyz=0 0 -1.5168762766021917 rpy=0 0 0
- joint 13_14: origin xyz=0.5662590046145844 0 -0.7164977032493582 rpy=0 0 0 -> xyz=0 0.21808915017884867 -0.16467341093985 rpy=0 0 0
- joint 14_15: axis 1 0 0 -> 0 0 1; origin xyz=0 0 -3.2463879372855704 rpy=0 0 0 -> xyz=0 0 -0.1671641089637273 rpy=0 0 0
- joint 15_16: axis 0 1 0 -> 1 0 0; origin xyz=0 0 -0.037709402398419765 rpy=0 0 0 -> xyz=0 0 -0.7154577019836661 rpy=0 0 0
- joint 1_2: axis 0 0 1 -> 1 0 0; origin xyz=-0.6603054616059846 0 0 rpy=0 0 0 -> xyz=-0.4515381130192819 0 -0.4165403014172513 rpy=0 0 0
- joint 2_3: axis 0 1 0 -> 0 1 1; origin xyz=-0.6999851105289431 0 0 rpy=0 0 0 -> xyz=0 0 -0.9711447529790068 rpy=0 0 0
- joint 3_4: axis 0 0 1 -> 1 0 1; origin xyz=-0.9377078975757741 0 0 rpy=0 0 0 -> xyz=0 0 -0.37664274529537023 rpy=0 0 0
- joint 5_6: axis 0 1 1 -> 0 0 1; origin xyz=-0.7053000467047588 0 -0.5638713473217492 rpy=0 0 0 -> xyz=0.29276890896063523 0 -0.4307286020103336 rpy=0 0 0
- joint 6_7: axis 0 1 1 -> 1 0 0; origin xyz=0 0 -1.3971126926698532 rpy=0 0 0 -> xyz=0 0 -0.2452807970919887 rpy=0 0 0
- joint 7_8: axis 0 0 1 -> 0 1 0; origin xyz=0 0 -1.6587615530986772 rpy=0 0 0 -> xyz=0 0 -1.0666585869148995 rpy=0 0 0
- joint 9_10: axis 1 0 0 -> 0 0 1; origin xyz=0.5847152839516425 0 0 rpy=0 0 0 -> xyz=0 -0.23610256542429114 -0.27350608386700165 rpy=0 0 0
