Commit message: commit

File: body3.urdf (robot description, URDF)
Before this commit: robot robot, 25 links, 24 joints
Links:
- link 0: geometry collision box size=1.5 1.5 0.8; visual box size=1.5 1.5 0.8
- link 1: geometry collision box size=0.26741079010654767 0.8206008305380301 0.8670453899775443; visual box size=0.26741079010654767 0.8206008305380301 0.8670453899775443
- link 10: geometry collision box size=0.11751740684898138 0.5956713199657321 0.028030414618231882; visual box size=0.11751740684898138 0.5956713199657321 0.028030414618231882
- link 11: geometry collision box size=0.4651426715819259 0.5667788991511361 0.7142539744148921; visual box size=0.4651426715819259 0.5667788991511361 0.7142539744148921
- link 12: geometry collision box size=0.39611128755453207 0.5940076640595665 0.857715610966876; visual box size=0.39611128755453207 0.5940076640595665 0.857715610966876
- link 13: geometry collision box size=0.7446692309542443 0.7688106657399588 0.2845108106010642; visual box size=0.7446692309542443 0.7688106657399588 0.2845108106010642
- link 14: geometry collision box size=0.6702263082676297 0.0808644822821214 0.8346317705320287; visual box size=0.6702263082676297 0.0808644822821214 0.8346317705320287
- link 15: geometry collision box size=0.5955574948361461 0.5289719552822103 0.9986973619537185; visual box size=0.5955574948361461 0.5289719552822103 0.9986973619537185
- link 16: geometry collision box size=0.16393401084154624 0.2822737083937703 1.0107176614858975; visual box size=0.16393401084154624 0.2822737083937703 1.0107176614858975
- link 17: geometry collision box size=0.2853816058376212 0.6478553971123123 0.05625971505365884; visual box size=0.2853816058376212 0.6478553971123123 0.05625971505365884
- link 18: geometry collision box size=0.2058608457210177 0.31341824318216027 0.5330226234604438; visual box size=0.2058608457210177 0.31341824318216027 0.5330226234604438
- link 19: geometry collision box size=0.7310935097946356 0.5914392503450112 0.8200504700662964; visual box size=0.7310935097946356 0.5914392503450112 0.8200504700662964
- link 2: geometry collision box size=0.19902107772747135 0.7635661010378931 0.981048924092703; visual box size=0.19902107772747135 0.7635661010378931 0.981048924092703
- link 20: geometry collision box size=0.6517170692689266 0.7250453504166596 0.116985893846272; visual box size=0.6517170692689266 0.7250453504166596 0.116985893846272
- link 21: geometry collision box size=0.6221458537545501 0.41090918685838185 0.18748951797386992; visual box size=0.6221458537545501 0.41090918685838185 0.18748951797386992
- link 22: geometry collision box size=0.378088435621847 0.216446301643463 1.3180428593938645; visual box size=0.378088435621847 0.216446301643463 1.3180428593938645
- link 23: geometry collision box size=0.04081408309452306 0.8754897147885089 0.14483923038293403; visual box size=0.04081408309452306 0.8754897147885089 0.14483923038293403
- link 24: geometry collision box size=0.12829674164779103 0.09724393861204328 0.1371179102232016; visual box size=0.12829674164779103 0.09724393861204328 0.1371179102232016
- link 3: geometry collision box size=0.8662009615841132 0.16306039384530657 0.37614333189742644; visual box size=0.8662009615841132 0.16306039384530657 0.37614333189742644
- link 4: geometry collision box size=0.9197112383757029 0.4755581910656259 0.18256115076063698; visual box size=0.9197112383757029 0.4755581910656259 0.18256115076063698
- link 5: geometry collision box size=0.21920221037288357 0.3190216748621627 0.17630804673113457; visual box size=0.21920221037288357 0.3190216748621627 0.17630804673113457
- link 6: geometry collision box size=0.8807849462756998 0.04204392501459786 1.2411308025082284; visual box size=0.8807849462756998 0.04204392501459786 1.2411308025082284
- link 7: geometry collision box size=0.983390365260045 0.6376835566944214 0.650023833596411; visual box size=0.983390365260045 0.6376835566944214 0.650023833596411
- link 8: geometry collision box size=0.8459216146793201 0.5924621577525853 0.7667479058121991; visual box size=0.8459216146793201 0.5924621577525853 0.7667479058121991
- link 9: geometry collision box size=0.7366575527700363 0.18608595000659556 0.33504283389072376; visual box size=0.7366575527700363 0.18608595000659556 0.33504283389072376
Joints:
- joint 0_1: axis 1 0 0 -> 0 1 0; origin xyz=-0.41732128959284337 0 4 rpy=0 0 0 -> xyz=-0.75 0 2 rpy=0 0 0
- joint 0_13: axis 1 0 0 -> 0 0 1; origin xyz=0 -0.536040548264686 4 rpy=0 0 0 -> xyz=0 -0.75 2 rpy=0 0 0
- joint 0_19: axis 0 1 1 -> 0 1 0; origin xyz=0 0.536040548264686 4 rpy=0 0 0 -> xyz=0 0.75 2 rpy=0 0 0
- joint 0_7: axis 1 1 1 -> 0 1 1; origin xyz=0.41732128959284337 0 4 rpy=0 0 0 -> xyz=0.75 0 2 rpy=0 0 0
- joint 10_11: axis 1 1 0 -> 1 0 0; origin xyz=0 0 -0.825406961644123 rpy=0 0 0 -> xyz=0 0 -0.028030414618231882 rpy=0 0 0
- joint 11_12: axis 0 1 1 -> 1 1 1; origin xyz=0 0 -2.0792359224876744 rpy=0 0 0 -> xyz=0 0 -0.7142539744148921 rpy=0 0 0
- joint 13_14: axis 1 0 0 -> 0 0 1; origin xyz=0 -1.3074235894721675 0 rpy=0 0 0 -> xyz=0 -0.7688106657399588 0 rpy=0 0 0
- joint 14_15: axis 0 0 1 -> 0 1 1; origin xyz=0 -1.1397736412814976 0 rpy=0 0 0 -> xyz=0 -0.0808644822821214 0 rpy=0 0 0
- joint 15_16: axis 1 0 0 -> 1 0 1; origin xyz=0 -0.4924707330019499 -0.5381873407497033 rpy=0 0 0 -> xyz=0 -0.26448597764110515 -0.49934868097685925 rpy=0 0 0
- joint 16_17: axis 1 0 0 -> 1 1 0; origin xyz=0 0 -2.4671305124874983 rpy=0 0 0 -> xyz=0 0 -1.0107176614858975 rpy=0 0 0
- joint 17_18: axis 1 0 1 -> 1 1 0; origin xyz=0 0 -0.6108691675613723 rpy=0 0 0 -> xyz=0 0 -0.05625971505365884 rpy=0 0 0
- joint 19_20: axis 0 1 1 -> 1 0 1; origin xyz=0 0.9462224997414614 0 rpy=0 0 0 -> xyz=0 0.5914392503450112 0 rpy=0 0 0
- joint 1_2: axis 1 0 0 -> 0 0 1; origin xyz=-0.6617411390171486 0 0 rpy=0 0 0 -> xyz=-0.26741079010654767 0 0 rpy=0 0 0
- joint 20_21: axis 1 0 1 -> 1 1 0; origin xyz=0 0.6306923729711901 0 rpy=0 0 0 -> xyz=0 0.7250453504166596 0 rpy=0 0 0
- joint 21_22: axis 0 1 0 -> 0 0 1; origin xyz=0 0.4386944886265243 -0.633378475068946 rpy=0 0 0 -> xyz=0 0.20545459342919092 -0.09374475898693496 rpy=0 0 0
- joint 22_23: axis 0 0 1 -> 1 0 1; origin xyz=0 0 -1.8001394957937404 rpy=0 0 0 -> xyz=0 0 -1.3180428593938645 rpy=0 0 0
- joint 23_24: axis 0 1 1 -> 1 0 1; origin xyz=0 0 -1.1571813749006679 rpy=0 0 0 -> xyz=0 0 -0.14483923038293403 rpy=0 0 0
- joint 2_3: axis 0 0 1 -> 1 1 0; origin xyz=-1.304849723800142 0 0 rpy=0 0 0 -> xyz=-0.19902107772747135 0 0 rpy=0 0 0
- joint 3_4: axis 0 0 1 -> 1 1 0; origin xyz=-0.4398961302284592 0 -0.6537219833356382 rpy=0 0 0 -> xyz=-0.4331004807920566 0 -0.18807166594871322 rpy=0 0 0
- joint 4_5: axis 1 1 1 -> 0 0 1; origin xyz=0 0 -1.6713885383255251 rpy=0 0 0 -> xyz=0 0 -0.18256115076063698 rpy=0 0 0
- joint 5_6: axis 1 1 1 -> 1 0 0; origin xyz=0 0 -1.7423500241124537 rpy=0 0 0 -> xyz=0 0 -0.17630804673113457 rpy=0 0 0
- joint 7_8: origin xyz=0.8481363291261281 0 0 rpy=0 0 0 -> xyz=0.983390365260045 0 0 rpy=0 0 0
- joint 8_9: axis 1 0 1 -> 0 1 1; origin xyz=0.5774559351995073 0 0 rpy=0 0 0 -> xyz=0.8459216146793201 0 0 rpy=0 0 0
- joint 9_10: axis 1 1 1 -> 1 1 0; origin xyz=0.6676939117807226 0 -0.2929920868406845 rpy=0 0 0 -> xyz=0.36832877638501815 0 -0.16752141694536188 rpy=0 0 0

File: body4.urdf (robot description, URDF)
Before this commit: robot robot, 33 links, 32 joints
Links:
- removed link 25
- removed link 26
- removed link 27
- removed link 28
- removed link 29
- removed link 30
- removed link 31
- removed link 32
- link 0: geometry collision box size=1.5 1.5 0.8; visual box size=1.5 1.5 0.8
- link 1: geometry collision box size=0.9720763299549751 0.11040559321661736 0.6687306195444088; visual box size=0.9720763299549751 0.11040559321661736 0.6687306195444088
- link 10: geometry collision box size=0.13274681762234486 0.9384991710254861 1.3378142982014645; visual box size=0.13274681762234486 0.9384991710254861 1.3378142982014645
- link 11: geometry collision box size=0.241104884843249 0.040380177882467505 0.016450655652969527; visual box size=0.241104884843249 0.040380177882467505 0.016450655652969527
- link 12: geometry collision box size=0.07223108974470926 0.6931934937639516 0.2457350461455661; visual box size=0.07223108974470926 0.6931934937639516 0.2457350461455661
- link 13: geometry collision box size=0.5949419364960706 0.6851617326083693 0.9359034215559933; visual box size=0.5949419364960706 0.6851617326083693 0.9359034215559933
- link 14: geometry collision box size=0.9131780695297272 0.9692162725667856 0.48396563489725586; visual box size=0.9131780695297272 0.9692162725667856 0.48396563489725586
- link 15: geometry collision box size=0.6812176981381437 0.2801164038216749 0.36729679548272165; visual box size=0.6812176981381437 0.2801164038216749 0.36729679548272165
- link 16: geometry collision box size=0.7996187941094406 0.7634340945955963 0.4864528572818852; visual box size=0.7996187941094406 0.7634340945955963 0.4864528572818852
- link 17: geometry collision box size=0.6401974268624878 0.29768791035194286 0.9114316681759929; visual box size=0.6401974268624878 0.29768791035194286 0.9114316681759929
- link 18: geometry collision box size=0.8391686323600244 0.9877827350359227 0.2021154745421221; visual box size=0.8391686323600244 0.9877827350359227 0.2021154745421221
- link 19: geometry collision box size=0.8563893140030474 0.7079633725694321 0.5928403652585207; visual box size=0.8563893140030474 0.7079633725694321 0.5928403652585207
- link 2: geometry collision box size=0.406383101268305 0.28726957841915834 0.9366922259663688; visual box size=0.406383101268305 0.28726957841915834 0.9366922259663688
- link 20: geometry collision box size=0.12350465788776932 0.45831447788274715 0.743545519582784; visual box size=0.12350465788776932 0.45831447788274715 0.743545519582784
- link 21: geometry collision box size=0.6974063129809458 0.20569975403430285 0.19876616932883606; visual box size=0.6974063129809458 0.20569975403430285 0.19876616932883606
- link 22: geometry collision box size=0.6593784037383477 0.43618024958478485 1.2388970063027056; visual box size=0.6593784037383477 0.43618024958478485 1.2388970063027056
- link 23: geometry collision box size=0.022491461719508776 0.6519060138415289 0.1721453274536514; visual box size=0.022491461719508776 0.6519060138415289 0.1721453274536514
- link 24: geometry collision box size=0.07981988094529069 0.5160955479790921 0.18895766624364307; visual box size=0.07981988094529069 0.5160955479790921 0.18895766624364307
- link 3: geometry collision box size=0.25663213408012886 0.277361182579307 0.9959797490847617; visual box size=0.25663213408012886 0.277361182579307 0.9959797490847617
- link 4: geometry collision box size=0.05301561389335463 0.8895925698705222 0.19969769156936634; visual box size=0.05301561389335463 0.8895925698705222 0.19969769156936634
- link 5: geometry collision box size=0.4624652605511401 0.8959652937766708 0.9675968139648221; visual box size=0.4624652605511401 0.8959652937766708 0.9675968139648221
- link 6: geometry collision box size=0.9830008319627818 0.6555455177144505 0.43270549446581175; visual box size=0.9830008319627818 0.6555455177144505 0.43270549446581175
- link 7: geometry collision box size=0.35251339633327106 0.940194273944308 0.40735267951897247; visual box size=0.35251339633327106 0.940194273944308 0.40735267951897247
- link 8: geometry collision box size=0.436113944360193 0.8467646078739507 0.8532866682713874; visual box size=0.436113944360193 0.8467646078739507 0.8532866682713874
- link 9: geometry collision box size=0.5721808031066536 0.9607620739150868 0.42296887162275676; visual box size=0.5721808031066536 0.9607620739150868 0.42296887162275676
Joints:
- removed joint 0_17
- removed joint 0_25
- removed joint 0_9
- removed joint 12_13
- removed joint 18_19
- removed joint 25_26
- removed joint 26_27
- removed joint 27_28
- removed joint 28_29
- removed joint 29_30
- removed joint 30_31
- removed joint 31_32
- removed joint 6_7
- added joint 0_13: type revolute, parent 0, child 13, origin xyz=0 -0.75 2 rpy=0 0 0, axis 0 0 1, limit lower=-3.14159 upper=3.14159 effort=0.0 velocity=0.0
- added joint 0_19: type revolute, parent 0, child 19, origin xyz=0 0.75 2 rpy=0 0 0, axis 0 1 1, limit lower=-3.14159 upper=3.14159 effort=0.0 velocity=0.0
- added joint 0_7: type revolute, parent 0, child 7, origin xyz=0.75 0 2 rpy=0 0 0, axis 0 1 1, limit lower=-3.14159 upper=3.14159 effort=0.0 velocity=0.0
- added joint 16_17: type revolute, parent 16, child 17, origin xyz=0 0 -0.4864528572818852 rpy=0 0 0, axis 1 1 0, limit lower=-3.14159 upper=3.14159 effort=0.0 velocity=0.0
- added joint 8_9: type revolute, parent 8, child 9, origin xyz=0.436113944360193 0 0 rpy=0 0 0, axis 0 1 1, limit lower=-3.14159 upper=3.14159 effort=0.0 velocity=0.0
- joint 0_1: axis 0 0 1 -> 0 1 0; origin xyz=-0.28529223645414287 0 4 rpy=0 0 0 -> xyz=-0.75 0 2 rpy=0 0 0
- joint 10_11: axis 1 0 1 -> 0 0 1; origin xyz=1.1049784049567508 0 0 rpy=0 0 0 -> xyz=0 0 -1.3378142982014645 rpy=0 0 0
- joint 11_12: axis 1 1 1 -> 1 0 0; origin xyz=0.6979812153957877 0 0 rpy=0 0 0 -> xyz=0 0 -0.016450655652969527 rpy=0 0 0
- joint 13_14: origin xyz=0.6474187507606182 0 -0.6072602560829968 rpy=0 0 0 -> xyz=0 -0.6851617326083693 0 rpy=0 0 0
- joint 14_15: axis 1 1 0 -> 0 0 1; origin xyz=0 0 -0.7204452435340766 rpy=0 0 0 -> xyz=0 -0.9692162725667856 0 rpy=0 0 0
- joint 15_16: axis 0 1 0 -> 0 0 1; origin xyz=0 0 -2.4845204448791467 rpy=0 0 0 -> xyz=0 -0.14005820191083745 -0.18364839774136082 rpy=0 0 0
- joint 17_18: axis 0 0 1 -> 1 1 1; origin xyz=0 -0.9725364231606399 0 rpy=0 0 0 -> xyz=0 0 -0.9114316681759929 rpy=0 0 0
- joint 19_20: axis 0 1 0 -> 1 0 1; origin xyz=0 -1.0189474208408602 0 rpy=0 0 0 -> xyz=0 0.7079633725694321 0 rpy=0 0 0
- joint 1_2: origin xyz=-1.2031628656149567 0 0 rpy=0 0 0 -> xyz=-0.9720763299549751 0 0 rpy=0 0 0
- joint 20_21: axis 1 0 1 -> 0 1 0; origin xyz=0 -0.9456158536699295 0 rpy=0 0 0 -> xyz=0 0.45831447788274715 0 rpy=0 0 0
- joint 21_22: axis 0 1 0 -> 1 0 1; origin xyz=0 -0.5780249142719927 -0.7326490974280584 rpy=0 0 0 -> xyz=0 0.10284987701715143 -0.09938308466441803 rpy=0 0 0
- joint 22_23: axis 0 0 1 -> 1 1 1; origin xyz=0 0 -2.7422984322156516 rpy=0 0 0 -> xyz=0 0 -1.2388970063027056 rpy=0 0 0
- joint 23_24: axis 0 1 1 -> 1 1 0; origin xyz=0 0 -0.1313463735690704 rpy=0 0 0 -> xyz=0 0 -0.1721453274536514 rpy=0 0 0
- joint 2_3: axis 1 1 1 -> 1 0 0; origin xyz=-1.0045551118378742 0 0 rpy=0 0 0 -> xyz=-0.406383101268305 0 0 rpy=0 0 0
- joint 3_4: axis 0 1 1 -> 1 0 0; origin xyz=-0.8347693461917494 0 0 rpy=0 0 0 -> xyz=-0.12831606704006443 0 -0.49798987454238086 rpy=0 0 0
- joint 4_5: origin xyz=-1.0997988688401446 0 0 rpy=0 0 0 -> xyz=0 0 -0.19969769156936634 rpy=0 0 0
- joint 5_6: axis 0 1 1 -> 1 1 1; origin xyz=-0.3929494252436307 0 -0.4525474327056057 rpy=0 0 0 -> xyz=0 0 -0.9675968139648221 rpy=0 0 0
- joint 7_8: origin xyz=0 0 -1.0897003465424706 rpy=0 0 0 -> xyz=0.35251339633327106 0 0 rpy=0 0 0
- joint 9_10: axis 1 0 1 -> 0 1 1; origin xyz=1.0523087542503684 0 0 rpy=0 0 0 -> xyz=0.2860904015533268 0 -0.21148443581137838 rpy=0 0 0
