Commit message: commit

File: body0.urdf (robot description, URDF)
Before this commit: robot robot, 17 links, 16 joints
Links:
- link 1: geometry collision box size=0.12228108172753238 0.041800665360371525 0.3874190520893195; visual box size=0.12228108172753238 0.041800665360371525 0.3874190520893195
- link 10: geometry collision box size=0.8024296887660426 0.008105270089565075 1.5442231085690195; visual box size=0.8024296887660426 0.008105270089565075 1.5442231085690195
- link 11: geometry collision box size=0.6044945308963908 0.9586506383984 0.04402900591548745; visual box size=0.6044945308963908 0.9586506383984 0.04402900591548745
- link 12: geometry collision box size=0.7223276299825092 0.4990047893874521 0.011747885515493182; visual box size=0.7223276299825092 0.4990047893874521 0.011747885515493182
- link 13: geometry collision box size=0.9657294381556446 0.32687104635894204 0.4668752115391125; visual box size=0.9657294381556446 0.32687104635894204 0.4668752115391125
- link 14: geometry collision box size=0.6443699878253394 0.5555689835601656 1.0770015167621245; visual box size=0.6443699878253394 0.5555689835601656 1.0770015167621245
- link 15: geometry collision box size=0.6510669886455813 0.8646874634426204 0.07236522730101946; visual box size=0.6510669886455813 0.8646874634426204 0.07236522730101946
- link 16: geometry collision box size=0.46899307178116956 0.6373400506712246 0.4506332559368561; visual box size=0.46899307178116956 0.6373400506712246 0.4506332559368561
- link 2: geometry collision box size=0.435242051426488 0.8328385130387006 1.5384063081681632; visual box size=0.435242051426488 0.8328385130387006 1.5384063081681632
- link 3: geometry collision box size=0.9883294007549555 0.19974990162523387 0.05728296444989989; visual box size=0.9883294007549555 0.19974990162523387 0.05728296444989989
- link 4: geometry collision box size=0.914744271543993 0.44264659156473185 0.004310727381937052; visual box size=0.914744271543993 0.44264659156473185 0.004310727381937052
- link 5: geometry collision box size=0.6594329857683123 0.20207089708287562 0.554250443334625; visual box size=0.6594329857683123 0.20207089708287562 0.554250443334625
- link 6: geometry collision box size=0.844728364302637 0.38095673087041315 1.28600988362806; visual box size=0.844728364302637 0.38095673087041315 1.28600988362806
- link 7: geometry collision box size=0.8279730763887236 0.23594867343843984 0.18441707251839215; visual box size=0.8279730763887236 0.23594867343843984 0.18441707251839215
- link 8: geometry collision box size=0.5086017586289632 0.23426518568512766 0.12957304385354793; visual box size=0.5086017586289632 0.23426518568512766 0.12957304385354793
- link 9: geometry collision box size=0.761873290830006 0.8173037736470997 0.34889822402585857; visual box size=0.761873290830006 0.8173037736470997 0.34889822402585857
Joints:
- joint 0_1: axis 1 1 0 -> 1 0 1
- joint 0_13: axis 0 1 0 -> 1 1 0
- joint 0_5: axis 0 1 1 -> 0 0 1
- joint 0_9: axis 0 1 0 -> 0 0 1
- joint 10_11: origin xyz=0 0 -1.197705955447554 rpy=0 0 0 -> xyz=0 0 -1.5442231085690195 rpy=0 0 0
- joint 11_12: axis 0 0 1 -> 1 0 0; origin xyz=0 0 -0.2710188445761256 rpy=0 0 0 -> xyz=0 0 -0.04402900591548745 rpy=0 0 0
- joint 13_14: axis 0 1 0 -> 1 0 0; origin xyz=0 0.1890271644141791 -0.33640309546636804 rpy=0 0 0 -> xyz=0 0.16343552317947102 -0.23343760576955624 rpy=0 0 0
- joint 14_15: axis 1 1 0 -> 0 1 1; origin xyz=0 0 -1.275105207340246 rpy=0 0 0 -> xyz=0 0 -1.0770015167621245 rpy=0 0 0
- joint 15_16: axis 1 1 0 -> 0 0 1; origin xyz=0 0 -0.2493924332519192 rpy=0 0 0 -> xyz=0 0 -0.07236522730101946 rpy=0 0 0
- joint 1_2: axis 0 1 0 -> 0 0 1; origin xyz=-0.33511727134948166 0 -0.18579788091235688 rpy=0 0 0 -> xyz=-0.06114054086376619 0 -0.19370952604465974 rpy=0 0 0
- joint 2_3: axis 0 1 0 -> 1 0 0; origin xyz=0 0 -0.6845951070633703 rpy=0 0 0 -> xyz=0 0 -1.5384063081681632 rpy=0 0 0
- joint 3_4: axis 0 1 0 -> 1 0 1; origin xyz=0 0 -0.05157313386257725 rpy=0 0 0 -> xyz=0 0 -0.05728296444989989 rpy=0 0 0
- joint 5_6: axis 1 1 0 -> 1 0 1; origin xyz=0.0059797550700806945 0 -0.4126410579759959 rpy=0 0 0 -> xyz=0.32971649288415616 0 -0.2771252216673125 rpy=0 0 0
- joint 6_7: origin xyz=0 0 -0.4674553661300461 rpy=0 0 0 -> xyz=0 0 -1.28600988362806 rpy=0 0 0
- joint 7_8: origin xyz=0 0 -0.21551419053083565 rpy=0 0 0 -> xyz=0 0 -0.18441707251839215 rpy=0 0 0
- joint 9_10: axis 0 0 1 -> 1 1 1; origin xyz=0 -0.35097200481440755 -0.15411266541985413 rpy=0 0 0 -> xyz=0 -0.40865188682354986 -0.17444911201292929 rpy=0 0 0

File: body1.urdf (robot description, URDF)
Before this commit: robot robot, 29 links, 28 joints
Links:
- removed link 25
- removed link 26
- removed link 27
- removed link 28
- link 1: geometry collision box size=0.22243847580136233 0.022239180690408977 0.8098769320848941; visual box size=0.22243847580136233 0.022239180690408977 0.8098769320848941
- link 10: geometry collision box size=0.6963361330825207 0.4162101707016993 0.8994650855511491; visual box size=0.6963361330825207 0.4162101707016993 0.8994650855511491
- link 11: geometry collision box size=0.11231357673847353 0.8144387037138998 0.06341867416114418; visual box size=0.11231357673847353 0.8144387037138998 0.06341867416114418
- link 12: geometry collision box size=0.4279249546950502 0.6300197085866626 0.6371162402877067; visual box size=0.4279249546950502 0.6300197085866626 0.6371162402877067
- link 13: geometry collision box size=0.5943447133777444 0.5854355155747518 0.39243958262996637; visual box size=0.5943447133777444 0.5854355155747518 0.39243958262996637
- link 14: geometry collision box size=0.1918204281740976 0.6676520903067827 0.7670103740741117; visual box size=0.1918204281740976 0.6676520903067827 0.7670103740741117
- link 15: geometry collision box size=0.20390074724112417 0.8141301513034164 0.5745814554366973; visual box size=0.20390074724112417 0.8141301513034164 0.5745814554366973
- link 16: geometry collision box size=0.19673733904106427 0.33179477167443794 0.12770691126430675; visual box size=0.19673733904106427 0.33179477167443794 0.12770691126430675
- link 17: geometry collision box size=0.03219850502202071 0.4867205372360074 0.8951022032835811; visual box size=0.03219850502202071 0.4867205372360074 0.8951022032835811
- link 18: geometry collision box size=0.30710010905090845 0.4682990429623909 0.5771908854521122; visual box size=0.30710010905090845 0.4682990429623909 0.5771908854521122
- link 19: geometry collision box size=0.11851187820496989 0.9098311813750964 0.869776992282439; visual box size=0.11851187820496989 0.9098311813750964 0.869776992282439
- link 2: geometry collision box size=0.6812459111015068 0.6236227577340923 0.85313360420814; visual box size=0.6812459111015068 0.6236227577340923 0.85313360420814
- link 20: geometry collision box size=0.9376417281415393 0.4411084858537956 0.21718802634040468; visual box size=0.9376417281415393 0.4411084858537956 0.21718802634040468
- link 21: geometry collision box size=0.18337267390319612 0.4646275049660935 0.9549006283567263; visual box size=0.18337267390319612 0.4646275049660935 0.9549006283567263
- link 22: geometry collision box size=0.8014611481517963 0.12800056070679755 0.864803928530621; visual box size=0.8014611481517963 0.12800056070679755 0.864803928530621
- link 23: geometry collision box size=0.5617079006631379 0.45022388109245604 0.12472084942394943; visual box size=0.5617079006631379 0.45022388109245604 0.12472084942394943
- link 24: geometry collision box size=0.5883184655090766 0.15372339479783015 0.6104752220454296; visual box size=0.5883184655090766 0.15372339479783015 0.6104752220454296
- link 3: geometry collision box size=0.331188984422373 0.3884779017718133 0.3701753714904952; visual box size=0.331188984422373 0.3884779017718133 0.3701753714904952
- link 4: geometry collision box size=0.8228538393333187 0.8379491203793291 0.25754028051038275; visual box size=0.8228538393333187 0.8379491203793291 0.25754028051038275
- link 5: geometry collision box size=0.76526877786306 0.10751904203894036 0.8549978113347292; visual box size=0.76526877786306 0.10751904203894036 0.8549978113347292
- link 6: geometry collision box size=0.9087669382336655 0.8696182372547238 0.4874619081548881; visual box size=0.9087669382336655 0.8696182372547238 0.4874619081548881
- link 7: geometry collision box size=0.8624294409008315 0.5221821548552875 0.25627927727607036; visual box size=0.8624294409008315 0.5221821548552875 0.25627927727607036
- link 8: geometry collision box size=0.47317809099617225 0.8982205679391114 0.7167356819922938; visual box size=0.47317809099617225 0.8982205679391114 0.7167356819922938
- link 9: geometry collision box size=0.7561531226735622 0.5302854559086662 0.27915920631667923; visual box size=0.7561531226735622 0.5302854559086662 0.27915920631667923
Joints:
- removed joint 0_15
- removed joint 0_22
- removed joint 0_8
- removed joint 12_13
- removed joint 18_19
- removed joint 24_25
- removed joint 25_26
- removed joint 26_27
- removed joint 27_28
- removed joint 6_7
- added joint 0_13: type revolute, parent 0, child 13, origin xyz=0 -0.75 2 rpy=0 0 0, axis 1 1 1, limit lower=-3.14159 upper=3.14159 effort=0.0 velocity=0.0
- added joint 0_19: type revolute, parent 0, child 19, origin xyz=0 0.75 2 rpy=0 0 0, axis 1 0 0, limit lower=-3.14159 upper=3.14159 effort=0.0 velocity=0.0
- added joint 0_7: type revolute, parent 0, child 7, origin xyz=0.75 0 2 rpy=0 0 0, axis 0 0 1, limit lower=-3.14159 upper=3.14159 effort=0.0 velocity=0.0
- added joint 14_15: type revolute, parent 14, child 15, origin xyz=0 -0.6676520903067827 0 rpy=0 0 0, axis 1 0 0, limit lower=-3.14159 upper=3.14159 effort=0.0 velocity=0.0
- added joint 21_22: type revolute, parent 21, child 22, origin xyz=0 0.23231375248304675 -0.47745031417836314 rpy=0 0 0, axis 0 1 0, limit lower=-3.14159 upper=3.14159 effort=0.0 velocity=0.0
- added joint 7_8: type revolute, parent 7, child 8, origin xyz=0.8624294409008315 0 0 rpy=0 0 0, axis 1 0 1, limit lower=-3.14159 upper=3.14159 effort=0.0 velocity=0.0
- joint 10_11: axis 1 0 0 -> 0 0 1; origin xyz=0.5676691240743692 0 0 rpy=0 0 0 -> xyz=0 0 -0.8994650855511491 rpy=0 0 0
- joint 11_12: axis 1 0 0 -> 1 0 1; origin xyz=0.15056764361987074 0 -0.08602107246784435 rpy=0 0 0 -> xyz=0 0 -0.06341867416114418 rpy=0 0 0
- joint 13_14: origin xyz=0 0 -1.159030535521866 rpy=0 0 0 -> xyz=0 -0.5854355155747518 0 rpy=0 0 0
- joint 15_16: axis 1 0 1 -> 1 1 1; origin xyz=0 -0.6772169183529062 0 rpy=0 0 0 -> xyz=0 -0.4070650756517082 -0.2872907277183486 rpy=0 0 0
- joint 16_17: axis 1 0 0 -> 1 1 0; origin xyz=0 -0.4269871454216021 0 rpy=0 0 0 -> xyz=0 0 -0.12770691126430675 rpy=0 0 0
- joint 17_18: axis 1 0 0 -> 1 0 1; origin xyz=0 -0.8305211523512608 0 rpy=0 0 0 -> xyz=0 0 -0.8951022032835811 rpy=0 0 0
- joint 19_20: axis 1 1 0 -> 0 0 1; origin xyz=0 0 -1.4277303665203707 rpy=0 0 0 -> xyz=0 0.9098311813750964 0 rpy=0 0 0
- joint 1_2: axis 1 1 1 -> 0 0 1; origin xyz=-0.5126919324777913 0 0 rpy=0 0 0 -> xyz=-0.22243847580136233 0 0 rpy=0 0 0
- joint 20_21: axis 1 0 0 -> 0 1 0; origin xyz=0 0 -0.08703985776590724 rpy=0 0 0 -> xyz=0 0.4411084858537956 0 rpy=0 0 0
- joint 22_23: axis 1 0 1 -> 0 1 0; origin xyz=0 0.6359521381373019 0 rpy=0 0 0 -> xyz=0 0 -0.864803928530621 rpy=0 0 0
- joint 23_24: axis 1 0 1 -> 0 1 0; origin xyz=0 0.6084636674703443 0 rpy=0 0 0 -> xyz=0 0 -0.12472084942394943 rpy=0 0 0
- joint 2_3: origin xyz=-0.26643980550734525 0 0 rpy=0 0 0 -> xyz=-0.6812459111015068 0 0 rpy=0 0 0
- joint 3_4: axis 1 1 1 -> 1 0 0; origin xyz=-0.7385440566924593 0 0 rpy=0 0 0 -> xyz=-0.1655944922111865 0 -0.1850876857452476 rpy=0 0 0
- joint 4_5: axis 0 1 0 -> 1 0 1; origin xyz=-0.492676788758288 0 -0.2512033654649823 rpy=0 0 0 -> xyz=0 0 -0.25754028051038275 rpy=0 0 0
- joint 5_6: axis 0 1 1 -> 0 0 1; origin xyz=0 0 -0.33122092922989044 rpy=0 0 0 -> xyz=0 0 -0.8549978113347292 rpy=0 0 0
- joint 8_9: axis 0 1 0 -> 0 1 1; origin xyz=0.9049937149172881 0 0 rpy=0 0 0 -> xyz=0.47317809099617225 0 0 rpy=0 0 0
- joint 9_10: axis 1 0 1 -> 1 1 0; origin xyz=0.751879339325681 0 0 rpy=0 0 0 -> xyz=0.3780765613367811 0 -0.13957960315833962 rpy=0 0 0

File: body2.urdf (robot description, URDF)
Before this commit: robot robot, 17 links, 16 joints
Links:
- added link 17, mass 1; collision box size=0.27470009213790814 0.9628519245725478 0.3765745830860897; visual box size=0.27470009213790814 0.9628519245725478 0.3765745830860897
- added link 18, mass 1; collision box size=0.9937376957799928 0.7022149175388596 0.49030984421606405; visual box size=0.9937376957799928 0.7022149175388596 0.49030984421606405
- added link 19, mass 1; collision box size=0.5105323818603812 0.24548830779132713 1.1030668139404407; visual box size=0.5105323818603812 0.24548830779132713 1.1030668139404407
- added link 20, mass 1; collision box size=0.10688307751254666 0.007567453176151817 0.0066233418434953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; visual box size=0.10688307751254666 0.007567453176151817 0.0066233418434953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
- link 1: geometry collision box size=0.07311924047980078 0.5987383266085363 0.06890018212021631; visual box size=0.07311924047980078 0.5987383266085363 0.06890018212021631
- link 10: geometry collision box size=0.8876044542431063 0.666453857199856 0.5641660960245947; visual box size=0.8876044542431063 0.666453857199856 0.5641660960245947
- link 11: geometry collision box size=0.18885980712630535 0.9760799886071233 0.35295576949852503; visual box size=0.18885980712630535 0.9760799886071233 0.35295576949852503
- link 12: geometry collision box size=0.2901820763994408 0.6383647390170017 0.42874990443387595; visual box size=0.2901820763994408 0.6383647390170017 0.42874990443387595
- link 13: geometry collision box size=0.8990990632903286 0.9855636877416878 0.06923418282965539; visual box size=0.8990990632903286 0.9855636877416878 0.06923418282965539
- link 14: geometry collision box size=0.41734836975280865 0.9014597022074874 0.2124157717788742; visual box size=0.41734836975280865 0.9014597022074874 0.2124157717788742
- link 15: geometry collision box size=0.2577347177756869 0.20654336177930122 1.3183500453914705; visual box size=0.2577347177756869 0.20654336177930122 1.3183500453914705
- link 16: geometry collision box size=0.07611471382061408 0.9733205739597137 0.9354911885611596; visual box size=0.07611471382061408 0.9733205739597137 0.9354911885611596
- link 2: geometry collision box size=0.09579072439431802 0.276587240207695 0.9786248692705803; visual box size=0.09579072439431802 0.276587240207695 0.9786248692705803
- link 3: geometry collision box size=0.277426108925407 0.06451724446808937 0.5056766150816641; visual box size=0.277426108925407 0.06451724446808937 0.5056766150816641
- link 4: geometry collision box size=0.24728994586846864 0.007243027975162852 0.4366373430401463; visual box size=0.24728994586846864 0.007243027975162852 0.4366373430401463
- link 5: geometry collision box size=0.1149224707445421 0.7574821510333509 0.6576860418781898; visual box size=0.1149224707445421 0.7574821510333509 0.6576860418781898
- link 6: geometry collision box size=0.20944780190558643 0.8368715216775164 0.5956125318451297; visual box size=0.20944780190558643 0.8368715216775164 0.5956125318451297
- link 7: geometry collision box size=0.6513562237423492 0.8181825963568818 0.19557728932550766; visual box size=0.6513562237423492 0.8181825963568818 0.19557728932550766
- link 8: geometry collision box size=0.29167854049253017 0.23914105085462822 0.00920269812434711; visual box size=0.29167854049253017 0.23914105085462822 0.00920269812434711
- link 9: geometry collision box size=0.3364684385236748 0.9192398065909937 1.0266312058510583; visual box size=0.3364684385236748 0.9192398065909937 1.0266312058510583
Joints:
- removed joint 0_13
- removed joint 0_5
- removed joint 0_9
- removed joint 10_11
- removed joint 15_16
- removed joint 5_6
- added joint 0_11: type revolute, parent 0, child 11, origin xyz=0 -0.75 2 rpy=0 0 0, axis 1 1 1, limit lower=-3.14159 upper=3.14159 effort=0.0 velocity=0.0
- added joint 0_16: type revolute, parent 0, child 16, origin xyz=0 0.75 2 rpy=0 0 0, axis 1 0 1, limit lower=-3.14159 upper=3.14159 effort=0.0 velocity=0.0
- added joint 0_6: type revolute, parent 0, child 6, origin xyz=0.75 0 2 rpy=0 0 0, axis 0 1 1, limit lower=-3.14159 upper=3.14159 effort=0.0 velocity=0.0
- added joint 12_13: type revolute, parent 12, child 13, origin xyz=0 -0.3191823695085009 -0.21437495221693798 rpy=0 0 0, axis 1 1 0, limit lower=-3.14159 upper=3.14159 effort=0.0 velocity=0.0
- added joint 16_17: type revolute, parent 16, child 17, origin xyz=0 0.9733205739597137 0 rpy=0 0 0, axis 1 0 0, limit lower=-3.14159 upper=3.14159 effort=0.0 velocity=0.0
- added joint 17_18: type revolute, parent 17, child 18, origin xyz=0 0.4814259622862739 -0.18828729154304485 rpy=0 0 0, axis 1 1 0, limit lower=-3.14159 upper=3.14159 effort=0.0 velocity=0.0
- added joint 18_19: type revolute, parent 18, child 19, origin xyz=0 0 -0.49030984421606405 rpy=0 0 0, axis 1 1 1, limit lower=-3.14159 upper=3.14159 effort=0.0 velocity=0.0
- added joint 19_20: type revolute, parent 19, child 20, origin xyz=0 0 -1.1030668139404407 rpy=0 0 0, axis 1 0 1, limit lower=-3.14159 upper=3.14159 effort=0.0 velocity=0.0
- added joint 4_5: type revolute, parent 4, child 5, origin xyz=0 0 -0.4366373430401463 rpy=0 0 0, axis 1 1 0, limit lower=-3.14159 upper=3.14159 effort=0.0 velocity=0.0
- added joint 8_9: type revolute, parent 8, child 9, origin xyz=0 0 -0.00920269812434711 rpy=0 0 0, axis 0 1 1, limit lower=-3.14159 upper=3.14159 effort=0.0 velocity=0.0
- joint 0_1: axis 0 0 1 -> 1 1 1
- joint 11_12: origin xyz=0 0 -1.5168762766021917 rpy=0 0 0 -> xyz=0 -0.9760799886071233 0 rpy=0 0 0
- joint 13_14: origin xyz=0 0.21808915017884867 -0.16467341093985 rpy=0 0 0 -> xyz=0 0 -0.06923418282965539 rpy=0 0 0
- joint 14_15: axis 0 0 1 -> 1 0 0; origin xyz=0 0 -0.1671641089637273 rpy=0 0 0 -> xyz=0 0 -0.2124157717788742 rpy=0 0 0
- joint 1_2: axis 1 0 0 -> 0 0 1; origin xyz=-0.4515381130192819 0 -0.4165403014172513 rpy=0 0 0 -> xyz=-0.07311924047980078 0 0 rpy=0 0 0
- joint 2_3: axis 0 1 1 -> 1 0 0; origin xyz=0 0 -0.9711447529790068 rpy=0 0 0 -> xyz=-0.04789536219715901 0 -0.48931243463529017 rpy=0 0 0
- joint 3_4: origin xyz=0 0 -0.37664274529537023 rpy=0 0 0 -> xyz=0 0 -0.5056766150816641 rpy=0 0 0
- joint 6_7: axis 1 0 0 -> 0 1 0; origin xyz=0 0 -0.2452807970919887 rpy=0 0 0 -> xyz=0.20944780190558643 0 0 rpy=0 0 0
- joint 7_8: axis 0 1 0 -> 0 0 1; origin xyz=0 0 -1.0666585869148995 rpy=0 0 0 -> xyz=0.3256781118711746 0 -0.09778864466275383 rpy=0 0 0
- joint 9_10: axis 0 0 1 -> 0 1 0; origin xyz=0 -0.23610256542429114 -0.27350608386700165 rpy=0 0 0 -> xyz=0 0 -1.0266312058510583 rpy=0 0 0
