Commit message: commit

File: body3.urdf (robot description, URDF)
Before this commit: robot robot, 25 links, 24 joints
Links:
- link 1: geometry collision box size=0.05738224560673355 0.23741784274289757 0.6045315257688684; visual box size=0.05738224560673355 0.23741784274289757 0.6045315257688684
- link 10: geometry collision box size=0.9893442582012629 0.008034417759784862 1.4554611236959727; visual box size=0.9893442582012629 0.008034417759784862 1.4554611236959727
- link 11: geometry collision box size=0.39574213753496634 0.08671109591349924 0.060794889373184655; visual box size=0.39574213753496634 0.08671109591349924 0.060794889373184655
- link 12: geometry collision box size=0.03919724314277029 0.0714839412256616 0.08374398693084274; visual box size=0.03919724314277029 0.0714839412256616 0.08374398693084274
- link 13: geometry collision box size=0.9393028836452529 0.25412788202751113 0.8842026076095828; visual box size=0.9393028836452529 0.25412788202751113 0.8842026076095828
- link 14: geometry collision box size=0.07394302579081058 0.3751101172440727 0.009650082758268286; visual box size=0.07394302579081058 0.3751101172440727 0.009650082758268286
- link 15: geometry collision box size=0.03839110914007826 0.45534728657416657 0.5930203121810415; visual box size=0.03839110914007826 0.45534728657416657 0.5930203121810415
- link 16: geometry collision box size=0.34612627833555487 0.058285194774905125 0.9632596283696517; visual box size=0.34612627833555487 0.058285194774905125 0.9632596283696517
- link 17: geometry collision box size=0.1620655951394402 0.3380884597144832 0.3385209032505026; visual box size=0.1620655951394402 0.3380884597144832 0.3385209032505026
- link 18: geometry collision box size=0.47264029967844845 0.5652870923756975 0.29821946837984575; visual box size=0.47264029967844845 0.5652870923756975 0.29821946837984575
- link 19: geometry collision box size=0.9793560999741125 0.10011075637710332 0.43532425011787323; visual box size=0.9793560999741125 0.10011075637710332 0.43532425011787323
- link 2: geometry collision box size=0.32134941478475854 0.9260789327678697 0.47277242871518244; visual box size=0.32134941478475854 0.9260789327678697 0.47277242871518244
- link 20: geometry collision box size=0.17104950052199375 0.8832406905184543 0.07383781941567102; visual box size=0.17104950052199375 0.8832406905184543 0.07383781941567102
- link 21: geometry collision box size=0.09052254552743988 0.5403869039419334 0.43337146911921853; visual box size=0.09052254552743988 0.5403869039419334 0.43337146911921853
- link 22: geometry collision box size=0.25814460717388943 0.2763075227315176 1.364239250109236; visual box size=0.25814460717388943 0.2763075227315176 1.364239250109236
- link 23: geometry collision box size=0.24625465169325034 0.8125035636574851 0.08529725732953972; visual box size=0.24625465169325034 0.8125035636574851 0.08529725732953972
- link 24: geometry collision box size=0.8397848290501293 0.6675668256059901 0.1504634925612244; visual box size=0.8397848290501293 0.6675668256059901 0.1504634925612244
- link 3: geometry collision box size=0.9997738592261386 0.5342464373314322 0.9303865564538629; visual box size=0.9997738592261386 0.5342464373314322 0.9303865564538629
- link 4: geometry collision box size=0.45965804288913303 0.8736971684246707 0.8786330324019288; visual box size=0.45965804288913303 0.8736971684246707 0.8786330324019288
- link 5: geometry collision box size=0.49284538237809095 0.40297653878910455 0.5766192250517024; visual box size=0.49284538237809095 0.40297653878910455 0.5766192250517024
- link 6: geometry collision box size=0.9381690872069791 0.750750557298655 0.1447477425463689; visual box size=0.9381690872069791 0.750750557298655 0.1447477425463689
- link 7: geometry collision box size=0.7055874299393511 0.03037774217567557 0.782024881664129; visual box size=0.7055874299393511 0.03037774217567557 0.782024881664129
- link 8: geometry collision box size=0.8839962345651574 0.3721140644789014 0.9200365001627796; visual box size=0.8839962345651574 0.3721140644789014 0.9200365001627796
- link 9: geometry collision box size=0.2960523519921038 0.5298232308014063 0.541351882700517; visual box size=0.2960523519921038 0.5298232308014063 0.541351882700517
Joints:
- joint 0_1: axis 0 1 0 -> 1 0 1
- joint 0_13: axis 0 0 1 -> 1 1 1
- joint 0_19: axis 0 1 0 -> 1 0 0
- joint 0_7: axis 0 1 1 -> 1 0 0
- joint 10_11: origin xyz=0 0 -0.028030414618231882 rpy=0 0 0 -> xyz=0 0 -1.4554611236959727 rpy=0 0 0
- joint 11_12: axis 1 1 1 -> 0 1 1; origin xyz=0 0 -0.7142539744148921 rpy=0 0 0 -> xyz=0 0 -0.060794889373184655 rpy=0 0 0
- joint 13_14: axis 0 0 1 -> 0 1 0; origin xyz=0 -0.7688106657399588 0 rpy=0 0 0 -> xyz=0 -0.25412788202751113 0 rpy=0 0 0
- joint 14_15: axis 0 1 1 -> 1 0 0; origin xyz=0 -0.0808644822821214 0 rpy=0 0 0 -> xyz=0 -0.3751101172440727 0 rpy=0 0 0
- joint 15_16: axis 1 0 1 -> 1 0 0; origin xyz=0 -0.26448597764110515 -0.49934868097685925 rpy=0 0 0 -> xyz=0 -0.22767364328708328 -0.2965101560905207 rpy=0 0 0
- joint 16_17: axis 1 1 0 -> 1 0 1; origin xyz=0 0 -1.0107176614858975 rpy=0 0 0 -> xyz=0 0 -0.9632596283696517 rpy=0 0 0
- joint 17_18: axis 1 1 0 -> 0 1 0; origin xyz=0 0 -0.05625971505365884 rpy=0 0 0 -> xyz=0 0 -0.3385209032505026 rpy=0 0 0
- joint 19_20: origin xyz=0 0.5914392503450112 0 rpy=0 0 0 -> xyz=0 0.10011075637710332 0 rpy=0 0 0
- joint 1_2: axis 0 0 1 -> 1 0 1; origin xyz=-0.26741079010654767 0 0 rpy=0 0 0 -> xyz=-0.05738224560673355 0 0 rpy=0 0 0
- joint 20_21: axis 1 1 0 -> 0 1 0; origin xyz=0 0.7250453504166596 0 rpy=0 0 0 -> xyz=0 0.8832406905184543 0 rpy=0 0 0
- joint 21_22: origin xyz=0 0.20545459342919092 -0.09374475898693496 rpy=0 0 0 -> xyz=0 0.2701934519709667 -0.21668573455960927 rpy=0 0 0
- joint 22_23: axis 1 0 1 -> 0 1 0; origin xyz=0 0 -1.3180428593938645 rpy=0 0 0 -> xyz=0 0 -1.364239250109236 rpy=0 0 0
- joint 23_24: axis 1 0 1 -> 0 1 1; origin xyz=0 0 -0.14483923038293403 rpy=0 0 0 -> xyz=0 0 -0.08529725732953972 rpy=0 0 0
- joint 2_3: axis 1 1 0 -> 0 1 0; origin xyz=-0.19902107772747135 0 0 rpy=0 0 0 -> xyz=-0.32134941478475854 0 0 rpy=0 0 0
- joint 3_4: axis 1 1 0 -> 0 1 1; origin xyz=-0.4331004807920566 0 -0.18807166594871322 rpy=0 0 0 -> xyz=-0.4998869296130693 0 -0.46519327822693146 rpy=0 0 0
- joint 4_5: axis 0 0 1 -> 1 0 1; origin xyz=0 0 -0.18256115076063698 rpy=0 0 0 -> xyz=0 0 -0.8786330324019288 rpy=0 0 0
- joint 5_6: axis 1 0 0 -> 1 1 1; origin xyz=0 0 -0.17630804673113457 rpy=0 0 0 -> xyz=0 0 -0.5766192250517024 rpy=0 0 0
- joint 7_8: axis 0 1 0 -> 1 1 1; origin xyz=0.983390365260045 0 0 rpy=0 0 0 -> xyz=0.7055874299393511 0 0 rpy=0 0 0
- joint 8_9: origin xyz=0.8459216146793201 0 0 rpy=0 0 0 -> xyz=0.8839962345651574 0 0 rpy=0 0 0
- joint 9_10: axis 1 1 0 -> 1 1 1; origin xyz=0.36832877638501815 0 -0.16752141694536188 rpy=0 0 0 -> xyz=0.1480261759960519 0 -0.2706759413502585 rpy=0 0 0
