Commit message: commit

File: body0.urdf (robot description, URDF)
Before this commit: robot robot, 17 links, 16 joints
Links:
- added link 17, mass 1; collision box size=0.1037864935106858 0.8300114617077825 0.07653584561094595; visual box size=0.1037864935106858 0.8300114617077825 0.07653584561094595
- added link 18, mass 1; collision box size=0.5506363838084969 0.3255033338308685 0.7418739870697488; visual box size=0.5506363838084969 0.3255033338308685 0.7418739870697488
- added link 19, mass 1; collision box size=0.5794957073657835 0.12815365452802185 0.5159048800220319; visual box size=0.5794957073657835 0.12815365452802185 0.5159048800220319
- added link 20, mass 1; collision box size=0.8438555922442371 0.9195409425873247 0.9196619407309652; visual box size=0.8438555922442371 0.9195409425873247 0.9196619407309652
- added link 21, mass 1; collision box size=0.05901037564718348 0.7659528842327329 0.5129080770985339; visual box size=0.05901037564718348 0.7659528842327329 0.5129080770985339
- added link 22, mass 1; collision box size=0.5574858792049897 0.3993882111347813 0.21646977063288794; visual box size=0.5574858792049897 0.3993882111347813 0.21646977063288794
- added link 23, mass 1; collision box size=0.5598905248693518 0.24697629654717135 1.2500725853338759; visual box size=0.5598905248693518 0.24697629654717135 1.2500725853338759
- added link 24, mass 1; collision box size=0.34761172125154916 0.193973764551848 1.1334576440332365; visual box size=0.34761172125154916 0.193973764551848 1.1334576440332365
- added link 25, mass 1; collision box size=0.5354788652317081 0.7693552955384096 0.13967075177676658; visual box size=0.5354788652317081 0.7693552955384096 0.13967075177676658
- added link 26, mass 1; collision box size=0.512013174124303 0.9366921756724736 0.037331687764691424; visual box size=0.512013174124303 0.9366921756724736 0.037331687764691424
- added link 27, mass 1; collision box size=0.9273283794134634 0.1430364631495885 0.8998940249430377; visual box size=0.9273283794134634 0.1430364631495885 0.8998940249430377
- added link 28, mass 1; collision box size=0.8606374637387865 0.8682463523792617 0.6139409661456888; visual box size=0.8606374637387865 0.8682463523792617 0.6139409661456888
- added link 29, mass 1; collision box size=0.5144912445261443 0.05256201261852034 0.5525572646171383; visual box size=0.5144912445261443 0.05256201261852034 0.5525572646171383
- added link 30, mass 1; collision box size=0.3250121369965544 0.09578789863810888 0.08916190089413907; visual box size=0.3250121369965544 0.09578789863810888 0.08916190089413907
- added link 31, mass 1; collision box size=0.3550234313527897 0.5585065485590243 1.1544700975709619; visual box size=0.3550234313527897 0.5585065485590243 1.1544700975709619
- added link 32, mass 1; collision box size=0.2645920386693418 0.4333751193654497 1.3563680015348991; visual box size=0.2645920386693418 0.4333751193654497 1.3563680015348991
- link 1: geometry collision box size=0.804029514606451 0.8061784263109566 0.3526429753392083; visual box size=0.804029514606451 0.8061784263109566 0.3526429753392083
- link 10: geometry collision box size=0.010974386803754177 0.6110095639071247 0.47240915097335134; visual box size=0.010974386803754177 0.6110095639071247 0.47240915097335134
- link 11: geometry collision box size=0.3802615663650566 0.4089441326079316 0.7062764631717903; visual box size=0.3802615663650566 0.4089441326079316 0.7062764631717903
- link 12: geometry collision box size=0.3763428946224874 0.4913060611065593 0.14291493379214115; visual box size=0.3763428946224874 0.4913060611065593 0.14291493379214115
- link 13: geometry collision box size=0.31081668519277683 0.5141359770253046 0.822722526391347; visual box size=0.31081668519277683 0.5141359770253046 0.822722526391347
- link 14: geometry collision box size=0.2813451013892403 0.5047994553876097 0.7591712767619561; visual box size=0.2813451013892403 0.5047994553876097 0.7591712767619561
- link 15: geometry collision box size=0.13329293479670434 0.0673280610727679 0.9888065859887156; visual box size=0.13329293479670434 0.0673280610727679 0.9888065859887156
- link 16: geometry collision box size=0.4511175361547195 0.8700643346683278 0.8520221372493284; visual box size=0.4511175361547195 0.8700643346683278 0.8520221372493284
- link 2: geometry collision box size=0.23409770836126864 0.7237250305608426 0.6827749990319854; visual box size=0.23409770836126864 0.7237250305608426 0.6827749990319854
- link 3: geometry collision box size=0.10165227081924322 0.42329257642242957 0.09176915046941303; visual box size=0.10165227081924322 0.42329257642242957 0.09176915046941303
- link 4: geometry collision box size=0.3111530878257709 0.20126990185083493 0.23708351754763268; visual box size=0.3111530878257709 0.20126990185083493 0.23708351754763268
- link 5: geometry collision box size=0.9413746370465742 0.28320877384824517 0.7105008444125589; visual box size=0.9413746370465742 0.28320877384824517 0.7105008444125589
- link 6: geometry collision box size=0.46381504552188124 0.11297335819983345 0.6949399668666074; visual box size=0.46381504552188124 0.11297335819983345 0.6949399668666074
- link 7: geometry collision box size=0.9011802522854883 0.1627821818450661 1.6252940572466372; visual box size=0.9011802522854883 0.1627821818450661 1.6252940572466372
- link 8: geometry collision box size=0.5402256663203483 0.7314319818962104 0.27976597588675545; visual box size=0.5402256663203483 0.7314319818962104 0.27976597588675545
- link 9: geometry collision box size=0.34793875277401787 0.5147115007868206 0.5496482472701112; visual box size=0.34793875277401787 0.5147115007868206 0.5496482472701112
Joints:
- removed joint 0_13
- removed joint 0_5
- added joint 0_17: type revolute, parent 0, child 17, origin xyz=0 -0.75 3 rpy=0 0 0, axis 0 0 1, limit lower=-3.14159 upper=3.14159 effort=0.0 velocity=0.0
- added joint 0_25: type revolute, parent 0, child 25, origin xyz=0 0.75 3 rpy=0 0 0, axis 1 0 0, limit lower=-3.14159 upper=3.14159 effort=0.0 velocity=0.0
- added joint 12_13: type revolute, parent 12, child 13, origin xyz=0.3763428946224874 0 0 rpy=0 0 0, axis 1 1 1, limit lower=-3.14159 upper=3.14159 effort=0.0 velocity=0.0
- added joint 17_18: type revolute, parent 17, child 18, origin xyz=0 -0.8300114617077825 0 rpy=0 0 0, axis 1 0 0, limit lower=-3.14159 upper=3.14159 effort=0.0 velocity=0.0
- added joint 18_19: type revolute, parent 18, child 19, origin xyz=0 -0.3255033338308685 0 rpy=0 0 0, axis 0 1 0, limit lower=-3.14159 upper=3.14159 effort=0.0 velocity=0.0
- added joint 19_20: type revolute, parent 19, child 20, origin xyz=0 -0.12815365452802185 0 rpy=0 0 0, axis 1 1 1, limit lower=-3.14159 upper=3.14159 effort=0.0 velocity=0.0
- added joint 20_21: type revolute, parent 20, child 21, origin xyz=0 -0.9195409425873247 0 rpy=0 0 0, axis 0 1 1, limit lower=-3.14159 upper=3.14159 effort=0.0 velocity=0.0
- added joint 21_22: type revolute, parent 21, child 22, origin xyz=0 -0.38297644211636644 -0.25645403854926696 rpy=0 0 0, axis 1 1 0, limit lower=-3.14159 upper=3.14159 effort=0.0 velocity=0.0
- added joint 22_23: type revolute, parent 22, child 23, origin xyz=0 0 -0.21646977063288794 rpy=0 0 0, axis 0 1 1, limit lower=-3.14159 upper=3.14159 effort=0.0 velocity=0.0
- added joint 23_24: type revolute, parent 23, child 24, origin xyz=0 0 -1.2500725853338759 rpy=0 0 0, axis 1 0 0, limit lower=-3.14159 upper=3.14159 effort=0.0 velocity=0.0
- added joint 25_26: type revolute, parent 25, child 26, origin xyz=0 0.7693552955384096 0 rpy=0 0 0, axis 0 1 0, limit lower=-3.14159 upper=3.14159 effort=0.0 velocity=0.0
- added joint 26_27: type revolute, parent 26, child 27, origin xyz=0 0.9366921756724736 0 rpy=0 0 0, axis 1 1 1, limit lower=-3.14159 upper=3.14159 effort=0.0 velocity=0.0
- added joint 27_28: type revolute, parent 27, child 28, origin xyz=0 0.1430364631495885 0 rpy=0 0 0, axis 0 1 1, limit lower=-3.14159 upper=3.14159 effort=0.0 velocity=0.0
- added joint 28_29: type revolute, parent 28, child 29, origin xyz=0 0.8682463523792617 0 rpy=0 0 0, axis 1 0 0, limit lower=-3.14159 upper=3.14159 effort=0.0 velocity=0.0
- added joint 29_30: type revolute, parent 29, child 30, origin xyz=0 0.02628100630926017 -0.27627863230856914 rpy=0 0 0, axis 1 1 1, limit lower=-3.14159 upper=3.14159 effort=0.0 velocity=0.0
- added joint 30_31: type revolute, parent 30, child 31, origin xyz=0 0 -0.08916190089413907 rpy=0 0 0, axis 1 0 0, limit lower=-3.14159 upper=3.14159 effort=0.0 velocity=0.0
- added joint 31_32: type revolute, parent 31, child 32, origin xyz=0 0 -1.1544700975709619 rpy=0 0 0, axis 1 0 0, limit lower=-3.14159 upper=3.14159 effort=0.0 velocity=0.0
- added joint 4_5: type revolute, parent 4, child 5, origin xyz=-0.3111530878257709 0 0 rpy=0 0 0, axis 1 0 0, limit lower=-3.14159 upper=3.14159 effort=0.0 velocity=0.0
- joint 0_1: axis 1 0 1 -> 0 0 1; origin xyz=-0.75 0 2 rpy=0 0 0 -> xyz=-0.75 0 3 rpy=0 0 0
- joint 0_9: axis 0 0 1 -> 1 0 0; origin xyz=0 -0.75 2 rpy=0 0 0 -> xyz=0.75 0 3 rpy=0 0 0
- joint 10_11: axis 1 0 1 -> 1 0 0; origin xyz=0 0 -1.5442231085690195 rpy=0 0 0 -> xyz=0.010974386803754177 0 0 rpy=0 0 0
- joint 11_12: axis 1 0 0 -> 1 0 1; origin xyz=0 0 -0.04402900591548745 rpy=0 0 0 -> xyz=0.3802615663650566 0 0 rpy=0 0 0
- joint 13_14: origin xyz=0 0.16343552317947102 -0.23343760576955624 rpy=0 0 0 -> xyz=0.15540834259638842 0 -0.4113612631956735 rpy=0 0 0
- joint 14_15: axis 0 1 1 -> 1 0 0; origin xyz=0 0 -1.0770015167621245 rpy=0 0 0 -> xyz=0 0 -0.7591712767619561 rpy=0 0 0
- joint 15_16: axis 0 0 1 -> 0 1 0; origin xyz=0 0 -0.07236522730101946 rpy=0 0 0 -> xyz=0 0 -0.9888065859887156 rpy=0 0 0
- joint 1_2: axis 0 0 1 -> 0 1 0; origin xyz=-0.06114054086376619 0 -0.19370952604465974 rpy=0 0 0 -> xyz=-0.804029514606451 0 0 rpy=0 0 0
- joint 2_3: axis 1 0 0 -> 0 0 1; origin xyz=0 0 -1.5384063081681632 rpy=0 0 0 -> xyz=-0.23409770836126864 0 0 rpy=0 0 0
- joint 3_4: axis 1 0 1 -> 1 1 0; origin xyz=0 0 -0.05728296444989989 rpy=0 0 0 -> xyz=-0.10165227081924322 0 0 rpy=0 0 0
- joint 5_6: axis 1 0 1 -> 0 1 1; origin xyz=0.32971649288415616 0 -0.2771252216673125 rpy=0 0 0 -> xyz=-0.4706873185232871 0 -0.35525042220627945 rpy=0 0 0
- joint 6_7: axis 1 1 0 -> 0 1 0; origin xyz=0 0 -1.28600988362806 rpy=0 0 0 -> xyz=0 0 -0.6949399668666074 rpy=0 0 0
- joint 7_8: axis 1 1 1 -> 1 0 0; origin xyz=0 0 -0.18441707251839215 rpy=0 0 0 -> xyz=0 0 -1.6252940572466372 rpy=0 0 0
- joint 9_10: axis 1 1 1 -> 1 1 0; origin xyz=0 -0.40865188682354986 -0.17444911201292929 rpy=0 0 0 -> xyz=0.34793875277401787 0 0 rpy=0 0 0

File: body3.urdf (robot description, URDF)
Before this commit: robot robot, 25 links, 24 joints
Links:
- added link 25, mass 1; collision box size=0.02989161078846614 0.7386942574281974 0.271835458958817; visual box size=0.02989161078846614 0.7386942574281974 0.271835458958817
- added link 26, mass 1; collision box size=0.6089953192058238 0.5513843766901655 1.1481715054140977; visual box size=0.6089953192058238 0.5513843766901655 1.1481715054140977
- added link 27, mass 1; collision box size=0.10830179817124652 0.06654366982639426 0.7525815004863108; visual box size=0.10830179817124652 0.06654366982639426 0.7525815004863108
- added link 28, mass 1; collision box size=0.27806024206173074 0.1891973639671337 0.6992469940995916; visual box size=0.27806024206173074 0.1891973639671337 0.6992469940995916
- link 1: geometry collision box size=0.6876676849063272 0.6053366308026952 0.7640794252501124; visual box size=0.6876676849063272 0.6053366308026952 0.7640794252501124
- link 10: geometry collision box size=0.036198386004061445 0.782949354216897 0.6878088311406287; visual box size=0.036198386004061445 0.782949354216897 0.6878088311406287
- link 11: geometry collision box size=0.39924449625629155 0.6736531864233964 0.9404596190103194; visual box size=0.39924449625629155 0.6736531864233964 0.9404596190103194
- link 12: geometry collision box size=0.9177248813125208 0.2874038422726676 0.1962407270446708; visual box size=0.9177248813125208 0.2874038422726676 0.1962407270446708
- link 13: geometry collision box size=0.027479100921945054 0.22515500546381384 0.1754785358163641; visual box size=0.027479100921945054 0.22515500546381384 0.1754785358163641
- link 14: geometry collision box size=0.449018775124449 0.20386602639404738 2.2282807371389652; visual box size=0.449018775124449 0.20386602639404738 2.2282807371389652
- link 15: geometry collision box size=0.04058304049947625 0.1594483256493432 0.2371720755825386; visual box size=0.04058304049947625 0.1594483256493432 0.2371720755825386
- link 16: geometry collision box size=0.5297974981311903 0.8332043591969172 0.1188823732287888; visual box size=0.5297974981311903 0.8332043591969172 0.1188823732287888
- link 17: geometry collision box size=0.229011141058991 0.18080807091116113 0.5085850336940188; visual box size=0.229011141058991 0.18080807091116113 0.5085850336940188
- link 18: geometry collision box size=0.28950351892153203 0.5481145851436627 0.5237841767040736; visual box size=0.28950351892153203 0.5481145851436627 0.5237841767040736
- link 19: geometry collision box size=0.6449434893495419 0.04879786186295598 1.7093037894163585; visual box size=0.6449434893495419 0.04879786186295598 1.7093037894163585
- link 2: geometry collision box size=0.8608207679151323 0.0435555910447053 0.6083644190611832; visual box size=0.8608207679151323 0.0435555910447053 0.6083644190611832
- link 20: geometry collision box size=0.5890823511133633 0.04983143429839809 0.7634179257355155; visual box size=0.5890823511133633 0.04983143429839809 0.7634179257355155
- link 21: geometry collision box size=0.94864394725426 0.702959667535773 0.1272782848481261; visual box size=0.94864394725426 0.702959667535773 0.1272782848481261
- link 22: geometry collision box size=0.17912429946462494 0.05802925784526458 0.019471672297639464; visual box size=0.17912429946462494 0.05802925784526458 0.019471672297639464
- link 23: geometry collision box size=0.3656406898030705 0.19328065006713369 0.3596858889972323; visual box size=0.3656406898030705 0.19328065006713369 0.3596858889972323
- link 24: geometry collision box size=0.6683026841271761 0.4401462989548772 0.4805056806699407; visual box size=0.6683026841271761 0.4401462989548772 0.4805056806699407
- link 3: geometry collision box size=0.9356671970923297 0.3594306742817098 0.02503805238221779; visual box size=0.9356671970923297 0.3594306742817098 0.02503805238221779
- link 4: geometry collision box size=0.323303274393001 0.5445781707744113 0.6750905256105788; visual box size=0.323303274393001 0.5445781707744113 0.6750905256105788
- link 5: geometry collision box size=0.3861884644738328 0.38042456503863187 1.0321733234269925; visual box size=0.3861884644738328 0.38042456503863187 1.0321733234269925
- link 6: geometry collision box size=0.15343091571988432 0.7864360511531704 0.69327897971451; visual box size=0.15343091571988432 0.7864360511531704 0.69327897971451
- link 7: geometry collision box size=0.8519291540502371 0.5843854724144664 0.8745476968584975; visual box size=0.8519291540502371 0.5843854724144664 0.8745476968584975
- link 8: geometry collision box size=0.2710358798168453 0.4619624621872316 0.6644244637204892; visual box size=0.2710358798168453 0.4619624621872316 0.6644244637204892
- link 9: geometry collision box size=0.19057351659614485 0.5595692720327974 0.7806669788085945; visual box size=0.19057351659614485 0.5595692720327974 0.7806669788085945
Joints:
- removed joint 0_13
- removed joint 0_19
- removed joint 0_7
- removed joint 14_15
- removed joint 21_22
- removed joint 7_8
- added joint 0_15: type revolute, parent 0, child 15, origin xyz=0 -0.75 3 rpy=0 0 0, axis 0 1 0, limit lower=-3.14159 upper=3.14159 effort=0.0 velocity=0.0
- added joint 0_22: type revolute, parent 0, child 22, origin xyz=0 0.75 3 rpy=0 0 0, axis 1 0 0, limit lower=-3.14159 upper=3.14159 effort=0.0 velocity=0.0
- added joint 0_8: type revolute, parent 0, child 8, origin xyz=0.75 0 3 rpy=0 0 0, axis 1 1 1, limit lower=-3.14159 upper=3.14159 effort=0.0 velocity=0.0
- added joint 12_13: type revolute, parent 12, child 13, origin xyz=0 0 -0.1962407270446708 rpy=0 0 0, axis 0 0 1, limit lower=-3.14159 upper=3.14159 effort=0.0 velocity=0.0
- added joint 18_19: type revolute, parent 18, child 19, origin xyz=0 -0.27405729257183137 -0.2618920883520368 rpy=0 0 0, axis 0 0 1, limit lower=-3.14159 upper=3.14159 effort=0.0 velocity=0.0
- added joint 24_25: type revolute, parent 24, child 25, origin xyz=0 0.4401462989548772 0 rpy=0 0 0, axis 1 0 0, limit lower=-3.14159 upper=3.14159 effort=0.0 velocity=0.0
- added joint 25_26: type revolute, parent 25, child 26, origin xyz=0 0.3693471287140987 -0.1359177294794085 rpy=0 0 0, axis 0 1 0, limit lower=-3.14159 upper=3.14159 effort=0.0 velocity=0.0
- added joint 26_27: type revolute, parent 26, child 27, origin xyz=0 0 -1.1481715054140977 rpy=0 0 0, axis 0 1 1, limit lower=-3.14159 upper=3.14159 effort=0.0 velocity=0.0
- added joint 27_28: type revolute, parent 27, child 28, origin xyz=0 0 -0.7525815004863108 rpy=0 0 0, axis 1 0 1, limit lower=-3.14159 upper=3.14159 effort=0.0 velocity=0.0
- added joint 6_7: type revolute, parent 6, child 7, origin xyz=0 0 -0.69327897971451 rpy=0 0 0, axis 0 1 0, limit lower=-3.14159 upper=3.14159 effort=0.0 velocity=0.0
- joint 0_1: axis 1 0 1 -> 0 0 1; origin xyz=-0.75 0 2 rpy=0 0 0 -> xyz=-0.75 0 3 rpy=0 0 0
- joint 10_11: axis 1 0 0 -> 0 1 0; origin xyz=0 0 -1.4554611236959727 rpy=0 0 0 -> xyz=0.036198386004061445 0 0 rpy=0 0 0
- joint 11_12: axis 0 1 1 -> 0 0 1; origin xyz=0 0 -0.060794889373184655 rpy=0 0 0 -> xyz=0.19962224812814577 0 -0.4702298095051597 rpy=0 0 0
- joint 13_14: axis 0 1 0 -> 1 0 0; origin xyz=0 -0.25412788202751113 0 rpy=0 0 0 -> xyz=0 0 -0.1754785358163641 rpy=0 0 0
- joint 15_16: axis 1 0 0 -> 1 0 1; origin xyz=0 -0.22767364328708328 -0.2965101560905207 rpy=0 0 0 -> xyz=0 -0.1594483256493432 0 rpy=0 0 0
- joint 16_17: axis 1 0 1 -> 0 1 1; origin xyz=0 0 -0.9632596283696517 rpy=0 0 0 -> xyz=0 -0.8332043591969172 0 rpy=0 0 0
- joint 17_18: axis 0 1 0 -> 1 1 0; origin xyz=0 0 -0.3385209032505026 rpy=0 0 0 -> xyz=0 -0.18080807091116113 0 rpy=0 0 0
- joint 19_20: axis 1 0 1 -> 0 1 0; origin xyz=0 0.10011075637710332 0 rpy=0 0 0 -> xyz=0 0 -1.7093037894163585 rpy=0 0 0
- joint 1_2: origin xyz=-0.05738224560673355 0 0 rpy=0 0 0 -> xyz=-0.6876676849063272 0 0 rpy=0 0 0
- joint 20_21: axis 0 1 0 -> 0 0 1; origin xyz=0 0.8832406905184543 0 rpy=0 0 0 -> xyz=0 0 -0.7634179257355155 rpy=0 0 0
- joint 22_23: axis 0 1 0 -> 1 1 1; origin xyz=0 0 -1.364239250109236 rpy=0 0 0 -> xyz=0 0.05802925784526458 0 rpy=0 0 0
- joint 23_24: axis 0 1 1 -> 1 1 0; origin xyz=0 0 -0.08529725732953972 rpy=0 0 0 -> xyz=0 0.19328065006713369 0 rpy=0 0 0
- joint 2_3: axis 0 1 0 -> 1 1 0; origin xyz=-0.32134941478475854 0 0 rpy=0 0 0 -> xyz=-0.8608207679151323 0 0 rpy=0 0 0
- joint 3_4: axis 0 1 1 -> 0 0 1; origin xyz=-0.4998869296130693 0 -0.46519327822693146 rpy=0 0 0 -> xyz=-0.9356671970923297 0 0 rpy=0 0 0
- joint 4_5: axis 1 0 1 -> 0 1 1; origin xyz=0 0 -0.8786330324019288 rpy=0 0 0 -> xyz=-0.1616516371965005 0 -0.3375452628052894 rpy=0 0 0
- joint 5_6: axis 1 1 1 -> 0 1 0; origin xyz=0 0 -0.5766192250517024 rpy=0 0 0 -> xyz=0 0 -1.0321733234269925 rpy=0 0 0
- joint 8_9: axis 0 1 1 -> 0 0 1; origin xyz=0.8839962345651574 0 0 rpy=0 0 0 -> xyz=0.2710358798168453 0 0 rpy=0 0 0
- joint 9_10: axis 1 1 1 -> 0 1 1; origin xyz=0.1480261759960519 0 -0.2706759413502585 rpy=0 0 0 -> xyz=0.19057351659614485 0 0 rpy=0 0 0
