Commit message: commit

File: body5.urdf (robot description, URDF)
Before this commit: robot robot, 29 links, 28 joints
Links:
- link 1: geometry collision box size=0.39193272144375446 0.28366113685801575 0.701383466493154; visual box size=0.39193272144375446 0.28366113685801575 0.701383466493154
- link 10: geometry collision box size=0.5804459720622157 0.984497049363341 0.3622869212812043; visual box size=0.5804459720622157 0.984497049363341 0.3622869212812043
- link 11: geometry collision box size=0.2704872343082477 0.34177889839355335 0.5435214230605151; visual box size=0.2704872343082477 0.34177889839355335 0.5435214230605151
- link 12: geometry collision box size=0.6812102323788055 0.1711244359187981 1.8144305319704244; visual box size=0.6812102323788055 0.1711244359187981 1.8144305319704244
- link 13: geometry collision box size=0.25766866923110676 0.24483860870409102 0.6854638010211774; visual box size=0.25766866923110676 0.24483860870409102 0.6854638010211774
- link 14: geometry collision box size=0.7153912149042381 0.2676568502673242 0.10010566700839829; visual box size=0.7153912149042381 0.2676568502673242 0.10010566700839829
- link 15: geometry collision box size=0.3718744566802268 0.5792121771683727 0.7050133147083496; visual box size=0.3718744566802268 0.5792121771683727 0.7050133147083496
- link 16: geometry collision box size=0.3362581124040619 0.08328874965330979 0.09837277907854114; visual box size=0.3362581124040619 0.08328874965330979 0.09837277907854114
- link 17: geometry collision box size=0.44621030838234843 0.6180366071721655 0.3738228709937155; visual box size=0.44621030838234843 0.6180366071721655 0.3738228709937155
- link 18: geometry collision box size=0.4109487817103783 0.6808500115339119 0.6034718430631822; visual box size=0.4109487817103783 0.6808500115339119 0.6034718430631822
- link 19: geometry collision box size=0.033842003365664564 0.41301745244681887 1.3974433217233582; visual box size=0.033842003365664564 0.41301745244681887 1.3974433217233582
- link 2: geometry collision box size=0.241642874180782 0.3912962338193321 0.7045667871231717; visual box size=0.241642874180782 0.3912962338193321 0.7045667871231717
- link 20: geometry collision box size=0.37928531577724167 0.07479561513590338 0.4414041826640734; visual box size=0.37928531577724167 0.07479561513590338 0.4414041826640734
- link 21: geometry collision box size=0.4738463366077461 0.3310223061988963 0.7611524956125686; visual box size=0.4738463366077461 0.3310223061988963 0.7611524956125686
- link 22: geometry collision box size=0.46428368318488034 0.8806627937096363 0.7892672546776018; visual box size=0.46428368318488034 0.8806627937096363 0.7892672546776018
- link 23: geometry collision box size=0.5228711649423005 0.7605392831195475 0.34392864412918633; visual box size=0.5228711649423005 0.7605392831195475 0.34392864412918633
- link 24: geometry collision box size=0.9105310985084119 0.566469731423579 0.9010768018443602; visual box size=0.9105310985084119 0.566469731423579 0.9010768018443602
- link 25: geometry collision box size=0.13124042996697483 0.29373030720776616 0.7565002301541233; visual box size=0.13124042996697483 0.29373030720776616 0.7565002301541233
- link 26: geometry collision box size=0.22704933480162615 0.18686412238657868 1.137319627571601; visual box size=0.22704933480162615 0.18686412238657868 1.137319627571601
- link 27: geometry collision box size=0.5047840531100016 0.4023808054954796 1.062675918609001; visual box size=0.5047840531100016 0.4023808054954796 1.062675918609001
- link 28: geometry collision box size=0.8096240522819118 0.13771563667094622 0.4000044538193981; visual box size=0.8096240522819118 0.13771563667094622 0.4000044538193981
- link 3: geometry collision box size=0.9170572438288018 0.39711622654727596 0.4860477801327622; visual box size=0.9170572438288018 0.39711622654727596 0.4860477801327622
- link 4: geometry collision box size=0.9336658677333168 0.913897221312311 0.32713290386133176; visual box size=0.9336658677333168 0.913897221312311 0.32713290386133176
- link 5: geometry collision box size=0.7976698483684235 0.5285671440452816 1.1505349552261221; visual box size=0.7976698483684235 0.5285671440452816 1.1505349552261221
- link 6: geometry collision box size=0.7913724519011263 0.8708532964493152 1.378865732156263; visual box size=0.7913724519011263 0.8708532964493152 1.378865732156263
- link 7: geometry collision box size=0.7843475658712564 0.9675571661626299 0.07059931261761498; visual box size=0.7843475658712564 0.9675571661626299 0.07059931261761498
- link 8: geometry collision box size=0.046925375028527894 0.23552042818847163 0.8603142675170478; visual box size=0.046925375028527894 0.23552042818847163 0.8603142675170478
- link 9: geometry collision box size=0.5242017776939347 0.45818967266672406 0.9288634143190145; visual box size=0.5242017776939347 0.45818967266672406 0.9288634143190145
Joints:
- joint 0_1: axis 1 0 0 -> 1 1 1
- joint 0_15: axis 1 1 0 -> 0 1 0
- joint 0_22: axis 0 0 1 -> 0 1 0
- joint 0_8: axis 0 0 1 -> 0 1 1
- joint 10_11: axis 0 1 0 -> 1 1 1; origin xyz=0.03117363023433073 0 0 rpy=0 0 0 -> xyz=0.5804459720622157 0 0 rpy=0 0 0
- joint 11_12: axis 1 1 1 -> 0 1 0; origin xyz=0.037035527534092116 0 -0.27239276658366696 rpy=0 0 0 -> xyz=0.13524361715412386 0 -0.27176071153025755 rpy=0 0 0
- joint 12_13: axis 1 1 0 -> 0 1 1; origin xyz=0 0 -0.939648048036766 rpy=0 0 0 -> xyz=0 0 -1.8144305319704244 rpy=0 0 0
- joint 13_14: axis 0 1 1 -> 1 0 0; origin xyz=0 0 -0.6030077073062268 rpy=0 0 0 -> xyz=0 0 -0.6854638010211774 rpy=0 0 0
- joint 15_16: axis 0 1 1 -> 1 1 0; origin xyz=0 -0.7905507572729643 0 rpy=0 0 0 -> xyz=0 -0.5792121771683727 0 rpy=0 0 0
- joint 16_17: axis 0 1 0 -> 1 1 1; origin xyz=0 -0.8320157729187685 0 rpy=0 0 0 -> xyz=0 -0.08328874965330979 0 rpy=0 0 0
- joint 17_18: axis 1 0 0 -> 1 0 1; origin xyz=0 -0.4720065069480902 0 rpy=0 0 0 -> xyz=0 -0.6180366071721655 0 rpy=0 0 0
- joint 18_19: axis 1 0 0 -> 0 0 1; origin xyz=0 -0.02287104595368794 -0.35596078443536044 rpy=0 0 0 -> xyz=0 -0.34042500576695595 -0.3017359215315911 rpy=0 0 0
- joint 19_20: axis 0 1 1 -> 1 0 0; origin xyz=0 0 -2.3298421440031705 rpy=0 0 0 -> xyz=0 0 -1.3974433217233582 rpy=0 0 0
- joint 1_2: origin xyz=-0.4979006927525672 0 0 rpy=0 0 0 -> xyz=-0.39193272144375446 0 0 rpy=0 0 0
- joint 20_21: axis 1 1 0 -> 1 1 1; origin xyz=0 0 -0.23878978342009116 rpy=0 0 0 -> xyz=0 0 -0.4414041826640734 rpy=0 0 0
- joint 22_23: axis 1 1 0 -> 0 1 0; origin xyz=0 0.3466227464231907 0 rpy=0 0 0 -> xyz=0 0.8806627937096363 0 rpy=0 0 0
- joint 23_24: axis 0 0 1 -> 0 1 1; origin xyz=0 0.5753661461131512 0 rpy=0 0 0 -> xyz=0 0.7605392831195475 0 rpy=0 0 0
- joint 24_25: axis 1 0 0 -> 1 1 1; origin xyz=0 0.3303744543170063 0 rpy=0 0 0 -> xyz=0 0.566469731423579 0 rpy=0 0 0
- joint 25_26: axis 1 0 0 -> 1 1 0; origin xyz=0 0.015855983249372818 -0.4205472402202497 rpy=0 0 0 -> xyz=0 0.14686515360388308 -0.37825011507706163 rpy=0 0 0
- joint 26_27: axis 1 0 0 -> 0 0 1; origin xyz=0 0 -2.5254352704082503 rpy=0 0 0 -> xyz=0 0 -1.137319627571601 rpy=0 0 0
- joint 27_28: axis 1 0 0 -> 1 0 1; origin xyz=0 0 -0.01743779744345275 rpy=0 0 0 -> xyz=0 0 -1.062675918609001 rpy=0 0 0
- joint 2_3: axis 0 0 1 -> 1 0 0; origin xyz=-0.08383422666175744 0 0 rpy=0 0 0 -> xyz=-0.241642874180782 0 0 rpy=0 0 0
- joint 3_4: axis 1 1 0 -> 1 0 1; origin xyz=-0.13272853285309316 0 0 rpy=0 0 0 -> xyz=-0.9170572438288018 0 0 rpy=0 0 0
- joint 4_5: axis 1 1 1 -> 1 0 0; origin xyz=-0.2460201151112963 0 -0.34422184814863577 rpy=0 0 0 -> xyz=-0.4668329338666584 0 -0.16356645193066588 rpy=0 0 0
- joint 5_6: axis 0 1 1 -> 1 1 0; origin xyz=0 0 -1.7272926979869319 rpy=0 0 0 -> xyz=0 0 -1.1505349552261221 rpy=0 0 0
- joint 6_7: axis 0 1 1 -> 1 0 1; origin xyz=0 0 -0.28996515310602805 rpy=0 0 0 -> xyz=0 0 -1.378865732156263 rpy=0 0 0
- joint 8_9: axis 0 1 0 -> 0 0 1; origin xyz=0.19424471719395509 0 0 rpy=0 0 0 -> xyz=0.046925375028527894 0 0 rpy=0 0 0
- joint 9_10: axis 0 1 0 -> 1 1 1; origin xyz=0.9245880583558892 0 0 rpy=0 0 0 -> xyz=0.5242017776939347 0 0 rpy=0 0 0

File: body6.urdf (robot description, URDF)
Before this commit: robot robot, 33 links, 32 joints
Links:
- link 1: geometry collision box size=0.20134852055804708 0.1814426291724358 0.20900695043812156; visual box size=0.20134852055804708 0.1814426291724358 0.20900695043812156
- link 10: geometry collision box size=0.3883716563585472 0.6785734679587557 0.3780427935799904; visual box size=0.3883716563585472 0.6785734679587557 0.3780427935799904
- link 11: geometry collision box size=0.34888122834129365 0.9994540962389482 0.014849367879184117; visual box size=0.34888122834129365 0.9994540962389482 0.014849367879184117
- link 12: geometry collision box size=0.8508769530003906 0.2338848180537414 0.6541175373032173; visual box size=0.8508769530003906 0.2338848180537414 0.6541175373032173
- link 13: geometry collision box size=0.8940446004101473 0.5125298427425552 0.24909207008464862; visual box size=0.8940446004101473 0.5125298427425552 0.24909207008464862
- link 14: geometry collision box size=0.823131078074701 0.8632190124574197 0.424681183732276; visual box size=0.823131078074701 0.8632190124574197 0.424681183732276
- link 15: geometry collision box size=0.7035197859044728 0.8618995981850005 0.6162505269575013; visual box size=0.7035197859044728 0.8618995981850005 0.6162505269575013
- link 16: geometry collision box size=0.49143745604950506 0.3600375050690735 1.5590682893102228; visual box size=0.49143745604950506 0.3600375050690735 1.5590682893102228
- link 17: geometry collision box size=0.07554191946740785 0.07589994959174662 0.46754118078079276; visual box size=0.07554191946740785 0.07589994959174662 0.46754118078079276
- link 18: geometry collision box size=0.8583988311058134 0.4962702790839162 0.5130359724470838; visual box size=0.8583988311058134 0.4962702790839162 0.5130359724470838
- link 19: geometry collision box size=0.5108558546471919 0.24788825612704135 0.025268908397556356; visual box size=0.5108558546471919 0.24788825612704135 0.025268908397556356
- link 2: geometry collision box size=0.7921538948203293 0.6420838014584539 0.16198083329050927; visual box size=0.7921538948203293 0.6420838014584539 0.16198083329050927
- link 20: geometry collision box size=0.8991315085416643 0.35898514332167053 0.932965187251653; visual box size=0.8991315085416643 0.35898514332167053 0.932965187251653
- link 21: geometry collision box size=0.8268221160289662 0.9375577658025762 0.8154649050808619; visual box size=0.8268221160289662 0.9375577658025762 0.8154649050808619
- link 22: geometry collision box size=0.7760370645324868 0.7905184788168479 2.4362543938597443; visual box size=0.7760370645324868 0.7905184788168479 2.4362543938597443
- link 23: geometry collision box size=0.1394028313812602 0.08667324992868541 0.15832779373618605; visual box size=0.1394028313812602 0.08667324992868541 0.15832779373618605
- link 24: geometry collision box size=0.8913597320759411 0.7854824337772565 0.005417812404069744; visual box size=0.8913597320759411 0.7854824337772565 0.005417812404069744
- link 25: geometry collision box size=0.5550265040616928 0.7853686942928727 0.06468391585710276; visual box size=0.5550265040616928 0.7853686942928727 0.06468391585710276
- link 26: geometry collision box size=0.7203020221938802 0.6184093137668258 0.5001304708335623; visual box size=0.7203020221938802 0.6184093137668258 0.5001304708335623
- link 27: geometry collision box size=0.49416330722827984 0.8642715226494239 0.6123024524307751; visual box size=0.49416330722827984 0.8642715226494239 0.6123024524307751
- link 28: geometry collision box size=0.7428611781276151 0.8950689416694813 0.4973537333815782; visual box size=0.7428611781276151 0.8950689416694813 0.4973537333815782
- link 29: geometry collision box size=0.782441164930626 0.3535120381908061 0.0845302191116083; visual box size=0.782441164930626 0.3535120381908061 0.0845302191116083
- link 3: geometry collision box size=0.896720344461185 0.48062430848115134 0.2959340223809185; visual box size=0.896720344461185 0.48062430848115134 0.2959340223809185
- link 30: geometry collision box size=0.5740953546447584 0.6999002061333817 0.9260664662434056; visual box size=0.5740953546447584 0.6999002061333817 0.9260664662434056
- link 31: geometry collision box size=0.8795237919811246 0.005414987959982298 0.43929866669973894; visual box size=0.8795237919811246 0.005414987959982298 0.43929866669973894
- link 32: geometry collision box size=0.07087879104273032 0.8416694439407513 1.2346348670568554; visual box size=0.07087879104273032 0.8416694439407513 1.2346348670568554
- link 4: geometry collision box size=0.21374345235409042 0.5441633912744078 0.9266341373353666; visual box size=0.21374345235409042 0.5441633912744078 0.9266341373353666
- link 5: geometry collision box size=0.579734463702439 0.6266904120294247 0.34143645894626407; visual box size=0.579734463702439 0.6266904120294247 0.34143645894626407
- link 6: geometry collision box size=0.4398965749234812 0.5547266081305897 2.3020732305992104; visual box size=0.4398965749234812 0.5547266081305897 2.3020732305992104
- link 7: geometry collision box size=0.9752948909075118 0.8420084017010393 0.29724515322025613; visual box size=0.9752948909075118 0.8420084017010393 0.29724515322025613
- link 8: geometry collision box size=0.8495450489986461 0.3607181146572699 0.0006816161805335286; visual box size=0.8495450489986461 0.3607181146572699 0.0006816161805335286
- link 9: geometry collision box size=0.5394143470394129 0.03282734277563293 0.5970342671370398; visual box size=0.5394143470394129 0.03282734277563293 0.5970342671370398
Joints:
- joint 0_1: axis 1 0 0 -> 0 1 1
- joint 0_25: axis 0 0 1 -> 0 1 1
- joint 0_9: axis 0 1 0 -> 0 0 1
- joint 10_11: origin xyz=0.41810953375164617 0 0 rpy=0 0 0 -> xyz=0.3883716563585472 0 0 rpy=0 0 0
- joint 11_12: axis 0 0 1 -> 1 0 0; origin xyz=0.7875329673919859 0 0 rpy=0 0 0 -> xyz=0.34888122834129365 0 0 rpy=0 0 0
- joint 12_13: axis 0 0 1 -> 1 1 1; origin xyz=0.7176643456261216 0 0 rpy=0 0 0 -> xyz=0.8508769530003906 0 0 rpy=0 0 0
- joint 13_14: axis 0 0 1 -> 1 1 1; origin xyz=0.40014611285024954 0 -0.11018258565837374 rpy=0 0 0 -> xyz=0.44702230020507366 0 -0.12454603504232431 rpy=0 0 0
- joint 14_15: axis 0 0 1 -> 1 0 0; origin xyz=0 0 -0.296139181643083 rpy=0 0 0 -> xyz=0 0 -0.424681183732276 rpy=0 0 0
- joint 15_16: axis 0 1 0 -> 1 1 1; origin xyz=0 0 -1.4345875419381076 rpy=0 0 0 -> xyz=0 0 -0.6162505269575013 rpy=0 0 0
- joint 17_18: axis 1 0 1 -> 0 0 1; origin xyz=0 -0.8787428406614863 0 rpy=0 0 0 -> xyz=0 -0.07589994959174662 0 rpy=0 0 0
- joint 18_19: axis 1 0 1 -> 0 0 1; origin xyz=0 -0.6521552621309835 0 rpy=0 0 0 -> xyz=0 -0.4962702790839162 0 rpy=0 0 0
- joint 19_20: axis 1 1 1 -> 1 0 0; origin xyz=0 -0.7848759079583053 0 rpy=0 0 0 -> xyz=0 -0.24788825612704135 0 rpy=0 0 0
- joint 1_2: axis 0 0 1 -> 1 0 0; origin xyz=-0.43220764212190965 0 0 rpy=0 0 0 -> xyz=-0.20134852055804708 0 0 rpy=0 0 0
- joint 20_21: axis 0 1 1 -> 0 0 1; origin xyz=0 -0.23649737038625807 0 rpy=0 0 0 -> xyz=0 -0.35898514332167053 0 rpy=0 0 0
- joint 21_22: axis 1 0 1 -> 0 1 1; origin xyz=0 -0.23835520012367806 -0.31246967842499485 rpy=0 0 0 -> xyz=0 -0.4687788829012881 -0.40773245254043095 rpy=0 0 0
- joint 22_23: axis 0 1 0 -> 1 1 0; origin xyz=0 0 -2.3035050631701286 rpy=0 0 0 -> xyz=0 0 -2.4362543938597443 rpy=0 0 0
- joint 23_24: origin xyz=0 0 -0.011479431907093803 rpy=0 0 0 -> xyz=0 0 -0.15832779373618605 rpy=0 0 0
- joint 25_26: origin xyz=0 0.7627912018801261 0 rpy=0 0 0 -> xyz=0 0.7853686942928727 0 rpy=0 0 0
- joint 26_27: origin xyz=0 0.24403427287626667 0 rpy=0 0 0 -> xyz=0 0.6184093137668258 0 rpy=0 0 0
- joint 27_28: axis 0 0 1 -> 1 0 0; origin xyz=0 0.7635139107611487 0 rpy=0 0 0 -> xyz=0 0.8642715226494239 0 rpy=0 0 0
- joint 28_29: axis 1 1 0 -> 0 1 0; origin xyz=0 0.5850114940406189 0 rpy=0 0 0 -> xyz=0 0.8950689416694813 0 rpy=0 0 0
- joint 29_30: axis 1 0 1 -> 1 1 1; origin xyz=0 0.07082100890094101 -0.4252074637846779 rpy=0 0 0 -> xyz=0 0.17675601909540306 -0.04226510955580415 rpy=0 0 0
- joint 2_3: axis 0 1 1 -> 0 0 1; origin xyz=-0.40348664723174177 0 0 rpy=0 0 0 -> xyz=-0.7921538948203293 0 0 rpy=0 0 0
- joint 30_31: origin xyz=0 0 -1.7079937662978928 rpy=0 0 0 -> xyz=0 0 -0.9260664662434056 rpy=0 0 0
- joint 31_32: axis 0 1 1 -> 0 1 0; origin xyz=0 0 -0.5300676248275351 rpy=0 0 0 -> xyz=0 0 -0.43929866669973894 rpy=0 0 0
- joint 3_4: axis 0 0 1 -> 1 0 0; origin xyz=-0.36294652367964075 0 0 rpy=0 0 0 -> xyz=-0.896720344461185 0 0 rpy=0 0 0
- joint 4_5: axis 1 1 0 -> 0 1 0; origin xyz=-0.9739358266797544 0 0 rpy=0 0 0 -> xyz=-0.21374345235409042 0 0 rpy=0 0 0
- joint 5_6: origin xyz=-0.21918941248203078 0 -0.03738749471064623 rpy=0 0 0 -> xyz=-0.2898672318512195 0 -0.17071822947313203 rpy=0 0 0
- joint 6_7: origin xyz=0 0 -1.8950221001781495 rpy=0 0 0 -> xyz=0 0 -2.3020732305992104 rpy=0 0 0
- joint 7_8: axis 0 1 1 -> 1 0 1; origin xyz=0 0 -0.6626065343778716 rpy=0 0 0 -> xyz=0 0 -0.29724515322025613 rpy=0 0 0
- joint 9_10: axis 1 0 1 -> 0 0 1; origin xyz=0.7327813769181848 0 0 rpy=0 0 0 -> xyz=0.5394143470394129 0 0 rpy=0 0 0
