Commit message: commit

File: body/body0.urdf (robot description, URDF)
Before this commit: robot robot, 39 links, 38 joints
Links:
- removed link 27
- removed link 28
- removed link 29
- removed link 30
- removed link 31
- removed link 32
- removed link 33
- removed link 34
- removed link 35
- removed link 36
- removed link 37
- removed link 38
- link 0: geometry collision box size=1.1326980480365167 1.4604549598621603 1.1495911874822367; visual box size=1.1326980480365167 1.4604549598621603 1.1495911874822367
- link 1: geometry collision box size=0.5911259352917371 0.93332310756875 1.1546349067615251; visual box size=0.5911259352917371 0.93332310756875 1.1546349067615251
- link 10: geometry collision box size=0.7635033992783462 1.3827190622329821 1.0642709630404854; visual box size=0.7635033992783462 1.3827190622329821 1.0642709630404854
- link 11: geometry collision box size=1.0574213304665299 0.8551611559298903 1.115083346786908; visual box size=1.0574213304665299 0.8551611559298903 1.115083346786908
- link 12: geometry collision box size=0.829068430584603 0.6428400092144579 0.7835193521262026; visual box size=0.829068430584603 0.6428400092144579 0.7835193521262026
- link 13: geometry collision box size=1.2046313309067815 0.5812111056891005 0.8992384827270729; visual box size=1.2046313309067815 0.5812111056891005 0.8992384827270729
- link 14: geometry collision box size=0.778172343506375 0.7320999421780046 1.7950366516683145; visual box size=0.778172343506375 0.7320999421780046 1.7950366516683145
- link 15: geometry collision box size=1.3265971836774668 0.5605587373040567 0.7913725864850975; visual box size=1.3265971836774668 0.5605587373040567 0.7913725864850975
- link 16: geometry collision box size=1.4092728941929897 0.5099584604675457 0.6809578837153264; visual box size=1.4092728941929897 0.5099584604675457 0.6809578837153264
- link 17: geometry collision box size=1.2160606340076694 0.7394525247010831 1.1725201044624094; visual box size=1.2160606340076694 0.7394525247010831 1.1725201044624094
- link 18: geometry collision box size=0.6216721361291382 1.4642851682008016 0.9701126012494025; visual box size=0.6216721361291382 1.4642851682008016 0.9701126012494025
- link 19: geometry collision box size=1.167526444648923 1.159766697637377 1.839130203001311; visual box size=1.167526444648923 1.159766697637377 1.839130203001311
- link 2: geometry collision box size=1.3286190087756724 1.4059184572649839 1.04441102695682; visual box size=1.3286190087756724 1.4059184572649839 1.04441102695682
- link 20: geometry collision box size=0.8026009358023456 0.7526912027271038 0.6685516822708764; visual box size=0.8026009358023456 0.7526912027271038 0.6685516822708764
- link 21: geometry collision box size=0.6724279479213507 1.3935405576710236 1.1656562653065912; visual box size=0.6724279479213507 1.3935405576710236 1.1656562653065912
- link 22: geometry collision box size=0.7846587068831593 0.5539739341090149 1.1078542577819295; visual box size=0.7846587068831593 0.5539739341090149 1.1078542577819295
- link 23: geometry collision box size=0.9041705824829385 1.1592287545407467 0.6886321241301319; visual box size=0.9041705824829385 1.1592287545407467 0.6886321241301319
- link 24: geometry collision box size=1.3365971486120785 1.3376933898447572 1.2362173555781921; visual box size=1.3365971486120785 1.3376933898447572 1.2362173555781921
- link 25: geometry collision box size=1.4275883092922914 0.8891611157166175 1.867609369237662; visual box size=1.4275883092922914 0.8891611157166175 1.867609369237662
- link 26: geometry collision box size=0.7975523548865062 1.071846529039648 0.37396776170573576; visual box size=0.7975523548865062 1.071846529039648 0.37396776170573576
- link 3: geometry collision box size=1.1620374803533982 1.1086674788919435 1.2058734965409381; visual box size=1.1620374803533982 1.1086674788919435 1.2058734965409381
- link 4: geometry collision box size=1.408037145829054 1.1732307412450127 1.2074376323574185; visual box size=1.408037145829054 1.1732307412450127 1.2074376323574185
- link 5: geometry collision box size=1.120438156610029 0.6831308725192868 1.348344003166277; visual box size=1.120438156610029 0.6831308725192868 1.348344003166277
- link 6: geometry collision box size=1.4949694912236156 1.419974158450127 2.5507929610627103; visual box size=1.4949694912236156 1.419974158450127 2.5507929610627103
- link 7: geometry collision box size=0.9027715433791239 0.8444339806212192 0.8974461687060703; visual box size=0.9027715433791239 0.8444339806212192 0.8974461687060703
- link 8: geometry collision box size=1.4968817671085364 0.7405856803217158 0.029555356752809403; visual box size=1.4968817671085364 0.7405856803217158 0.029555356752809403
- link 9: geometry collision box size=1.0796173862915888 1.457618555750209 1.4117860542917207; visual box size=1.0796173862915888 1.457618555750209 1.4117860542917207
Joints:
- removed joint 14_15
- removed joint 26_27
- removed joint 27_28
- removed joint 28_29
- removed joint 2_12
- removed joint 2_30
- removed joint 30_31
- removed joint 31_32
- removed joint 32_33
- removed joint 33_34
- removed joint 34_35
- removed joint 35_36
- removed joint 36_37
- removed joint 37_38
- removed joint 8_9
- added joint 11_12: type revolute, parent 11, child 12, origin xyz=0.5287106652332649 0 0 rpy=0 0 0, axis 1 0 0, limit lower=-3.14159 upper=3.14159 effort=0.0 velocity=0.0
- added joint 2_15: type revolute, parent 2, child 15, origin xyz=0 -0.7029592286324919 0 rpy=0 0 0, axis 1 0 0, limit lower=-3.14159 upper=3.14159 effort=0.0 velocity=0.0
- added joint 2_9: type revolute, parent 2, child 9, origin xyz=0.6643095043878362 0 0 rpy=0 0 0, axis 1 0 0, limit lower=-3.14159 upper=3.14159 effort=0.0 velocity=0.0
- joint 0_1: origin xyz=0 0 0.6281807429604901 rpy=0 0 0 -> xyz=0 0 1.1495911874822367 rpy=0 0 0
- joint 10_11: axis 0 1 0 -> 1 1 0; origin xyz=0 0 -0.07627990541991282 rpy=0 0 0 -> xyz=0.7635033992783462 0 0 rpy=0 0 0
- joint 12_13: origin xyz=1.186283673654179 0 0 rpy=0 0 0 -> xyz=0 0 -0.7835193521262026 rpy=0 0 0
- joint 13_14: axis 0 0 1 -> 0 1 0; origin xyz=0.6285258973016234 0 0 rpy=0 0 0 -> xyz=0 0 -0.8992384827270729 rpy=0 0 0
- joint 15_16: axis 0 0 1 -> 0 1 1; origin xyz=0.8176243475488892 0 0 rpy=0 0 0 -> xyz=0 -0.5605587373040567 0 rpy=0 0 0
- joint 16_17: axis 0 0 1 -> 1 1 0; origin xyz=0.5859389580484464 0 0 rpy=0 0 0 -> xyz=0 -0.5099584604675457 0 rpy=0 0 0
- joint 17_18: axis 0 1 1 -> 1 0 0; origin xyz=0.7349621797575796 0 0 rpy=0 0 0 -> xyz=0 -0.36972626235054157 0 rpy=0 0 0
- joint 18_19: axis 1 0 1 -> 1 1 1; origin xyz=0 0 -0.5811988241624679 rpy=0 0 0 -> xyz=0 0 -0.9701126012494025 rpy=0 0 0
- joint 19_20: axis 0 1 0 -> 1 1 1; origin xyz=0 0 -1.1924699661445908 rpy=0 0 0 -> xyz=0 0 -1.839130203001311 rpy=0 0 0
- joint 1_2: axis 0 0 1 -> 1 0 1; origin xyz=0 0 1.3261119645548214 rpy=0 0 0 -> xyz=0 0 1.1546349067615251 rpy=0 0 0
- joint 21_22: origin xyz=0 -1.29804181633593 0 rpy=0 0 0 -> xyz=0 1.3935405576710236 0 rpy=0 0 0
- joint 22_23: axis 1 1 0 -> 0 1 0; origin xyz=0 -0.8628400347522525 0 rpy=0 0 0 -> xyz=0 0.5539739341090149 0 rpy=0 0 0
- joint 23_24: axis 1 0 0 -> 0 1 0; origin xyz=0 -0.74117455622991 0 rpy=0 0 0 -> xyz=0 0.5796143772703733 0 rpy=0 0 0
- joint 24_25: axis 1 0 1 -> 0 0 1; origin xyz=0 -1.3943935364916855 0 rpy=0 0 0 -> xyz=0 0 -1.2362173555781921 rpy=0 0 0
- joint 25_26: origin xyz=0 -0.9044585174072277 0 rpy=0 0 0 -> xyz=0 0 -1.867609369237662 rpy=0 0 0
- joint 2_21: axis 0 0 1 -> 1 0 1; origin xyz=0 -0.3254424698448381 0 rpy=0 0 0 -> xyz=0 0.7029592286324919 0 rpy=0 0 0
- joint 2_3: axis 0 0 1 -> 1 1 1; origin xyz=-0.46419112679645613 0 0 rpy=0 0 0 -> xyz=-0.6643095043878362 0 0 rpy=0 0 0
- joint 3_4: axis 0 1 1 -> 1 1 0; origin xyz=-0.9373517628276159 0 0 rpy=0 0 0 -> xyz=-1.1620374803533982 0 0 rpy=0 0 0
- joint 4_5: origin xyz=-1.3703454797555845 0 0 rpy=0 0 0 -> xyz=-1.408037145829054 0 0 rpy=0 0 0
- joint 5_6: axis 1 0 1 -> 0 1 0; origin xyz=-1.0218304350042478 0 0 rpy=0 0 0 -> xyz=-0.5602190783050145 0 0 rpy=0 0 0
- joint 6_7: axis 1 0 1 -> 0 1 1; origin xyz=-0.8638738895624946 0 0 rpy=0 0 0 -> xyz=0 0 -2.5507929610627103 rpy=0 0 0
- joint 7_8: axis 0 0 1 -> 1 0 0; origin xyz=-0.618592816775417 0 0 rpy=0 0 0 -> xyz=0 0 -0.8974461687060703 rpy=0 0 0
- joint 9_10: axis 0 1 1 -> 0 0 1; origin xyz=0 0 -2.0953086686429048 rpy=0 0 0 -> xyz=1.0796173862915888 0 0 rpy=0 0 0

Commit message: commit

File: body/body0.urdf (robot description, URDF)
Before this commit: robot robot, 33 links, 32 joints
Links:
- removed link 29
- removed link 30
- removed link 31
- removed link 32
- link 1: geometry collision box size=0.46816235906027015 0.20167082001915182 0.9753088394571031; visual box size=0.46816235906027015 0.20167082001915182 0.9753088394571031
- link 10: geometry collision box size=0.2929497695050721 0.7674109683458304 0.6340332790917258; visual box size=0.2929497695050721 0.7674109683458304 0.6340332790917258
- link 11: geometry collision box size=0.5589976723575089 0.5527732802351987 0.8886108068096893; visual box size=0.5589976723575089 0.5527732802351987 0.8886108068096893
- link 12: geometry collision box size=0.9830484417910529 0.6527085628149256 2.8714384976835245; visual box size=0.9830484417910529 0.6527085628149256 2.8714384976835245
- link 13: geometry collision box size=0.6250234513002859 0.3360361725592593 0.3833161818209701; visual box size=0.6250234513002859 0.3360361725592593 0.3833161818209701
- link 14: geometry collision box size=0.40981755459337843 0.6836179745577944 0.34524532049550544; visual box size=0.40981755459337843 0.6836179745577944 0.34524532049550544
- link 15: geometry collision box size=0.5595238457498594 0.35383836315199035 0.5095887407748433; visual box size=0.5595238457498594 0.35383836315199035 0.5095887407748433
- link 16: geometry collision box size=0.910164372203179 0.8692218119672526 0.588487428883142; visual box size=0.910164372203179 0.8692218119672526 0.588487428883142
- link 17: geometry collision box size=0.76081710388661 0.6932940520813832 0.4141886650697001; visual box size=0.76081710388661 0.6932940520813832 0.4141886650697001
- link 18: geometry collision box size=0.14022566661570324 0.5906878374769473 0.8219655429908778; visual box size=0.14022566661570324 0.5906878374769473 0.8219655429908778
- link 19: geometry collision box size=0.6445479571076548 0.17948652122802333 2.8763203704033726; visual box size=0.6445479571076548 0.17948652122802333 2.8763203704033726
- link 2: geometry collision box size=0.46683019196946884 0.8146151791041796 0.36140418108844274; visual box size=0.46683019196946884 0.8146151791041796 0.36140418108844274
- link 20: geometry collision box size=0.3107597639657864 0.3080878642713498 0.1685681497159743; visual box size=0.3107597639657864 0.3080878642713498 0.1685681497159743
- link 21: geometry collision box size=0.559311006111609 0.08256749706565303 0.5551114798806531; visual box size=0.559311006111609 0.08256749706565303 0.5551114798806531
- link 22: geometry collision box size=0.9286777387693409 0.31933485727963384 0.6396505951736504; visual box size=0.9286777387693409 0.31933485727963384 0.6396505951736504
- link 23: geometry collision box size=0.7015293127570502 0.7274319148047473 0.22210302647981073; visual box size=0.7015293127570502 0.7274319148047473 0.22210302647981073
- link 24: geometry collision box size=0.5951039584639463 0.8812596387934295 0.37912995756117074; visual box size=0.5951039584639463 0.8812596387934295 0.37912995756117074
- link 25: geometry collision box size=0.7520978204596142 0.5820507490331495 0.9228163946963437; visual box size=0.7520978204596142 0.5820507490331495 0.9228163946963437
- link 26: geometry collision box size=0.6499189337334399 0.3383079551499928 3.5942675101520916; visual box size=0.6499189337334399 0.3383079551499928 3.5942675101520916
- link 27: geometry collision box size=0.42160448597611244 0.7481946008190965 0.002473337149124653; visual box size=0.42160448597611244 0.7481946008190965 0.002473337149124653
- link 28: geometry collision box size=0.7964780211569602 0.7653690539265703 0.0032591526987838754; visual box size=0.7964780211569602 0.7653690539265703 0.0032591526987838754
- link 3: geometry collision box size=0.8490933337254969 0.188251563736187 0.29349405373439486; visual box size=0.8490933337254969 0.188251563736187 0.29349405373439486
- link 4: geometry collision box size=0.9333510285691292 0.8086959839070829 0.7187542660790924; visual box size=0.9333510285691292 0.8086959839070829 0.7187542660790924
- link 5: geometry collision box size=0.5860768613264882 0.3356455162103291 1.0891264080854164; visual box size=0.5860768613264882 0.3356455162103291 1.0891264080854164
- link 6: geometry collision box size=0.9658629429148562 0.27832181301174175 2.118728822107539; visual box size=0.9658629429148562 0.27832181301174175 2.118728822107539
- link 7: geometry collision box size=0.8164287426857211 0.34004311862037473 0.3921447698070448; visual box size=0.8164287426857211 0.34004311862037473 0.3921447698070448
- link 8: geometry collision box size=0.3181587572338288 0.19685571009110825 0.4528225932487221; visual box size=0.3181587572338288 0.19685571009110825 0.4528225932487221
- link 9: geometry collision box size=0.6968662017403002 0.531938161770873 0.03197453149034668; visual box size=0.6968662017403002 0.531938161770873 0.03197453149034668
Joints:
- removed joint 0_17
- removed joint 0_25
- removed joint 0_9
- removed joint 14_15
- removed joint 21_22
- removed joint 28_29
- removed joint 29_30
- removed joint 30_31
- removed joint 31_32
- removed joint 7_8
- added joint 0_15: type revolute, parent 0, child 15, origin xyz=0 -0.75 4 rpy=0 0 0, axis 1 0 0, limit lower=-3.14159 upper=3.14159 effort=0.0 velocity=0.0
- added joint 0_22: type revolute, parent 0, child 22, origin xyz=0 0.75 4 rpy=0 0 0, axis 1 0 0, limit lower=-3.14159 upper=3.14159 effort=0.0 velocity=0.0
- added joint 0_8: type revolute, parent 0, child 8, origin xyz=0.75 0 4 rpy=0 0 0, axis 0 0 1, limit lower=-3.14159 upper=3.14159 effort=0.0 velocity=0.0
- added joint 16_17: type revolute, parent 16, child 17, origin xyz=0 -0.8692218119672526 0 rpy=0 0 0, axis 0 0 1, limit lower=-3.14159 upper=3.14159 effort=0.0 velocity=0.0
- added joint 24_25: type revolute, parent 24, child 25, origin xyz=0 0.8812596387934295 0 rpy=0 0 0, axis 1 1 0, limit lower=-3.14159 upper=3.14159 effort=0.0 velocity=0.0
- added joint 8_9: type revolute, parent 8, child 9, origin xyz=0.3181587572338288 0 0 rpy=0 0 0, axis 1 0 0, limit lower=-3.14159 upper=3.14159 effort=0.0 velocity=0.0
- joint 0_1: origin xyz=-0.75 0 1 rpy=0 0 0 -> xyz=-0.75 0 4 rpy=0 0 0
- joint 10_11: axis 0 0 1 -> 0 1 1; origin xyz=0.3646006235644291 0 0 rpy=0 0 0 -> xyz=0.2929497695050721 0 0 rpy=0 0 0
- joint 11_12: axis 1 0 0 -> 0 1 1; origin xyz=0.04463733385183821 0 0 rpy=0 0 0 -> xyz=0.27949883617875443 0 -0.44430540340484465 rpy=0 0 0
- joint 12_13: axis 1 0 1 -> 1 1 0; origin xyz=0.11224885597541623 0 0 rpy=0 0 0 -> xyz=0 0 -2.8714384976835245 rpy=0 0 0
- joint 13_14: axis 1 1 0 -> 1 0 0; origin xyz=0.25792599174839065 0 -0.455051457876974 rpy=0 0 0 -> xyz=0 0 -0.3833161818209701 rpy=0 0 0
- joint 15_16: axis 1 1 0 -> 0 0 1; origin xyz=0 0 -0.19506814336396583 rpy=0 0 0 -> xyz=0 -0.35383836315199035 0 rpy=0 0 0
- joint 17_18: axis 0 1 0 -> 0 0 1; origin xyz=0 -0.684973864093664 0 rpy=0 0 0 -> xyz=0 -0.6932940520813832 0 rpy=0 0 0
- joint 18_19: axis 1 0 1 -> 0 1 0; origin xyz=0 -0.11833273397104538 0 rpy=0 0 0 -> xyz=0 -0.29534391873847365 -0.4109827714954389 rpy=0 0 0
- joint 19_20: axis 1 0 1 -> 0 1 1; origin xyz=0 -0.8904141081756023 0 rpy=0 0 0 -> xyz=0 0 -2.8763203704033726 rpy=0 0 0
- joint 1_2: axis 1 0 0 -> 0 1 0; origin xyz=-0.06959089762238424 0 0 rpy=0 0 0 -> xyz=-0.46816235906027015 0 0 rpy=0 0 0
- joint 20_21: axis 1 1 0 -> 0 1 0; origin xyz=0 -0.30327893202892553 0 rpy=0 0 0 -> xyz=0 0 -0.1685681497159743 rpy=0 0 0
- joint 22_23: axis 1 0 1 -> 1 1 1; origin xyz=0 0 -0.35620507808403906 rpy=0 0 0 -> xyz=0 0.31933485727963384 0 rpy=0 0 0
- joint 23_24: axis 1 1 1 -> 1 1 0; origin xyz=0 0 -0.12538039352635452 rpy=0 0 0 -> xyz=0 0.7274319148047473 0 rpy=0 0 0
- joint 25_26: axis 1 0 0 -> 0 1 1; origin xyz=0 0.5927561764984922 0 rpy=0 0 0 -> xyz=0 0.29102537451657473 -0.46140819734817184 rpy=0 0 0
- joint 26_27: axis 0 1 0 -> 1 1 1; origin xyz=0 0.07206797701673684 0 rpy=0 0 0 -> xyz=0 0 -3.5942675101520916 rpy=0 0 0
- joint 27_28: origin xyz=0 0.754418290620009 0 rpy=0 0 0 -> xyz=0 0 -0.002473337149124653 rpy=0 0 0
- joint 2_3: origin xyz=-0.2668410073120002 0 0 rpy=0 0 0 -> xyz=-0.46683019196946884 0 0 rpy=0 0 0
- joint 3_4: axis 0 0 1 -> 1 0 0; origin xyz=-0.76780578184084 0 0 rpy=0 0 0 -> xyz=-0.8490933337254969 0 0 rpy=0 0 0
- joint 4_5: axis 1 0 1 -> 1 0 0; origin xyz=-0.8902624474507072 0 0 rpy=0 0 0 -> xyz=-0.4666755142845646 0 -0.3593771330395462 rpy=0 0 0
- joint 5_6: axis 1 0 0 -> 0 1 1; origin xyz=-0.38279228418557915 0 -0.10662676882532696 rpy=0 0 0 -> xyz=0 0 -1.0891264080854164 rpy=0 0 0
- joint 6_7: axis 1 0 1 -> 0 1 1; origin xyz=0 0 -0.4633372114674241 rpy=0 0 0 -> xyz=0 0 -2.118728822107539 rpy=0 0 0
- joint 9_10: axis 1 0 1 -> 0 0 1; origin xyz=0.6761609173842691 0 0 rpy=0 0 0 -> xyz=0.6968662017403002 0 0 rpy=0 0 0
