Commit message: new robot

File: body/body0.urdf (robot description, URDF)
Before this commit: robot robot, 33 links, 32 joints
Links:
- removed link 10
- removed link 11
- removed link 12
- removed link 13
- removed link 14
- removed link 15
- removed link 16
- removed link 17
- removed link 18
- removed link 19
- removed link 20
- removed link 21
- removed link 22
- removed link 23
- removed link 24
- removed link 25
- removed link 26
- removed link 27
- removed link 28
- removed link 29
- removed link 30
- removed link 31
- removed link 32
- removed link 6
- removed link 7
- removed link 8
- removed link 9
- link 0: geometry collision box size=1 1 1; visual box size=1 1 1
- link 1: geometry collision box size=1 1 1; visual box size=1 1 1
- link 2: geometry collision box size=1 1 1; visual box size=1 1 1
- link 3: geometry collision box size=1 1 1; visual box size=1 1 1
- link 4: geometry collision box size=1 1 1; visual box size=1 1 1
- link 5: geometry collision box size=1 1 1; visual box size=1 1 1
Joints:
- removed joint 0_17
- removed joint 0_25
- removed joint 0_9
- removed joint 10_11
- removed joint 11_12
- removed joint 12_13
- removed joint 13_14
- removed joint 14_15
- removed joint 15_16
- removed joint 17_18
- removed joint 18_19
- removed joint 19_20
- removed joint 20_21
- removed joint 21_22
- removed joint 22_23
- removed joint 23_24
- removed joint 25_26
- removed joint 26_27
- removed joint 27_28
- removed joint 28_29
- removed joint 29_30
- removed joint 30_31
- removed joint 31_32
- removed joint 5_6
- removed joint 6_7
- removed joint 7_8
- removed joint 9_10
- joint 0_1: axis 0 0 1 -> 1 0 0; origin xyz=-0.75 0 3 rpy=0 0 0 -> xyz=0 0 1 rpy=0 0 0
- joint 1_2: axis 1 0 1 -> 1 1 1; origin xyz=-0.8107394240697886 0 0 rpy=0 0 0 -> xyz=0 0 0.5 rpy=0 0 0
- joint 2_3: axis 0 1 1 -> 1 0 1; origin xyz=-0.24854259989576166 0 0 rpy=0 0 0 -> xyz=0 0 0.5 rpy=0 0 0
- joint 3_4: axis 1 1 1 -> 0 1 1; origin xyz=-0.279577807566076 0 0 rpy=0 0 0 -> xyz=0 0 0.5 rpy=0 0 0
- joint 4_5: axis 1 0 1 -> 0 0 1; origin xyz=-0.5478626361291992 0 0 rpy=0 0 0 -> xyz=0 0 0.5 rpy=0 0 0

File: body/body1.urdf (robot description, URDF)
Before this commit: robot robot, 21 links, 20 joints
Links:
- removed link 10
- removed link 11
- removed link 12
- removed link 13
- removed link 14
- removed link 15
- removed link 16
- removed link 17
- removed link 18
- removed link 19
- removed link 20
- removed link 6
- removed link 7
- removed link 8
- removed link 9
- link 0: geometry collision box size=1 1 1; visual box size=1 1 1
- link 1: geometry collision box size=1 1 1; visual box size=1 1 1
- link 2: geometry collision box size=1 1 1; visual box size=1 1 1
- link 3: geometry collision box size=1 1 1; visual box size=1 1 1
- link 4: geometry collision box size=1 1 1; visual box size=1 1 1
- link 5: geometry collision box size=1 1 1; visual box size=1 1 1
Joints:
- removed joint 0_11
- removed joint 0_16
- removed joint 0_6
- removed joint 11_12
- removed joint 12_13
- removed joint 13_14
- removed joint 14_15
- removed joint 16_17
- removed joint 17_18
- removed joint 18_19
- removed joint 19_20
- removed joint 6_7
- removed joint 7_8
- removed joint 8_9
- removed joint 9_10
- joint 0_1: axis 0 0 1 -> 1 1 0; origin xyz=-0.75 0 3 rpy=0 0 0 -> xyz=0 0 1 rpy=0 0 0
- joint 1_2: origin xyz=-0.8250087508596406 0 0 rpy=0 0 0 -> xyz=0 0 0.5 rpy=0 0 0
- joint 2_3: axis 0 1 0 -> 1 1 1; origin xyz=-0.18313482726810654 0 -0.06156945542327352 rpy=0 0 0 -> xyz=0 0 0.5 rpy=0 0 0
- joint 3_4: axis 1 0 0 -> 1 1 1; origin xyz=0 0 -0.8666666666666667 rpy=0 0 0 -> xyz=0 0 0.5 rpy=0 0 0
- joint 4_5: axis 0 1 1 -> 1 0 0; origin xyz=0 0 -0.8666666666666667 rpy=0 0 0 -> xyz=0 0 0.5 rpy=0 0 0

File: body/body2.urdf (robot description, URDF)
Before this commit: robot robot, 33 links, 32 joints
Links:
- removed link 1
- removed link 10
- removed link 11
- removed link 12
- removed link 13
- removed link 14
- removed link 15
- removed link 16
- removed link 17
- removed link 18
- removed link 19
- removed link 2
- removed link 20
- removed link 21
- removed link 22
- removed link 23
- removed link 24
- removed link 25
- removed link 26
- removed link 27
- removed link 28
- removed link 29
- removed link 3
- removed link 30
- removed link 31
- removed link 32
- removed link 4
- removed link 5
- removed link 6
- removed link 7
- removed link 8
- removed link 9
- link 0: geometry collision box size=1 1 1; visual box size=1 1 1
Joints:
- removed joint 0_1
- removed joint 0_17
- removed joint 0_25
- removed joint 0_9
- removed joint 10_11
- removed joint 11_12
- removed joint 12_13
- removed joint 13_14
- removed joint 14_15
- removed joint 15_16
- removed joint 17_18
- removed joint 18_19
- removed joint 19_20
- removed joint 1_2
- removed joint 20_21
- removed joint 21_22
- removed joint 22_23
- removed joint 23_24
- removed joint 25_26
- removed joint 26_27
- removed joint 27_28
- removed joint 28_29
- removed joint 29_30
- removed joint 2_3
- removed joint 30_31
- removed joint 31_32
- removed joint 3_4
- removed joint 4_5
- removed joint 5_6
- removed joint 6_7
- removed joint 7_8
- removed joint 9_10

File: body/body3.urdf (robot description, URDF)
Before this commit: robot robot, 33 links, 32 joints
Links:
- removed link 10
- removed link 11
- removed link 12
- removed link 13
- removed link 14
- removed link 15
- removed link 16
- removed link 17
- removed link 18
- removed link 19
- removed link 20
- removed link 21
- removed link 22
- removed link 23
- removed link 24
- removed link 25
- removed link 26
- removed link 27
- removed link 28
- removed link 29
- removed link 30
- removed link 31
- removed link 32
- removed link 7
- removed link 8
- removed link 9
- link 0: geometry collision box size=1 1 1; visual box size=1 1 1
- link 1: geometry collision box size=1 1 1; visual box size=1 1 1
- link 2: geometry collision box size=1 1 1; visual box size=1 1 1
- link 3: geometry collision box size=1 1 1; visual box size=1 1 1
- link 4: geometry collision box size=1 1 1; visual box size=1 1 1
- link 5: geometry collision box size=1 1 1; visual box size=1 1 1
- link 6: geometry collision box size=1 1 1; visual box size=1 1 1
Joints:
- removed joint 0_17
- removed joint 0_25
- removed joint 0_9
- removed joint 10_11
- removed joint 11_12
- removed joint 12_13
- removed joint 13_14
- removed joint 14_15
- removed joint 15_16
- removed joint 17_18
- removed joint 18_19
- removed joint 19_20
- removed joint 20_21
- removed joint 21_22
- removed joint 22_23
- removed joint 23_24
- removed joint 25_26
- removed joint 26_27
- removed joint 27_28
- removed joint 28_29
- removed joint 29_30
- removed joint 30_31
- removed joint 31_32
- removed joint 6_7
- removed joint 7_8
- removed joint 9_10
- joint 0_1: axis 1 0 0 -> 1 1 1; origin xyz=-0.75 0 3 rpy=0 0 0 -> xyz=0 0 1 rpy=0 0 0
- joint 1_2: axis 0 0 1 -> 0 1 0; origin xyz=-0.3758210655284704 0 0 rpy=0 0 0 -> xyz=0 0 0.5 rpy=0 0 0
- joint 2_3: axis 1 0 1 -> 0 1 0; origin xyz=-0.2846391621508364 0 0 rpy=0 0 0 -> xyz=0 0 0.5 rpy=0 0 0
- joint 3_4: axis 1 1 1 -> 1 0 0; origin xyz=-0.2796975766972919 0 0 rpy=0 0 0 -> xyz=0 0 0.5 rpy=0 0 0
- joint 4_5: axis 0 0 1 -> 0 1 1; origin xyz=-0.2102107280634422 0 0 rpy=0 0 0 -> xyz=0 0 0.5 rpy=0 0 0
- joint 5_6: axis 1 0 1 -> 0 0 1; origin xyz=-0.3065282276362638 0 -0.4533725198534372 rpy=0 0 0 -> xyz=0 0 0.5 rpy=0 0 0

File: body/body4.urdf (robot description, URDF)
Before this commit: robot robot, 25 links, 24 joints
Links:
- removed link 10
- removed link 11
- removed link 12
- removed link 13
- removed link 14
- removed link 15
- removed link 16
- removed link 17
- removed link 18
- removed link 19
- removed link 20
- removed link 21
- removed link 22
- removed link 23
- removed link 24
- removed link 6
- removed link 7
- removed link 8
- removed link 9
- link 0: geometry collision box size=1 1 1; visual box size=1 1 1
- link 1: geometry collision box size=1 1 1; visual box size=1 1 1
- link 2: geometry collision box size=1 1 1; visual box size=1 1 1
- link 3: geometry collision box size=1 1 1; visual box size=1 1 1
- link 4: geometry collision box size=1 1 1; visual box size=1 1 1
- link 5: geometry collision box size=1 1 1; visual box size=1 1 1
Joints:
- removed joint 0_13
- removed joint 0_19
- removed joint 0_7
- removed joint 10_11
- removed joint 11_12
- removed joint 13_14
- removed joint 14_15
- removed joint 15_16
- removed joint 16_17
- removed joint 17_18
- removed joint 19_20
- removed joint 20_21
- removed joint 21_22
- removed joint 22_23
- removed joint 23_24
- removed joint 5_6
- removed joint 7_8
- removed joint 8_9
- removed joint 9_10
- joint 0_1: axis 1 0 1 -> 1 0 0; origin xyz=-0.75 0 3 rpy=0 0 0 -> xyz=0 0 1 rpy=0 0 0
- joint 1_2: axis 1 1 1 -> 1 0 1; origin xyz=-0.06701426826088874 0 0 rpy=0 0 0 -> xyz=0 0 0.5 rpy=0 0 0
- joint 2_3: axis 1 0 0 -> 1 0 1; origin xyz=-0.7676011936736991 0 0 rpy=0 0 0 -> xyz=0 0 0.5 rpy=0 0 0
- joint 3_4: axis 1 0 0 -> 1 1 0; origin xyz=-0.04753814992528543 0 -0.27595737685733907 rpy=0 0 0 -> xyz=0 0 0.5 rpy=0 0 0
- joint 4_5: axis 0 0 1 -> 1 1 1; origin xyz=0 0 -0.8666666666666667 rpy=0 0 0 -> xyz=0 0 0.5 rpy=0 0 0

File: body/body5.urdf (robot description, URDF)
Before this commit: robot robot, 25 links, 24 joints
Links:
- removed link 10
- removed link 11
- removed link 12
- removed link 13
- removed link 14
- removed link 15
- removed link 16
- removed link 17
- removed link 18
- removed link 19
- removed link 20
- removed link 21
- removed link 22
- removed link 23
- removed link 24
- removed link 3
- removed link 4
- removed link 5
- removed link 6
- removed link 7
- removed link 8
- removed link 9
- link 0: geometry collision box size=1 1 1; visual box size=1 1 1
- link 1: geometry collision box size=1 1 1; visual box size=1 1 1
- link 2: geometry collision box size=1 1 1; visual box size=1 1 1
Joints:
- removed joint 0_13
- removed joint 0_19
- removed joint 0_7
- removed joint 10_11
- removed joint 11_12
- removed joint 13_14
- removed joint 14_15
- removed joint 15_16
- removed joint 16_17
- removed joint 17_18
- removed joint 19_20
- removed joint 20_21
- removed joint 21_22
- removed joint 22_23
- removed joint 23_24
- removed joint 2_3
- removed joint 3_4
- removed joint 4_5
- removed joint 5_6
- removed joint 7_8
- removed joint 8_9
- removed joint 9_10
- joint 0_1: axis 0 0 1 -> 0 1 1; origin xyz=-0.75 0 3 rpy=0 0 0 -> xyz=0 0 1 rpy=0 0 0
- joint 1_2: axis 0 1 0 -> 0 1 1; origin xyz=-0.18441944797222531 0 0 rpy=0 0 0 -> xyz=0 0 0.5 rpy=0 0 0

File: body/body6.urdf (robot description, URDF)
Before this commit: robot robot, 33 links, 32 joints
Links:
- removed link 10
- removed link 11
- removed link 12
- removed link 13
- removed link 14
- removed link 15
- removed link 16
- removed link 17
- removed link 18
- removed link 19
- removed link 20
- removed link 21
- removed link 22
- removed link 23
- removed link 24
- removed link 25
- removed link 26
- removed link 27
- removed link 28
- removed link 29
- removed link 30
- removed link 31
- removed link 32
- removed link 9
- link 0: geometry collision box size=1 1 1; visual box size=1 1 1
- link 1: geometry collision box size=1 1 1; visual box size=1 1 1
- link 2: geometry collision box size=1 1 1; visual box size=1 1 1
- link 3: geometry collision box size=1 1 1; visual box size=1 1 1
- link 4: geometry collision box size=1 1 1; visual box size=1 1 1
- link 5: geometry collision box size=1 1 1; visual box size=1 1 1
- link 6: geometry collision box size=1 1 1; visual box size=1 1 1
- link 7: geometry collision box size=1 1 1; visual box size=1 1 1
- link 8: geometry collision box size=1 1 1; visual box size=1 1 1
Joints:
- removed joint 0_17
- removed joint 0_25
- removed joint 0_9
- removed joint 10_11
- removed joint 11_12
- removed joint 12_13
- removed joint 13_14
- removed joint 14_15
- removed joint 15_16
- removed joint 17_18
- removed joint 18_19
- removed joint 19_20
- removed joint 20_21
- removed joint 21_22
- removed joint 22_23
- removed joint 23_24
- removed joint 25_26
- removed joint 26_27
- removed joint 27_28
- removed joint 28_29
- removed joint 29_30
- removed joint 30_31
- removed joint 31_32
- removed joint 9_10
- joint 0_1: axis 0 1 1 -> 0 1 0; origin xyz=-0.75 0 3 rpy=0 0 0 -> xyz=0 0 1 rpy=0 0 0
- joint 1_2: axis 1 0 1 -> 1 1 0; origin xyz=-0.13316846584099795 0 0 rpy=0 0 0 -> xyz=0 0 0.5 rpy=0 0 0
- joint 2_3: axis 0 1 0 -> 1 0 1; origin xyz=-0.27052354055851024 0 0 rpy=0 0 0 -> xyz=0 0 0.5 rpy=0 0 0
- joint 3_4: axis 0 1 1 -> 0 1 0; origin xyz=-0.795122970664722 0 0 rpy=0 0 0 -> xyz=0 0 0.5 rpy=0 0 0
- joint 4_5: axis 0 0 1 -> 1 0 0; origin xyz=-0.5122420619993618 0 0 rpy=0 0 0 -> xyz=0 0 0.5 rpy=0 0 0
- joint 5_6: origin xyz=-0.19439927765235332 0 -0.3142254645476624 rpy=0 0 0 -> xyz=0 0 0.5 rpy=0 0 0
- joint 6_7: axis 1 1 0 -> 1 0 0; origin xyz=0 0 -0.8666666666666667 rpy=0 0 0 -> xyz=0 0 0.5 rpy=0 0 0
- joint 7_8: axis 0 0 1 -> 0 1 0; origin xyz=0 0 -0.8666666666666667 rpy=0 0 0 -> xyz=0 0 0.5 rpy=0 0 0

File: body/body7.urdf (robot description, URDF)
Before this commit: robot robot, 21 links, 20 joints
Links:
- removed link 10
- removed link 11
- removed link 12
- removed link 13
- removed link 14
- removed link 15
- removed link 16
- removed link 17
- removed link 18
- removed link 19
- removed link 20
- link 0: geometry collision box size=1 1 1; visual box size=1 1 1
- link 1: geometry collision box size=1 1 1; visual box size=1 1 1
- link 2: geometry collision box size=1 1 1; visual box size=1 1 1
- link 3: geometry collision box size=1 1 1; visual box size=1 1 1
- link 4: geometry collision box size=1 1 1; visual box size=1 1 1
- link 5: geometry collision box size=1 1 1; visual box size=1 1 1
- link 6: geometry collision box size=1 1 1; visual box size=1 1 1
- link 7: geometry collision box size=1 1 1; visual box size=1 1 1
- link 8: geometry collision box size=1 1 1; visual box size=1 1 1
- link 9: geometry collision box size=1 1 1; visual box size=1 1 1
Joints:
- removed joint 0_11
- removed joint 0_16
- removed joint 0_6
- removed joint 11_12
- removed joint 12_13
- removed joint 13_14
- removed joint 14_15
- removed joint 16_17
- removed joint 17_18
- removed joint 18_19
- removed joint 19_20
- removed joint 9_10
- added joint 5_6: type revolute, parent 5, child 6, origin xyz=0 0 0.5 rpy=0 0 0, axis 0 0 1, limit lower=-3.14159 upper=3.14159 effort=0.0 velocity=0.0
- joint 0_1: axis 1 0 0 -> 1 1 0; origin xyz=-0.75 0 3 rpy=0 0 0 -> xyz=0 0 1 rpy=0 0 0
- joint 1_2: axis 0 1 0 -> 0 1 1; origin xyz=-0.8764409937066527 0 0 rpy=0 0 0 -> xyz=0 0 0.5 rpy=0 0 0
- joint 2_3: origin xyz=-0.4150870480596061 0 -0.49116172247302375 rpy=0 0 0 -> xyz=0 0 0.5 rpy=0 0 0
- joint 3_4: origin xyz=0 0 -0.8666666666666667 rpy=0 0 0 -> xyz=0 0 0.5 rpy=0 0 0
- joint 4_5: axis 1 0 1 -> 0 1 0; origin xyz=0 0 -0.8666666666666667 rpy=0 0 0 -> xyz=0 0 0.5 rpy=0 0 0
- joint 6_7: axis 1 1 1 -> 0 0 1; origin xyz=0.726697355015988 0 0 rpy=0 0 0 -> xyz=0 0 0.5 rpy=0 0 0
- joint 7_8: axis 1 1 0 -> 1 1 1; origin xyz=0.0012843622358860163 0 -0.02015642978379517 rpy=0 0 0 -> xyz=0 0 0.5 rpy=0 0 0
- joint 8_9: axis 1 0 1 -> 1 1 0; origin xyz=0 0 -0.8666666666666667 rpy=0 0 0 -> xyz=0 0 0.5 rpy=0 0 0

File: body/body8.urdf (robot description, URDF)
Before this commit: robot robot, 25 links, 24 joints
Links:
- removed link 10
- removed link 11
- removed link 12
- removed link 13
- removed link 14
- removed link 15
- removed link 16
- removed link 17
- removed link 18
- removed link 19
- removed link 20
- removed link 21
- removed link 22
- removed link 23
- removed link 24
- removed link 4
- removed link 5
- removed link 6
- removed link 7
- removed link 8
- removed link 9
- link 0: geometry collision box size=1 1 1; visual box size=1 1 1
- link 1: geometry collision box size=1 1 1; visual box size=1 1 1
- link 2: geometry collision box size=1 1 1; visual box size=1 1 1
- link 3: geometry collision box size=1 1 1; visual box size=1 1 1
Joints:
- removed joint 0_13
- removed joint 0_19
- removed joint 0_7
- removed joint 10_11
- removed joint 11_12
- removed joint 13_14
- removed joint 14_15
- removed joint 15_16
- removed joint 16_17
- removed joint 17_18
- removed joint 19_20
- removed joint 20_21
- removed joint 21_22
- removed joint 22_23
- removed joint 23_24
- removed joint 3_4
- removed joint 4_5
- removed joint 5_6
- removed joint 7_8
- removed joint 8_9
- removed joint 9_10
- joint 0_1: axis 1 1 1 -> 1 0 0; origin xyz=-0.75 0 3 rpy=0 0 0 -> xyz=0 0 1 rpy=0 0 0
- joint 1_2: axis 1 1 0 -> 0 0 1; origin xyz=-0.1140829050749983 0 0 rpy=0 0 0 -> xyz=0 0 0.5 rpy=0 0 0
- joint 2_3: axis 1 1 1 -> 0 0 1; origin xyz=-0.10813499629303891 0 0 rpy=0 0 0 -> xyz=0 0 0.5 rpy=0 0 0

File: body/body9.urdf (robot description, URDF)
Before this commit: robot robot, 29 links, 28 joints
Links:
- removed link 10
- removed link 11
- removed link 12
- removed link 13
- removed link 14
- removed link 15
- removed link 16
- removed link 17
- removed link 18
- removed link 19
- removed link 20
- removed link 21
- removed link 22
- removed link 23
- removed link 24
- removed link 25
- removed link 26
- removed link 27
- removed link 28
- removed link 4
- removed link 5
- removed link 6
- removed link 7
- removed link 8
- removed link 9
- link 0: geometry collision box size=1 1 1; visual box size=1 1 1
- link 1: geometry collision box size=1 1 1; visual box size=1 1 1
- link 2: geometry collision box size=1 1 1; visual box size=1 1 1
- link 3: geometry collision box size=1 1 1; visual box size=1 1 1
Joints:
- removed joint 0_15
- removed joint 0_22
- removed joint 0_8
- removed joint 10_11
- removed joint 11_12
- removed joint 12_13
- removed joint 13_14
- removed joint 15_16
- removed joint 16_17
- removed joint 17_18
- removed joint 18_19
- removed joint 19_20
- removed joint 20_21
- removed joint 22_23
- removed joint 23_24
- removed joint 24_25
- removed joint 25_26
- removed joint 26_27
- removed joint 27_28
- removed joint 3_4
- removed joint 4_5
- removed joint 5_6
- removed joint 6_7
- removed joint 8_9
- removed joint 9_10
- joint 0_1: axis 1 0 1 -> 0 1 0; origin xyz=-0.75 0 3 rpy=0 0 0 -> xyz=0 0 1 rpy=0 0 0
- joint 1_2: axis 1 0 0 -> 1 1 0; origin xyz=-0.7576222097940801 0 0 rpy=0 0 0 -> xyz=0 0 0.5 rpy=0 0 0
- joint 2_3: axis 1 0 0 -> 1 1 1; origin xyz=-0.8213243410933474 0 0 rpy=0 0 0 -> xyz=0 0 0.5 rpy=0 0 0
