Commit message: commit

File: body/body0.urdf (robot description, URDF)
Before this commit: robot robot, 6 links, 5 joints
Links:
- added link 10, mass 1; collision box size=0.9211844743123464 0.9878578031715437 0.5187445189589275; visual box size=0.9211844743123464 0.9878578031715437 0.5187445189589275
- added link 6, mass 1; collision box size=0.7327855285585734 0.8208808784665294 0.7017646511514473; visual box size=0.7327855285585734 0.8208808784665294 0.7017646511514473
- added link 7, mass 1; collision box size=0.755579261781896 0.6192909931751284 0.6245673042773904; visual box size=0.755579261781896 0.6192909931751284 0.6245673042773904
- added link 8, mass 1; collision box size=0.9436502436005325 0.614480617690911 0.613948374104308; visual box size=0.9436502436005325 0.614480617690911 0.613948374104308
- added link 9, mass 1; collision box size=0.5564879281537936 0.7149034830977936 0.8003319521505021; visual box size=0.5564879281537936 0.7149034830977936 0.8003319521505021
- link 3: geometry collision box size=0.5780627600622406 0.5758719700728414 0.7237221563120494; visual box size=0.5780627600622406 0.5758719700728414 0.7237221563120494
- link 4: geometry collision box size=0.6873404900726703 0.5621188163808113 0.8491040491451776; visual box size=0.6873404900726703 0.5621188163808113 0.8491040491451776
- link 5: geometry collision box size=0.955027617856099 0.7659638397009222 0.8515643578556096; visual box size=0.955027617856099 0.7659638397009222 0.8515643578556096
Joints:
- removed joint 2_3
- added joint 1_3: type revolute, parent 1, child 3, origin xyz=0 0.5 0.5 rpy=0 0 0, axis 1 0 0, limit lower=-3.14159 upper=3.14159 effort=0.0 velocity=0.0
- added joint 2_7: type revolute, parent 2, child 7, origin xyz=-0.5 0 0.5 rpy=0 0 0, axis 1 1 1, limit lower=-3.14159 upper=3.14159 effort=0.0 velocity=0.0
- added joint 5_6: type revolute, parent 5, child 6, origin xyz=0 0.7659638397009222 0 rpy=0 0 0, axis 1 1 0, limit lower=-3.14159 upper=3.14159 effort=0.0 velocity=0.0
- added joint 7_8: type revolute, parent 7, child 8, origin xyz=-0.755579261781896 0 0 rpy=0 0 0, axis 0 1 1, limit lower=-3.14159 upper=3.14159 effort=0.0 velocity=0.0
- added joint 8_9: type revolute, parent 8, child 9, origin xyz=-0.9436502436005325 0 0 rpy=0 0 0, axis 0 0 1, limit lower=-3.14159 upper=3.14159 effort=0.0 velocity=0.0
- added joint 9_10: type revolute, parent 9, child 10, origin xyz=-0.5564879281537936 0 0 rpy=0 0 0, axis 1 0 0, limit lower=-3.14159 upper=3.14159 effort=0.0 velocity=0.0
- joint 0_1: axis 1 0 0 -> 0 1 1
- joint 1_2: axis 1 1 1 -> 0 1 0; origin xyz=0 0 0.5 rpy=0 0 0 -> xyz=0 0 1 rpy=0 0 0
- joint 3_4: axis 0 1 1 -> 0 0 1; origin xyz=0 0 0.5 rpy=0 0 0 -> xyz=0 0.5758719700728414 0 rpy=0 0 0
- joint 4_5: axis 0 0 1 -> 0 1 0; origin xyz=0 0 0.5 rpy=0 0 0 -> xyz=0 0.5621188163808113 0 rpy=0 0 0

File: body/body3.urdf (robot description, URDF)
Before this commit: robot robot, 7 links, 6 joints
Links:
- added link 10, mass 1; collision box size=0.9011992503543738 0.8869355559955499 0.8103593755943503; visual box size=0.9011992503543738 0.8869355559955499 0.8103593755943503
- added link 11, mass 1; collision box size=0.7079780228788236 0.7012132870022528 0.5130545991137891; visual box size=0.7079780228788236 0.7012132870022528 0.5130545991137891
- added link 12, mass 1; collision box size=0.6395192087516973 0.5957559606049477 0.581153758452355; visual box size=0.6395192087516973 0.5957559606049477 0.581153758452355
- added link 13, mass 1; collision box size=0.7133393947864348 0.8959150788396438 0.9417435722954098; visual box size=0.7133393947864348 0.8959150788396438 0.9417435722954098
- added link 7, mass 1; collision box size=0.5315949677710285 0.8060663476405208 0.5558930576625681; visual box size=0.5315949677710285 0.8060663476405208 0.5558930576625681
- added link 8, mass 1; collision box size=0.7415012546175808 0.6098091908093749 0.7285924391075145; visual box size=0.7415012546175808 0.6098091908093749 0.7285924391075145
- added link 9, mass 1; collision box size=0.9198264075027995 0.8723044519014493 0.632751672684787; visual box size=0.9198264075027995 0.8723044519014493 0.632751672684787
Joints:
- added joint 10_11: type revolute, parent 10, child 11, origin xyz=0 0.8869355559955499 0 rpy=0 0 0, axis 0 1 0, limit lower=-3.14159 upper=3.14159 effort=0.0 velocity=0.0
- added joint 12_13: type revolute, parent 12, child 13, origin xyz=0 -0.5957559606049477 0 rpy=0 0 0, axis 0 1 1, limit lower=-3.14159 upper=3.14159 effort=0.0 velocity=0.0
- added joint 1_7: type revolute, parent 1, child 7, origin xyz=0 0.5 0.5 rpy=0 0 0, axis 1 0 0, limit lower=-3.14159 upper=3.14159 effort=0.0 velocity=0.0
- added joint 2_12: type revolute, parent 2, child 12, origin xyz=0 -0.5 0.5 rpy=0 0 0, axis 0 1 0, limit lower=-3.14159 upper=3.14159 effort=0.0 velocity=0.0
- added joint 7_8: type revolute, parent 7, child 8, origin xyz=0 0.8060663476405208 0 rpy=0 0 0, axis 0 0 1, limit lower=-3.14159 upper=3.14159 effort=0.0 velocity=0.0
- added joint 8_9: type revolute, parent 8, child 9, origin xyz=0 0.6098091908093749 0 rpy=0 0 0, axis 1 1 0, limit lower=-3.14159 upper=3.14159 effort=0.0 velocity=0.0
- added joint 9_10: type revolute, parent 9, child 10, origin xyz=0 0.8723044519014493 0 rpy=0 0 0, axis 1 0 1, limit lower=-3.14159 upper=3.14159 effort=0.0 velocity=0.0
- joint 0_1: axis 1 1 1 -> 1 0 0
- joint 1_2: origin xyz=0 0 0.5 rpy=0 0 0 -> xyz=0 0 1 rpy=0 0 0
- joint 2_3: origin xyz=0 0 0.5 rpy=0 0 0 -> xyz=0 0 1 rpy=0 0 0
- joint 3_4: axis 1 0 0 -> 0 0 1; origin xyz=0 0 0.5 rpy=0 0 0 -> xyz=0 0 1 rpy=0 0 0
- joint 4_5: axis 0 1 1 -> 0 0 1; origin xyz=0 0 0.5 rpy=0 0 0 -> xyz=0 0 1 rpy=0 0 0
- joint 5_6: axis 0 0 1 -> 0 1 1; origin xyz=0 0 0.5 rpy=0 0 0 -> xyz=0 0 1 rpy=0 0 0

File: body/body4.urdf (robot description, URDF)
Before this commit: robot robot, 6 links, 5 joints
Links:
- added link 10, mass 1; collision box size=0.8577592824954561 0.6753719534497843 0.9210923377932484; visual box size=0.8577592824954561 0.6753719534497843 0.9210923377932484
- added link 6, mass 1; collision box size=1 1 1; visual box size=1 1 1
- added link 7, mass 1; collision box size=1 1 1; visual box size=1 1 1
- added link 8, mass 1; collision box size=0.7896654857427658 0.935141779249739 0.5391778068303933; visual box size=0.7896654857427658 0.935141779249739 0.5391778068303933
- added link 9, mass 1; collision box size=0.7348806603390565 0.688638734542644 0.9338407234897356; visual box size=0.7348806603390565 0.688638734542644 0.9338407234897356
Joints:
- added joint 4_8: type revolute, parent 4, child 8, origin xyz=0.5 0 0.5 rpy=0 0 0, axis 1 0 0, limit lower=-3.14159 upper=3.14159 effort=0.0 velocity=0.0
- added joint 5_6: type revolute, parent 5, child 6, origin xyz=0 0 1 rpy=0 0 0, axis 0 0 1, limit lower=-3.14159 upper=3.14159 effort=0.0 velocity=0.0
- added joint 6_7: type revolute, parent 6, child 7, origin xyz=0 0 1 rpy=0 0 0, axis 0 1 0, limit lower=-3.14159 upper=3.14159 effort=0.0 velocity=0.0
- added joint 6_9: type revolute, parent 6, child 9, origin xyz=0 0.5 0.5 rpy=0 0 0, axis 1 1 0, limit lower=-3.14159 upper=3.14159 effort=0.0 velocity=0.0
- added joint 9_10: type revolute, parent 9, child 10, origin xyz=0 0.688638734542644 0 rpy=0 0 0, axis 1 0 0, limit lower=-3.14159 upper=3.14159 effort=0.0 velocity=0.0
- joint 0_1: axis 1 0 0 -> 1 1 0
- joint 1_2: origin xyz=0 0 0.5 rpy=0 0 0 -> xyz=0 0 1 rpy=0 0 0
- joint 2_3: axis 1 0 1 -> 0 0 1; origin xyz=0 0 0.5 rpy=0 0 0 -> xyz=0 0 1 rpy=0 0 0
- joint 3_4: axis 1 1 0 -> 0 1 0; origin xyz=0 0 0.5 rpy=0 0 0 -> xyz=0 0 1 rpy=0 0 0
- joint 4_5: origin xyz=0 0 0.5 rpy=0 0 0 -> xyz=0 0 1 rpy=0 0 0

File: body/body9.urdf (robot description, URDF)
Before this commit: robot robot, 4 links, 3 joints
Links:
- added link 10, mass 1; collision box size=0.7670157896656031 0.9950139094643311 0.7344473980683208; visual box size=0.7670157896656031 0.9950139094643311 0.7344473980683208
- added link 11, mass 1; collision box size=0.6571370553983436 0.8891423724878975 0.8052194247113569; visual box size=0.6571370553983436 0.8891423724878975 0.8052194247113569
- added link 12, mass 1; collision box size=0.7287096536678966 0.8002442131776308 0.8908728208233672; visual box size=0.7287096536678966 0.8002442131776308 0.8908728208233672
- added link 13, mass 1; collision box size=0.6001965755742663 0.8479318122288166 0.5157735036222717; visual box size=0.6001965755742663 0.8479318122288166 0.5157735036222717
- added link 14, mass 1; collision box size=0.5901628541786734 0.5140293974200951 0.9782618774596648; visual box size=0.5901628541786734 0.5140293974200951 0.9782618774596648
- added link 15, mass 1; collision box size=0.6688944661729981 0.8233411706096092 0.83782057542247; visual box size=0.6688944661729981 0.8233411706096092 0.83782057542247
- added link 16, mass 1; collision box size=0.8735403458136817 0.5084472549893317 0.6411813394609317; visual box size=0.8735403458136817 0.5084472549893317 0.6411813394609317
- added link 17, mass 1; collision box size=0.522741624834822 0.8883967999762443 0.8753071774710519; visual box size=0.522741624834822 0.8883967999762443 0.8753071774710519
- added link 18, mass 1; collision box size=0.7252437262314617 0.8229594027879847 0.7733708177488425; visual box size=0.7252437262314617 0.8229594027879847 0.7733708177488425
- added link 19, mass 1; collision box size=0.9490705191645225 0.7637923802537407 0.7907967015694866; visual box size=0.9490705191645225 0.7637923802537407 0.7907967015694866
- added link 20, mass 1; collision box size=0.8055591046328208 0.6062099139210279 0.5945310217600474; visual box size=0.8055591046328208 0.6062099139210279 0.5945310217600474
- added link 21, mass 1; collision box size=0.7428340175403404 0.6625493541480882 0.6114225759563661; visual box size=0.7428340175403404 0.6625493541480882 0.6114225759563661
- added link 22, mass 1; collision box size=0.9422012228653787 0.9195956847090956 0.8019965164215572; visual box size=0.9422012228653787 0.9195956847090956 0.8019965164215572
- added link 23, mass 1; collision box size=0.781047929210392 0.5834172345413845 0.5292095107458645; visual box size=0.781047929210392 0.5834172345413845 0.5292095107458645
- added link 24, mass 1; collision box size=0.9320569190323261 0.9487627706883164 0.5033957941753963; visual box size=0.9320569190323261 0.9487627706883164 0.5033957941753963
- added link 4, mass 1; collision box size=1 1 1; visual box size=1 1 1
- added link 5, mass 1; collision box size=1 1 1; visual box size=1 1 1
- added link 6, mass 1; collision box size=1 1 1; visual box size=1 1 1
- added link 7, mass 1; collision box size=1 1 1; visual box size=1 1 1
- added link 8, mass 1; collision box size=1 1 1; visual box size=1 1 1
- added link 9, mass 1; collision box size=1 1 1; visual box size=1 1 1
Joints:
- added joint 10_11: type revolute, parent 10, child 11, origin xyz=0 -0.9950139094643311 0 rpy=0 0 0, axis 1 1 0, limit lower=-3.14159 upper=3.14159 effort=0.0 velocity=0.0
- added joint 11_12: type revolute, parent 11, child 12, origin xyz=0 -0.8891423724878975 0 rpy=0 0 0, axis 1 1 0, limit lower=-3.14159 upper=3.14159 effort=0.0 velocity=0.0
- added joint 12_13: type revolute, parent 12, child 13, origin xyz=0 -0.8002442131776308 0 rpy=0 0 0, axis 0 0 1, limit lower=-3.14159 upper=3.14159 effort=0.0 velocity=0.0
- added joint 13_14: type revolute, parent 13, child 14, origin xyz=0 -0.8479318122288166 0 rpy=0 0 0, axis 0 0 1, limit lower=-3.14159 upper=3.14159 effort=0.0 velocity=0.0
- added joint 16_17: type revolute, parent 16, child 17, origin xyz=-0.8735403458136817 0 0 rpy=0 0 0, axis 1 0 1, limit lower=-3.14159 upper=3.14159 effort=0.0 velocity=0.0
- added joint 17_18: type revolute, parent 17, child 18, origin xyz=-0.522741624834822 0 0 rpy=0 0 0, axis 0 0 1, limit lower=-3.14159 upper=3.14159 effort=0.0 velocity=0.0
- added joint 18_19: type revolute, parent 18, child 19, origin xyz=-0.7252437262314617 0 0 rpy=0 0 0, axis 0 1 0, limit lower=-3.14159 upper=3.14159 effort=0.0 velocity=0.0
- added joint 19_20: type revolute, parent 19, child 20, origin xyz=-0.9490705191645225 0 0 rpy=0 0 0, axis 1 0 1, limit lower=-3.14159 upper=3.14159 effort=0.0 velocity=0.0
- added joint 1_10: type revolute, parent 1, child 10, origin xyz=0 -0.5 0.5 rpy=0 0 0, axis 0 1 0, limit lower=-3.14159 upper=3.14159 effort=0.0 velocity=0.0
- added joint 21_22: type revolute, parent 21, child 22, origin xyz=-0.7428340175403404 0 0 rpy=0 0 0, axis 0 1 0, limit lower=-3.14159 upper=3.14159 effort=0.0 velocity=0.0
- added joint 22_23: type revolute, parent 22, child 23, origin xyz=-0.9422012228653787 0 0 rpy=0 0 0, axis 1 0 1, limit lower=-3.14159 upper=3.14159 effort=0.0 velocity=0.0
- added joint 23_24: type revolute, parent 23, child 24, origin xyz=-0.781047929210392 0 0 rpy=0 0 0, axis 1 0 1, limit lower=-3.14159 upper=3.14159 effort=0.0 velocity=0.0
- added joint 3_4: type revolute, parent 3, child 4, origin xyz=0 0 1 rpy=0 0 0, axis 1 0 1, limit lower=-3.14159 upper=3.14159 effort=0.0 velocity=0.0
- added joint 4_5: type revolute, parent 4, child 5, origin xyz=0 0 1 rpy=0 0 0, axis 0 1 0, limit lower=-3.14159 upper=3.14159 effort=0.0 velocity=0.0
- added joint 5_15: type revolute, parent 5, child 15, origin xyz=-0.5 0 0.5 rpy=0 0 0, axis 1 1 1, limit lower=-3.14159 upper=3.14159 effort=0.0 velocity=0.0
- added joint 5_6: type revolute, parent 5, child 6, origin xyz=0 0 1 rpy=0 0 0, axis 1 0 1, limit lower=-3.14159 upper=3.14159 effort=0.0 velocity=0.0
- added joint 6_7: type revolute, parent 6, child 7, origin xyz=0 0 1 rpy=0 0 0, axis 0 1 1, limit lower=-3.14159 upper=3.14159 effort=0.0 velocity=0.0
- added joint 7_8: type revolute, parent 7, child 8, origin xyz=0 0 1 rpy=0 0 0, axis 0 0 1, limit lower=-3.14159 upper=3.14159 effort=0.0 velocity=0.0
- added joint 8_16: type revolute, parent 8, child 16, origin xyz=-0.5 0 0.5 rpy=0 0 0, axis 1 1 0, limit lower=-3.14159 upper=3.14159 effort=0.0 velocity=0.0
- added joint 8_9: type revolute, parent 8, child 9, origin xyz=0 0 1 rpy=0 0 0, axis 0 1 1, limit lower=-3.14159 upper=3.14159 effort=0.0 velocity=0.0
- added joint 9_21: type revolute, parent 9, child 21, origin xyz=-0.5 0 0.5 rpy=0 0 0, axis 1 0 1, limit lower=-3.14159 upper=3.14159 effort=0.0 velocity=0.0
- joint 0_1: axis 0 1 0 -> 1 0 1
- joint 1_2: axis 1 1 0 -> 0 1 0; origin xyz=0 0 0.5 rpy=0 0 0 -> xyz=0 0 1 rpy=0 0 0
- joint 2_3: axis 1 1 1 -> 0 1 1; origin xyz=0 0 0.5 rpy=0 0 0 -> xyz=0 0 1 rpy=0 0 0
