Commit message: commit

File: body/body0.urdf (robot description, URDF)
Before this commit: robot robot, 11 links, 10 joints
Links:
- removed link 10
- removed link 8
- removed link 9
- link 1: geometry collision box size=0.02834747652200631 0.8357651039198697 0.43276706790505337; visual box size=0.02834747652200631 0.8357651039198697 0.43276706790505337
- link 2: geometry collision box size=0.6958328667684435 0.26633056045725956 0.8018263669964836; visual box size=0.6958328667684435 0.26633056045725956 0.8018263669964836
- link 3: geometry collision box size=0.9452706955539223 0.9014274576114836 0.030589983033553536; visual box size=0.9452706955539223 0.9014274576114836 0.030589983033553536
- link 4: geometry collision box size=0.6495461355254983 0.009204938554384978 0.8812338589221554; visual box size=0.6495461355254983 0.009204938554384978 0.8812338589221554
- link 5: geometry collision box size=0.9690406502940995 0.7258526014465152 0.5276294143623982; visual box size=0.9690406502940995 0.7258526014465152 0.5276294143623982
- link 6: geometry collision box size=0.9391670189485866 0.5528595762929651 0.34570041470875246; visual box size=0.9391670189485866 0.5528595762929651 0.34570041470875246
- link 7: geometry collision box size=0.7609477375418205 0.9522444552911937 0.926506623785866; visual box size=0.7609477375418205 0.9522444552911937 0.926506623785866
Joints:
- removed joint 0_5
- removed joint 0_6
- removed joint 3_4
- removed joint 7_8
- removed joint 8_9
- removed joint 9_10
- added joint 0_4: type revolute, parent 0, child 4, origin xyz=0.35 0 0.7 rpy=0 0 0, axis 1 1 0, limit lower=-3.14159 upper=3.14159 effort=0.0 velocity=0.0
- added joint 4_5: type revolute, parent 4, child 5, origin xyz=0.6495461355254983 0 0.8812338589221554 rpy=0 0 0, axis 1 0 1, limit lower=-3.14159 upper=3.14159 effort=0.0 velocity=0.0
- added joint 5_6: type revolute, parent 5, child 6, origin xyz=0.9690406502940995 0 0.5276294143623982 rpy=0 0 0, axis 0 0 1, limit lower=-3.14159 upper=3.14159 effort=0.0 velocity=0.0
- joint 0_1: axis 1 1 1 -> 0 0 1
- joint 1_2: axis 1 0 0 -> 1 1 0; origin xyz=-0.1019744021739154 0 0.7311837167794242 rpy=0 0 0 -> xyz=-0.02834747652200631 0 0.43276706790505337 rpy=0 0 0
- joint 2_3: axis 0 1 1 -> 1 1 0; origin xyz=-0.2794823660111103 0 0.7657254516291417 rpy=0 0 0 -> xyz=-0.6958328667684435 0 0.8018263669964836 rpy=0 0 0
- joint 6_7: axis 1 1 1 -> 0 1 0; origin xyz=0 -0.9614779889500835 0.5392234688708106 rpy=0 0 0 -> xyz=0.9391670189485866 0 0.34570041470875246 rpy=0 0 0

File: body/body1.urdf (robot description, URDF)
Before this commit: robot robot, 11 links, 10 joints
Links:
- removed link 10
- removed link 2
- removed link 3
- removed link 4
- removed link 5
- removed link 6
- removed link 7
- removed link 8
- removed link 9
- link 1: geometry collision box size=0.25158329759496567 0.2122188106686006 0.035734441736370415; visual box size=0.25158329759496567 0.2122188106686006 0.035734441736370415
Joints:
- removed joint 0_5
- removed joint 0_6
- removed joint 1_2
- removed joint 2_3
- removed joint 3_4
- removed joint 6_7
- removed joint 7_8
- removed joint 8_9
- removed joint 9_10

File: body/body100.urdf (robot description, URDF)
Before this commit: robot robot, 11 links, 10 joints
Links:
- removed link 10
- removed link 9
- link 1: geometry collision box size=0.02834747652200631 0.8357651039198697 0.43276706790505337; visual box size=0.02834747652200631 0.8357651039198697 0.43276706790505337
- link 2: geometry collision box size=0.6958328667684435 0.26633056045725956 0.8018263669964836; visual box size=0.6958328667684435 0.26633056045725956 0.8018263669964836
- link 3: geometry collision box size=0.9452706955539223 0.9014274576114836 0.030589983033553536; visual box size=0.9452706955539223 0.9014274576114836 0.030589983033553536
- link 4: geometry collision box size=0.6495461355254983 0.009204938554384978 0.8812338589221554; visual box size=0.6495461355254983 0.009204938554384978 0.8812338589221554
- link 5: geometry collision box size=0.9690406502940995 0.7258526014465152 0.5276294143623982; visual box size=0.9690406502940995 0.7258526014465152 0.5276294143623982
- link 6: geometry collision box size=0.41910192675324365 0.05570723100789343 0.916069348441991; visual box size=0.41910192675324365 0.05570723100789343 0.916069348441991
- link 7: geometry collision box size=0.9391670189485866 0.5528595762929651 0.34570041470875246; visual box size=0.9391670189485866 0.5528595762929651 0.34570041470875246
- link 8: geometry collision box size=0.7609477375418205 0.9522444552911937 0.926506623785866; visual box size=0.7609477375418205 0.9522444552911937 0.926506623785866
Joints:
- removed joint 0_6
- removed joint 8_9
- removed joint 9_10
- added joint 5_6: type revolute, parent 5, child 6, origin xyz=0.9690406502940995 0 0.5276294143623982 rpy=0 0 0, axis 1 0 0, limit lower=-3.14159 upper=3.14159 effort=0.0 velocity=0.0
- joint 0_5: axis 0 1 0 -> 1 0 1
- joint 1_2: axis 1 0 0 -> 1 1 0; origin xyz=-0.1019744021739154 0 0.7311837167794242 rpy=0 0 0 -> xyz=-0.02834747652200631 0 0.43276706790505337 rpy=0 0 0
- joint 2_3: axis 0 1 1 -> 1 1 0; origin xyz=-0.2794823660111103 0 0.7657254516291417 rpy=0 0 0 -> xyz=-0.6958328667684435 0 0.8018263669964836 rpy=0 0 0
- joint 3_4: axis 1 1 1 -> 1 1 0; origin xyz=-0.761925427594386 0 0.6179261849630812 rpy=0 0 0 -> xyz=-0.9452706955539223 0 0.030589983033553536 rpy=0 0 0
- joint 6_7: axis 1 1 1 -> 0 0 1; origin xyz=0 -0.9614779889500835 0.5392234688708106 rpy=0 0 0 -> xyz=0.41910192675324365 0 0.916069348441991 rpy=0 0 0
- joint 7_8: axis 1 1 0 -> 0 1 0; origin xyz=0 -0.9685567743379022 0.19687904392603262 rpy=0 0 0 -> xyz=0.9391670189485866 0 0.34570041470875246 rpy=0 0 0

File: body/body101.urdf (robot description, URDF)
Before this commit: robot robot, 10 links, 9 joints
Links:
- removed link 3
- removed link 4
- removed link 5
- removed link 6
- removed link 7
- removed link 8
- removed link 9
- link 1: geometry collision box size=0.38985211310481016 0.46263554305186805 0.9633005509025323; visual box size=0.38985211310481016 0.46263554305186805 0.9633005509025323
- link 2: geometry collision box size=0.7987736171349602 0.2122188106686006 0.23994900084508952; visual box size=0.7987736171349602 0.2122188106686006 0.23994900084508952
Joints:
- removed joint 0_5
- removed joint 2_3
- removed joint 3_4
- removed joint 5_6
- removed joint 6_7
- removed joint 7_8
- removed joint 8_9
- joint 0_1: axis 1 1 1 -> 0 1 0
- joint 1_2: axis 1 0 0 -> 0 0 1; origin xyz=-0.1019744021739154 0 0.7311837167794242 rpy=0 0 0 -> xyz=-0.38985211310481016 0 0.9633005509025323 rpy=0 0 0

File: body/body102.urdf (robot description, URDF)
Before this commit: robot robot, 11 links, 10 joints
Links:
- removed link 10
- removed link 7
- removed link 8
- removed link 9
- link 1: geometry collision box size=0.5507846417600732 0.1917441039952995 0.7171480392684303; visual box size=0.5507846417600732 0.1917441039952995 0.7171480392684303
- link 2: geometry collision box size=0.23192200537667162 0.1516223763528861 0.9258354717730075; visual box size=0.23192200537667162 0.1516223763528861 0.9258354717730075
- link 3: geometry collision box size=0.7412518562014903 0.6714114753695926 0.0640314382269973; visual box size=0.7412518562014903 0.6714114753695926 0.0640314382269973
- link 4: geometry collision box size=0.04278902933945994 0.7800764890835564 0.8235705112332644; visual box size=0.04278902933945994 0.7800764890835564 0.8235705112332644
- link 5: geometry collision box size=0.47274908866546683 0.7188239240658031 0.8788128002554817; visual box size=0.47274908866546683 0.7188239240658031 0.8788128002554817
- link 6: geometry collision box size=0.3949634040007439 0.8009087709852283 0.44462105605076063; visual box size=0.3949634040007439 0.8009087709852283 0.44462105605076063
Joints:
- removed joint 0_5
- removed joint 0_6
- removed joint 2_3
- removed joint 6_7
- removed joint 7_8
- removed joint 8_9
- removed joint 9_10
- added joint 0_3: type revolute, parent 0, child 3, origin xyz=0 0.35 0.7 rpy=0 0 0, axis 1 0 1, limit lower=-3.14159 upper=3.14159 effort=0.0 velocity=0.0
- added joint 4_5: type revolute, parent 4, child 5, origin xyz=0 0.7800764890835564 0.8235705112332644 rpy=0 0 0, axis 1 0 0, limit lower=-3.14159 upper=3.14159 effort=0.0 velocity=0.0
- added joint 5_6: type revolute, parent 5, child 6, origin xyz=0 0.7188239240658031 0.8788128002554817 rpy=0 0 0, axis 1 1 0, limit lower=-3.14159 upper=3.14159 effort=0.0 velocity=0.0
- joint 0_1: axis 1 1 1 -> 1 0 0; origin xyz=-0.35 0 0.7 rpy=0 0 0 -> xyz=0.35 0 0.7 rpy=0 0 0
- joint 1_2: axis 1 0 0 -> 0 1 0; origin xyz=-0.1019744021739154 0 0.7311837167794242 rpy=0 0 0 -> xyz=0.5507846417600732 0 0.7171480392684303 rpy=0 0 0
- joint 3_4: axis 1 1 1 -> 0 1 0; origin xyz=-0.761925427594386 0 0.6179261849630812 rpy=0 0 0 -> xyz=0 0.6714114753695926 0.0640314382269973 rpy=0 0 0

File: body/body103.urdf (robot description, URDF)
Before this commit: robot robot, 11 links, 10 joints
Links:
- removed link 10
- removed link 6
- removed link 7
- removed link 8
- removed link 9
- link 1: geometry collision box size=0.8268053039341334 0.7651626025054384 0.22192817569031764; visual box size=0.8268053039341334 0.7651626025054384 0.22192817569031764
- link 2: geometry collision box size=0.36024490950020127 0.9220033436961468 0.8268716790242738; visual box size=0.36024490950020127 0.9220033436961468 0.8268716790242738
- link 3: geometry collision box size=0.2144004325789165 0.9274756314280604 0.8289200487784194; visual box size=0.2144004325789165 0.9274756314280604 0.8289200487784194
- link 4: geometry collision box size=0.8004478385429662 0.19343561801924003 0.30984995729953557; visual box size=0.8004478385429662 0.19343561801924003 0.30984995729953557
- link 5: geometry collision box size=0.08671825263492183 0.7312759796520136 0.6717014565164733; visual box size=0.08671825263492183 0.7312759796520136 0.6717014565164733
Joints:
- removed joint 0_5
- removed joint 0_6
- removed joint 1_2
- removed joint 6_7
- removed joint 7_8
- removed joint 8_9
- removed joint 9_10
- added joint 0_2: type revolute, parent 0, child 2, origin xyz=0 0.35 0.7 rpy=0 0 0, axis 1 0 1, limit lower=-3.14159 upper=3.14159 effort=0.0 velocity=0.0
- added joint 4_5: type revolute, parent 4, child 5, origin xyz=0 0.19343561801924003 0.30984995729953557 rpy=0 0 0, axis 1 1 0, limit lower=-3.14159 upper=3.14159 effort=0.0 velocity=0.0
- joint 0_1: axis 1 1 1 -> 0 0 1; origin xyz=-0.35 0 0.7 rpy=0 0 0 -> xyz=0 -0.35 0.7 rpy=0 0 0
- joint 2_3: axis 0 1 1 -> 1 0 1; origin xyz=-0.2794823660111103 0 0.7657254516291417 rpy=0 0 0 -> xyz=0 0.9220033436961468 0.8268716790242738 rpy=0 0 0
- joint 3_4: origin xyz=-0.761925427594386 0 0.6179261849630812 rpy=0 0 0 -> xyz=0 0.9274756314280604 0.8289200487784194 rpy=0 0 0

File: body/body104.urdf (robot description, URDF)
Before this commit: robot robot, 11 links, 10 joints
Links:
- link 5: geometry collision box size=0.7735937030276743 0.9601271002174996 0.16585644239491049; visual box size=0.7735937030276743 0.9601271002174996 0.16585644239491049
- link 8: geometry collision box size=0.29878889785386775 0.36118993472238414 0.1659560571297456; visual box size=0.29878889785386775 0.36118993472238414 0.1659560571297456
- link 9: geometry collision box size=0.26381193894997024 0.33185448722063815 0.8174003109567611; visual box size=0.26381193894997024 0.33185448722063815 0.8174003109567611
Joints:
- joint 8_9: axis 1 0 1 -> 0 0 1
- joint 9_10: axis 1 1 0 -> 1 0 1; origin xyz=0 -0.33185448722063815 0.33612164567091696 rpy=0 0 0 -> xyz=0 -0.33185448722063815 0.8174003109567611 rpy=0 0 0

File: body/body105.urdf (robot description, URDF)
Before this commit: robot robot, 10 links, 9 joints
Links:
- removed link 9
- link 1: geometry collision box size=0.02834747652200631 0.8357651039198697 0.43276706790505337; visual box size=0.02834747652200631 0.8357651039198697 0.43276706790505337
- link 2: geometry collision box size=0.6958328667684435 0.26633056045725956 0.8018263669964836; visual box size=0.6958328667684435 0.26633056045725956 0.8018263669964836
- link 3: geometry collision box size=0.9452706955539223 0.9014274576114836 0.030589983033553536; visual box size=0.9452706955539223 0.9014274576114836 0.030589983033553536
- link 4: geometry collision box size=0.6495461355254983 0.009204938554384978 0.8812338589221554; visual box size=0.6495461355254983 0.009204938554384978 0.8812338589221554
- link 5: geometry collision box size=0.9690406502940995 0.7258526014465152 0.5276294143623982; visual box size=0.9690406502940995 0.7258526014465152 0.5276294143623982
- link 6: geometry collision box size=0.41910192675324365 0.05570723100789343 0.916069348441991; visual box size=0.41910192675324365 0.05570723100789343 0.916069348441991
- link 7: geometry collision box size=0.9391670189485866 0.5528595762929651 0.34570041470875246; visual box size=0.9391670189485866 0.5528595762929651 0.34570041470875246
- link 8: geometry collision box size=0.7609477375418205 0.9522444552911937 0.926506623785866; visual box size=0.7609477375418205 0.9522444552911937 0.926506623785866
Joints:
- removed joint 0_4
- removed joint 8_9
- added joint 3_4: type revolute, parent 3, child 4, origin xyz=-0.9452706955539223 0 0.030589983033553536 rpy=0 0 0, axis 1 1 0, limit lower=-3.14159 upper=3.14159 effort=0.0 velocity=0.0
- joint 0_5: axis 0 1 0 -> 1 0 1; origin xyz=0 -0.35 0.7 rpy=0 0 0 -> xyz=0.35 0 0.7 rpy=0 0 0
- joint 1_2: axis 1 0 0 -> 1 1 0; origin xyz=-0.1019744021739154 0 0.7311837167794242 rpy=0 0 0 -> xyz=-0.02834747652200631 0 0.43276706790505337 rpy=0 0 0
- joint 2_3: axis 0 1 1 -> 1 1 0; origin xyz=-0.2794823660111103 0 0.7657254516291417 rpy=0 0 0 -> xyz=-0.6958328667684435 0 0.8018263669964836 rpy=0 0 0
- joint 5_6: axis 0 1 0 -> 1 0 0; origin xyz=0 -0.9601271002174996 0.9751029769612911 rpy=0 0 0 -> xyz=0.9690406502940995 0 0.5276294143623982 rpy=0 0 0
- joint 6_7: axis 1 1 1 -> 0 0 1; origin xyz=0 -0.9614779889500835 0.5392234688708106 rpy=0 0 0 -> xyz=0.41910192675324365 0 0.916069348441991 rpy=0 0 0
- joint 7_8: axis 1 0 1 -> 0 1 0; origin xyz=0 -0.9685567743379022 0.19687904392603262 rpy=0 0 0 -> xyz=0.9391670189485866 0 0.34570041470875246 rpy=0 0 0

File: body/body106.urdf (robot description, URDF)
Before this commit: robot robot, 12 links, 11 joints
Links:
- removed link 10
- removed link 11
- removed link 3
- removed link 4
- removed link 5
- removed link 6
- removed link 7
- removed link 8
- removed link 9
- link 1: geometry collision box size=0.38985211310481016 0.46263554305186805 0.9633005509025323; visual box size=0.38985211310481016 0.46263554305186805 0.9633005509025323
- link 2: geometry collision box size=0.7987736171349602 0.2122188106686006 0.035734441736370415; visual box size=0.7987736171349602 0.2122188106686006 0.035734441736370415
Joints:
- removed joint 0_6
- removed joint 0_7
- removed joint 10_11
- removed joint 2_3
- removed joint 3_4
- removed joint 4_5
- removed joint 7_8
- removed joint 8_9
- removed joint 9_10
- joint 0_1: axis 1 1 1 -> 0 1 0
- joint 1_2: axis 1 1 1 -> 0 0 1; origin xyz=-0.6827908250947565 0 0.4974180340567149 rpy=0 0 0 -> xyz=-0.38985211310481016 0 0.9633005509025323 rpy=0 0 0

File: body/body107.urdf (robot description, URDF)
Before this commit: robot robot, 11 links, 10 joints
Links:
- removed link 10
- removed link 7
- removed link 8
- removed link 9
- link 1: geometry collision box size=0.5507846417600732 0.1917441039952995 0.7171480392684303; visual box size=0.5507846417600732 0.1917441039952995 0.7171480392684303
- link 2: geometry collision box size=0.23192200537667162 0.1516223763528861 0.9258354717730075; visual box size=0.23192200537667162 0.1516223763528861 0.9258354717730075
- link 3: geometry collision box size=0.7412518562014903 0.6714114753695926 0.0640314382269973; visual box size=0.7412518562014903 0.6714114753695926 0.0640314382269973
- link 4: geometry collision box size=0.04278902933945994 0.7800764890835564 0.8235705112332644; visual box size=0.04278902933945994 0.7800764890835564 0.8235705112332644
- link 5: geometry collision box size=0.47274908866546683 0.7188239240658031 0.8788128002554817; visual box size=0.47274908866546683 0.7188239240658031 0.8788128002554817
- link 6: geometry collision box size=0.3949634040007439 0.8009087709852283 0.44462105605076063; visual box size=0.3949634040007439 0.8009087709852283 0.44462105605076063
Joints:
- removed joint 0_5
- removed joint 0_6
- removed joint 2_3
- removed joint 6_7
- removed joint 7_8
- removed joint 8_9
- removed joint 9_10
- added joint 0_3: type revolute, parent 0, child 3, origin xyz=0 0.35 0.7 rpy=0 0 0, axis 1 0 1, limit lower=-3.14159 upper=3.14159 effort=0.0 velocity=0.0
- added joint 4_5: type revolute, parent 4, child 5, origin xyz=0 0.7800764890835564 0.8235705112332644 rpy=0 0 0, axis 1 0 0, limit lower=-3.14159 upper=3.14159 effort=0.0 velocity=0.0
- added joint 5_6: type revolute, parent 5, child 6, origin xyz=0 0.7188239240658031 0.8788128002554817 rpy=0 0 0, axis 1 1 0, limit lower=-3.14159 upper=3.14159 effort=0.0 velocity=0.0
- joint 0_1: axis 1 1 1 -> 1 0 0; origin xyz=-0.35 0 0.7 rpy=0 0 0 -> xyz=0.35 0 0.7 rpy=0 0 0
- joint 1_2: axis 1 0 0 -> 0 1 0; origin xyz=-0.1019744021739154 0 0.7311837167794242 rpy=0 0 0 -> xyz=0.5507846417600732 0 0.7171480392684303 rpy=0 0 0
- joint 3_4: axis 1 1 1 -> 0 1 0; origin xyz=-0.761925427594386 0 0.6179261849630812 rpy=0 0 0 -> xyz=0 0.6714114753695926 0.0640314382269973 rpy=0 0 0

File: body/body108.urdf (robot description, URDF)
Before this commit: robot robot, 11 links, 10 joints
Links:
- removed link 10
- removed link 6
- removed link 7
- removed link 8
- removed link 9
- link 1: geometry collision box size=0.8268053039341334 0.7651626025054384 0.22192817569031764; visual box size=0.8268053039341334 0.7651626025054384 0.22192817569031764
- link 2: geometry collision box size=0.36024490950020127 0.9220033436961468 0.8268716790242738; visual box size=0.36024490950020127 0.9220033436961468 0.8268716790242738
- link 3: geometry collision box size=0.7323477044226232 0.9274756314280604 0.8289200487784194; visual box size=0.7323477044226232 0.9274756314280604 0.8289200487784194
- link 4: geometry collision box size=0.8004478385429662 0.19343561801924003 0.30984995729953557; visual box size=0.8004478385429662 0.19343561801924003 0.30984995729953557
- link 5: geometry collision box size=0.08671825263492183 0.7312759796520136 0.6717014565164733; visual box size=0.08671825263492183 0.7312759796520136 0.6717014565164733
Joints:
- removed joint 0_5
- removed joint 0_6
- removed joint 1_2
- removed joint 6_7
- removed joint 7_8
- removed joint 8_9
- removed joint 9_10
- added joint 0_2: type revolute, parent 0, child 2, origin xyz=0 0.35 0.7 rpy=0 0 0, axis 1 0 1, limit lower=-3.14159 upper=3.14159 effort=0.0 velocity=0.0
- added joint 4_5: type revolute, parent 4, child 5, origin xyz=0 0.19343561801924003 0.30984995729953557 rpy=0 0 0, axis 1 1 0, limit lower=-3.14159 upper=3.14159 effort=0.0 velocity=0.0
- joint 0_1: axis 1 1 1 -> 0 0 1; origin xyz=-0.35 0 0.7 rpy=0 0 0 -> xyz=0 -0.35 0.7 rpy=0 0 0
- joint 2_3: axis 0 1 1 -> 1 0 1; origin xyz=-0.2794823660111103 0 0.7657254516291417 rpy=0 0 0 -> xyz=0 0.9220033436961468 0.8268716790242738 rpy=0 0 0
- joint 3_4: origin xyz=-0.761925427594386 0 0.6179261849630812 rpy=0 0 0 -> xyz=0 0.9274756314280604 0.8289200487784194 rpy=0 0 0

File: body/body109.urdf (robot description, URDF)
Before this commit: robot robot, 11 links, 10 joints
Links:
- link 5: geometry collision box size=0.7735937030276743 0.9601271002174996 0.16585644239491049; visual box size=0.7735937030276743 0.9601271002174996 0.16585644239491049
- link 8: geometry collision box size=0.29878889785386775 0.36118993472238414 0.1659560571297456; visual box size=0.29878889785386775 0.36118993472238414 0.1659560571297456
- link 9: geometry collision box size=0.26381193894997024 0.33185448722063815 0.8174003109567611; visual box size=0.26381193894997024 0.33185448722063815 0.8174003109567611
Joints:
- joint 7_8: axis 1 1 0 -> 0 0 1
- joint 8_9: axis 1 0 0 -> 0 0 1
- joint 9_10: axis 1 1 0 -> 1 0 1; origin xyz=0 -0.33185448722063815 0.33612164567091696 rpy=0 0 0 -> xyz=0 -0.33185448722063815 0.8174003109567611 rpy=0 0 0

File: body/body110.urdf (robot description, URDF)
Before this commit: robot robot, 11 links, 10 joints
Links:
- removed link 10
- removed link 9
- link 1: geometry collision box size=0.02834747652200631 0.8357651039198697 0.43276706790505337; visual box size=0.02834747652200631 0.8357651039198697 0.43276706790505337
- link 2: geometry collision box size=0.6958328667684435 0.26633056045725956 0.8018263669964836; visual box size=0.6958328667684435 0.26633056045725956 0.8018263669964836
- link 3: geometry collision box size=0.9452706955539223 0.9014274576114836 0.030589983033553536; visual box size=0.9452706955539223 0.9014274576114836 0.030589983033553536
- link 4: geometry collision box size=0.6495461355254983 0.009204938554384978 0.8812338589221554; visual box size=0.6495461355254983 0.009204938554384978 0.8812338589221554
- link 5: geometry collision box size=0.9690406502940995 0.7258526014465152 0.5276294143623982; visual box size=0.9690406502940995 0.7258526014465152 0.5276294143623982
- link 6: geometry collision box size=0.41910192675324365 0.05570723100789343 0.916069348441991; visual box size=0.41910192675324365 0.05570723100789343 0.916069348441991
- link 7: geometry collision box size=0.9391670189485866 0.5528595762929651 0.34570041470875246; visual box size=0.9391670189485866 0.5528595762929651 0.34570041470875246
- link 8: geometry collision box size=0.7609477375418205 0.9522444552911937 0.926506623785866; visual box size=0.7609477375418205 0.9522444552911937 0.926506623785866
Joints:
- removed joint 0_6
- removed joint 8_9
- removed joint 9_10
- added joint 5_6: type revolute, parent 5, child 6, origin xyz=0.9690406502940995 0 0.5276294143623982 rpy=0 0 0, axis 1 0 0, limit lower=-3.14159 upper=3.14159 effort=0.0 velocity=0.0
- joint 0_5: axis 0 1 0 -> 1 0 1
- joint 1_2: axis 1 0 0 -> 1 1 0; origin xyz=-0.1019744021739154 0 0.7311837167794242 rpy=0 0 0 -> xyz=-0.02834747652200631 0 0.43276706790505337 rpy=0 0 0
- joint 2_3: axis 0 1 1 -> 1 1 0; origin xyz=-0.2794823660111103 0 0.7657254516291417 rpy=0 0 0 -> xyz=-0.6958328667684435 0 0.8018263669964836 rpy=0 0 0
- joint 3_4: axis 1 1 1 -> 1 1 0; origin xyz=-0.761925427594386 0 0.6179261849630812 rpy=0 0 0 -> xyz=-0.9452706955539223 0 0.030589983033553536 rpy=0 0 0
- joint 6_7: axis 1 1 1 -> 0 0 1; origin xyz=0 -0.9614779889500835 0.5392234688708106 rpy=0 0 0 -> xyz=0.41910192675324365 0 0.916069348441991 rpy=0 0 0
- joint 7_8: axis 1 1 0 -> 0 1 0; origin xyz=0 -0.9685567743379022 0.19687904392603262 rpy=0 0 0 -> xyz=0.9391670189485866 0 0.34570041470875246 rpy=0 0 0
