Commit message: commit

File: body/body111.urdf (robot description, URDF)
Before this commit: robot robot, 10 links, 9 joints
Links:
- removed link 3
- removed link 4
- removed link 5
- removed link 6
- removed link 7
- removed link 8
- removed link 9
- link 1: geometry collision box size=0.38985211310481016 0.46263554305186805 0.9633005509025323; visual box size=0.38985211310481016 0.46263554305186805 0.9633005509025323
- link 2: geometry collision box size=0.7987736171349602 0.2122188106686006 0.035734441736370415; visual box size=0.7987736171349602 0.2122188106686006 0.035734441736370415
Joints:
- removed joint 0_4
- removed joint 0_5
- removed joint 2_3
- removed joint 5_6
- removed joint 6_7
- removed joint 7_8
- removed joint 8_9
- joint 0_1: axis 1 1 1 -> 0 1 0
- joint 1_2: axis 0 1 1 -> 1 0 1; origin xyz=-0.1019744021739154 0 0.7311837167794242 rpy=0 0 0 -> xyz=-0.38985211310481016 0 0.9633005509025323 rpy=0 0 0

File: body/body112.urdf (robot description, URDF)
Before this commit: robot robot, 11 links, 10 joints
Links:
- removed link 10
- removed link 7
- removed link 8
- removed link 9
- link 1: geometry collision box size=0.5507846417600732 0.1917441039952995 0.7171480392684303; visual box size=0.5507846417600732 0.1917441039952995 0.7171480392684303
- link 2: geometry collision box size=0.23192200537667162 0.1516223763528861 0.9258354717730075; visual box size=0.23192200537667162 0.1516223763528861 0.9258354717730075
- link 3: geometry collision box size=0.7412518562014903 0.6714114753695926 0.0640314382269973; visual box size=0.7412518562014903 0.6714114753695926 0.0640314382269973
- link 4: geometry collision box size=0.04278902933945994 0.7800764890835564 0.8235705112332644; visual box size=0.04278902933945994 0.7800764890835564 0.8235705112332644
- link 5: geometry collision box size=0.47274908866546683 0.7188239240658031 0.8788128002554817; visual box size=0.47274908866546683 0.7188239240658031 0.8788128002554817
- link 6: geometry collision box size=0.3949634040007439 0.8009087709852283 0.44462105605076063; visual box size=0.3949634040007439 0.8009087709852283 0.44462105605076063
Joints:
- removed joint 0_5
- removed joint 0_6
- removed joint 2_3
- removed joint 6_7
- removed joint 7_8
- removed joint 8_9
- removed joint 9_10
- added joint 0_3: type revolute, parent 0, child 3, origin xyz=0 0.35 0.7 rpy=0 0 0, axis 1 0 1, limit lower=-3.14159 upper=3.14159 effort=0.0 velocity=0.0
- added joint 4_5: type revolute, parent 4, child 5, origin xyz=0 0.7800764890835564 0.8235705112332644 rpy=0 0 0, axis 1 0 0, limit lower=-3.14159 upper=3.14159 effort=0.0 velocity=0.0
- added joint 5_6: type revolute, parent 5, child 6, origin xyz=0 0.7188239240658031 0.8788128002554817 rpy=0 0 0, axis 1 1 0, limit lower=-3.14159 upper=3.14159 effort=0.0 velocity=0.0
- joint 0_1: axis 1 1 1 -> 1 0 0; origin xyz=-0.35 0 0.7 rpy=0 0 0 -> xyz=0.35 0 0.7 rpy=0 0 0
- joint 1_2: axis 1 0 0 -> 0 1 0; origin xyz=-0.1019744021739154 0 0.7311837167794242 rpy=0 0 0 -> xyz=0.5507846417600732 0 0.7171480392684303 rpy=0 0 0
- joint 3_4: axis 1 1 1 -> 0 1 0; origin xyz=-0.761925427594386 0 0.6179261849630812 rpy=0 0 0 -> xyz=0 0.6714114753695926 0.0640314382269973 rpy=0 0 0

File: body/body113.urdf (robot description, URDF)
Before this commit: robot robot, 10 links, 9 joints
Links:
- removed link 6
- removed link 7
- removed link 8
- removed link 9
- link 1: geometry collision box size=0.8268053039341334 0.7651626025054384 0.22192817569031764; visual box size=0.8268053039341334 0.7651626025054384 0.22192817569031764
- link 2: geometry collision box size=0.36024490950020127 0.9220033436961468 0.8268716790242738; visual box size=0.36024490950020127 0.9220033436961468 0.8268716790242738
- link 3: geometry collision box size=0.2144004325789165 0.9274756314280604 0.8289200487784194; visual box size=0.2144004325789165 0.9274756314280604 0.8289200487784194
- link 4: geometry collision box size=0.8004478385429662 0.19343561801924003 0.30984995729953557; visual box size=0.8004478385429662 0.19343561801924003 0.30984995729953557
- link 5: geometry collision box size=0.08671825263492183 0.7312759796520136 0.6717014565164733; visual box size=0.08671825263492183 0.7312759796520136 0.6717014565164733
Joints:
- removed joint 0_4
- removed joint 0_5
- removed joint 1_2
- removed joint 5_6
- removed joint 6_7
- removed joint 7_8
- removed joint 8_9
- added joint 0_2: type revolute, parent 0, child 2, origin xyz=0 0.35 0.7 rpy=0 0 0, axis 1 0 1, limit lower=-3.14159 upper=3.14159 effort=0.0 velocity=0.0
- added joint 3_4: type revolute, parent 3, child 4, origin xyz=0 0.9274756314280604 0.8289200487784194 rpy=0 0 0, axis 1 1 1, limit lower=-3.14159 upper=3.14159 effort=0.0 velocity=0.0
- added joint 4_5: type revolute, parent 4, child 5, origin xyz=0 0.19343561801924003 0.30984995729953557 rpy=0 0 0, axis 1 1 0, limit lower=-3.14159 upper=3.14159 effort=0.0 velocity=0.0
- joint 0_1: axis 1 1 1 -> 0 0 1; origin xyz=-0.35 0 0.7 rpy=0 0 0 -> xyz=0 -0.35 0.7 rpy=0 0 0
- joint 2_3: axis 0 1 1 -> 1 0 1; origin xyz=-0.2794823660111103 0 0.7657254516291417 rpy=0 0 0 -> xyz=0 0.9220033436961468 0.8268716790242738 rpy=0 0 0

File: body/body114.urdf (robot description, URDF)
Before this commit: robot robot, 12 links, 11 joints
Links:
- removed link 11
- link 10: geometry collision box size=0.003383119374356758 0.6779342495476912 0.33789686162786514; visual box size=0.003383119374356758 0.6779342495476912 0.33789686162786514
- link 5: geometry collision box size=0.7735937030276743 0.9601271002174996 0.16585644239491049; visual box size=0.7735937030276743 0.9601271002174996 0.16585644239491049
- link 8: geometry collision box size=0.29878889785386775 0.36118993472238414 0.1659560571297456; visual box size=0.29878889785386775 0.36118993472238414 0.1659560571297456
- link 9: geometry collision box size=0.26381193894997024 0.33185448722063815 0.8174003109567611; visual box size=0.26381193894997024 0.33185448722063815 0.8174003109567611
Joints:
- removed joint 0_7
- removed joint 10_11
- removed joint 5_6
- added joint 0_6: type revolute, parent 0, child 6, origin xyz=0 -0.35 0.7 rpy=0 0 0, axis 0 1 0, limit lower=-3.14159 upper=3.14159 effort=0.0 velocity=0.0
- added joint 6_7: type revolute, parent 6, child 7, origin xyz=0 -0.9614779889500835 0.5392234688708106 rpy=0 0 0, axis 1 1 1, limit lower=-3.14159 upper=3.14159 effort=0.0 velocity=0.0
- joint 8_9: axis 1 1 0 -> 0 0 1
- joint 9_10: origin xyz=0 -0.4231806365506502 0.768119941477691 rpy=0 0 0 -> xyz=0 -0.33185448722063815 0.8174003109567611 rpy=0 0 0

File: body/body115.urdf (robot description, URDF)
Before this commit: robot robot, 11 links, 10 joints
Links:
- removed link 10
- removed link 8
- removed link 9
- link 1: geometry collision box size=0.02834747652200631 0.8357651039198697 0.43276706790505337; visual box size=0.02834747652200631 0.8357651039198697 0.43276706790505337
- link 2: geometry collision box size=0.6958328667684435 0.26633056045725956 0.8018263669964836; visual box size=0.6958328667684435 0.26633056045725956 0.8018263669964836
- link 3: geometry collision box size=0.9452706955539223 0.9014274576114836 0.030589983033553536; visual box size=0.9452706955539223 0.9014274576114836 0.030589983033553536
- link 4: geometry collision box size=0.6495461355254983 0.009204938554384978 0.8812338589221554; visual box size=0.6495461355254983 0.009204938554384978 0.8812338589221554
- link 5: geometry collision box size=0.9690406502940995 0.7258526014465152 0.5276294143623982; visual box size=0.9690406502940995 0.7258526014465152 0.5276294143623982
- link 6: geometry collision box size=0.41910192675324365 0.05570723100789343 0.916069348441991; visual box size=0.41910192675324365 0.05570723100789343 0.916069348441991
- link 7: geometry collision box size=0.9391670189485866 0.5528595762929651 0.34570041470875246; visual box size=0.9391670189485866 0.5528595762929651 0.34570041470875246
Joints:
- removed joint 0_5
- removed joint 0_6
- removed joint 3_4
- removed joint 7_8
- removed joint 8_9
- removed joint 9_10
- added joint 0_4: type revolute, parent 0, child 4, origin xyz=0.35 0 0.7 rpy=0 0 0, axis 1 1 0, limit lower=-3.14159 upper=3.14159 effort=0.0 velocity=0.0
- added joint 4_5: type revolute, parent 4, child 5, origin xyz=0.6495461355254983 0 0.8812338589221554 rpy=0 0 0, axis 1 0 1, limit lower=-3.14159 upper=3.14159 effort=0.0 velocity=0.0
- added joint 5_6: type revolute, parent 5, child 6, origin xyz=0.9690406502940995 0 0.5276294143623982 rpy=0 0 0, axis 1 0 0, limit lower=-3.14159 upper=3.14159 effort=0.0 velocity=0.0
- joint 1_2: axis 1 0 0 -> 1 1 0; origin xyz=-0.1019744021739154 0 0.7311837167794242 rpy=0 0 0 -> xyz=-0.02834747652200631 0 0.43276706790505337 rpy=0 0 0
- joint 2_3: axis 0 1 1 -> 1 1 0; origin xyz=-0.2794823660111103 0 0.7657254516291417 rpy=0 0 0 -> xyz=-0.6958328667684435 0 0.8018263669964836 rpy=0 0 0
- joint 6_7: axis 1 1 1 -> 0 0 1; origin xyz=0 -0.9614779889500835 0.5392234688708106 rpy=0 0 0 -> xyz=0.41910192675324365 0 0.916069348441991 rpy=0 0 0

File: body/body116.urdf (robot description, URDF)
Before this commit: robot robot, 10 links, 9 joints
Links:
- removed link 4
- removed link 5
- removed link 6
- removed link 7
- removed link 8
- removed link 9
- link 1: geometry collision box size=0.6827908250947565 0.6442456994239817 0.4974180340567149; visual box size=0.6827908250947565 0.6442456994239817 0.4974180340567149
- link 2: geometry collision box size=0.38985211310481016 0.46263554305186805 0.9633005509025323; visual box size=0.38985211310481016 0.46263554305186805 0.9633005509025323
- link 3: geometry collision box size=0.7987736171349602 0.2122188106686006 0.035734441736370415; visual box size=0.7987736171349602 0.2122188106686006 0.035734441736370415
Joints:
- removed joint 0_5
- removed joint 0_6
- removed joint 3_4
- removed joint 6_7
- removed joint 7_8
- removed joint 8_9
- joint 1_2: axis 1 0 0 -> 0 1 0; origin xyz=-0.1019744021739154 0 0.7311837167794242 rpy=0 0 0 -> xyz=-0.6827908250947565 0 0.4974180340567149 rpy=0 0 0
- joint 2_3: axis 0 1 1 -> 1 0 1; origin xyz=-0.2794823660111103 0 0.7657254516291417 rpy=0 0 0 -> xyz=-0.38985211310481016 0 0.9633005509025323 rpy=0 0 0

File: body/body117.urdf (robot description, URDF)
Before this commit: robot robot, 11 links, 10 joints
Links:
- removed link 10
- removed link 7
- removed link 8
- removed link 9
- link 1: geometry collision box size=0.5507846417600732 0.1917441039952995 0.7171480392684303; visual box size=0.5507846417600732 0.1917441039952995 0.7171480392684303
- link 2: geometry collision box size=0.23192200537667162 0.1516223763528861 0.9258354717730075; visual box size=0.23192200537667162 0.1516223763528861 0.9258354717730075
- link 3: geometry collision box size=0.7412518562014903 0.6714114753695926 0.0640314382269973; visual box size=0.7412518562014903 0.6714114753695926 0.0640314382269973
- link 4: geometry collision box size=0.04278902933945994 0.7800764890835564 0.8235705112332644; visual box size=0.04278902933945994 0.7800764890835564 0.8235705112332644
- link 5: geometry collision box size=0.47274908866546683 0.7188239240658031 0.8788128002554817; visual box size=0.47274908866546683 0.7188239240658031 0.8788128002554817
- link 6: geometry collision box size=0.3949634040007439 0.8009087709852283 0.44462105605076063; visual box size=0.3949634040007439 0.8009087709852283 0.44462105605076063
Joints:
- removed joint 0_5
- removed joint 0_6
- removed joint 2_3
- removed joint 6_7
- removed joint 7_8
- removed joint 8_9
- removed joint 9_10
- added joint 0_3: type revolute, parent 0, child 3, origin xyz=0 0.35 0.7 rpy=0 0 0, axis 1 0 1, limit lower=-3.14159 upper=3.14159 effort=0.0 velocity=0.0
- added joint 4_5: type revolute, parent 4, child 5, origin xyz=0 0.7800764890835564 0.8235705112332644 rpy=0 0 0, axis 1 0 0, limit lower=-3.14159 upper=3.14159 effort=0.0 velocity=0.0
- added joint 5_6: type revolute, parent 5, child 6, origin xyz=0 0.7188239240658031 0.8788128002554817 rpy=0 0 0, axis 1 1 0, limit lower=-3.14159 upper=3.14159 effort=0.0 velocity=0.0
- joint 0_1: axis 1 1 1 -> 1 0 0; origin xyz=-0.35 0 0.7 rpy=0 0 0 -> xyz=0.35 0 0.7 rpy=0 0 0
- joint 1_2: axis 1 0 0 -> 0 1 0; origin xyz=-0.1019744021739154 0 0.7311837167794242 rpy=0 0 0 -> xyz=0.5507846417600732 0 0.7171480392684303 rpy=0 0 0
- joint 3_4: axis 1 1 1 -> 0 1 0; origin xyz=-0.761925427594386 0 0.6179261849630812 rpy=0 0 0 -> xyz=0 0.6714114753695926 0.0640314382269973 rpy=0 0 0

Commit message: commit

File: body/body0.urdf (robot description, URDF)
Before this commit: robot robot, 11 links, 10 joints
Links:
- removed link 10
- removed link 8
- removed link 9
- link 1: geometry collision box size=0.6958328667684435 0.26633056045725956 0.8018263669964836; visual box size=0.6958328667684435 0.26633056045725956 0.8018263669964836
- link 2: geometry collision box size=0.030589983033553536 0.0254458609934608 0.5414124727934966; visual box size=0.030589983033553536 0.0254458609934608 0.5414124727934966
- link 3: geometry collision box size=0.9690406502940995 0.7258526014465152 0.5276294143623982; visual box size=0.9690406502940995 0.7258526014465152 0.5276294143623982
- link 4: geometry collision box size=0.23308445025757263 0.2308665415409843 0.2187810373376886; visual box size=0.23308445025757263 0.2308665415409843 0.2187810373376886
- link 5: geometry collision box size=0.4161799388943461 0.9162698355052942 0.9221885624698875; visual box size=0.4161799388943461 0.9162698355052942 0.9221885624698875
- link 6: geometry collision box size=0.12088995980580641 0.3326951853601291 0.7214844075832684; visual box size=0.12088995980580641 0.3326951853601291 0.7214844075832684
- link 7: geometry collision box size=0.5077172505113161 0.9101850589387533 0.18984972911602638; visual box size=0.5077172505113161 0.9101850589387533 0.18984972911602638
Joints:
- removed joint 0_5
- removed joint 0_6
- removed joint 3_4
- removed joint 7_8
- removed joint 8_9
- removed joint 9_10
- added joint 0_4: type revolute, parent 0, child 4, origin xyz=0.35 0 0.7 rpy=0 0 0, axis 1 0 0, limit lower=-3.14159 upper=3.14159 effort=0.0 velocity=0.0
- added joint 4_5: type revolute, parent 4, child 5, origin xyz=0.23308445025757263 0 0.2187810373376886 rpy=0 0 0, axis 0 1 1, limit lower=-3.14159 upper=3.14159 effort=0.0 velocity=0.0
- added joint 5_6: type revolute, parent 5, child 6, origin xyz=0.4161799388943461 0 0.9221885624698875 rpy=0 0 0, axis 1 0 1, limit lower=-3.14159 upper=3.14159 effort=0.0 velocity=0.0
- joint 0_1: axis 1 1 0 -> 1 0 1
- joint 1_2: axis 1 0 1 -> 0 1 1; origin xyz=-0.2794823660111103 0 0.7657254516291417 rpy=0 0 0 -> xyz=-0.6958328667684435 0 0.8018263669964836 rpy=0 0 0
- joint 2_3: axis 1 0 1 -> 0 1 1; origin xyz=-0.6179261849630812 0 0.13224085421692466 rpy=0 0 0 -> xyz=-0.030589983033553536 0 0.5414124727934966 rpy=0 0 0
- joint 6_7: axis 1 0 0 -> 0 0 1; origin xyz=0 -0.5959789505447018 0.7076761524222557 rpy=0 0 0 -> xyz=0.12088995980580641 0 0.7214844075832684 rpy=0 0 0

File: body/body1 2.urdf (robot description, URDF)
Before this commit: robot robot, 10 links, 9 joints
Links:
- removed link 4
- removed link 5
- removed link 6
- removed link 7
- removed link 8
- removed link 9
- link 1: geometry collision box size=0.33113745196273026 0.5998551847634835 0.8045694845140354; visual box size=0.33113745196273026 0.5998551847634835 0.8045694845140354
- link 2: geometry collision box size=0.8610088608533248 0.798438940577426 0.7970975626354962; visual box size=0.8610088608533248 0.798438940577426 0.7970975626354962
- link 3: geometry collision box size=0.08323413780389788 0.0166906301155596 0.014559974924812313; visual box size=0.08323413780389788 0.0166906301155596 0.014559974924812313
Joints:
- removed joint 0_6
- removed joint 3_4
- removed joint 4_5
- removed joint 6_7
- removed joint 7_8
- removed joint 8_9
- joint 0_1: axis 1 1 0 -> 0 1 1; origin xyz=0.35 0 0.7 rpy=0 0 0 -> xyz=0 0.35 0.7 rpy=0 0 0
- joint 1_2: axis 1 0 1 -> 0 1 1; origin xyz=0.9364359028718386 0 0.25823287309055987 rpy=0 0 0 -> xyz=0 0.5998551847634835 0.8045694845140354 rpy=0 0 0
- joint 2_3: axis 1 0 1 -> 0 1 1; origin xyz=0.9874559311566145 0 0.3765165628179754 rpy=0 0 0 -> xyz=0 0.798438940577426 0.7970975626354962 rpy=0 0 0

File: body/body1.urdf (robot description, URDF)
Before this commit: robot robot, 8 links, 7 joints
Links:
- removed link 4
- removed link 5
- removed link 6
- removed link 7
- link 1: geometry collision box size=0.33113745196273026 0.5998551847634835 0.8045694845140354; visual box size=0.33113745196273026 0.5998551847634835 0.8045694845140354
- link 2: geometry collision box size=0.8610088608533248 0.798438940577426 0.7970975626354962; visual box size=0.8610088608533248 0.798438940577426 0.7970975626354962
- link 3: geometry collision box size=0.08323413780389788 0.0166906301155596 0.014559974924812313; visual box size=0.08323413780389788 0.0166906301155596 0.014559974924812313
Joints:
- removed joint 0_4
- removed joint 4_5
- removed joint 5_6
- removed joint 6_7
- joint 0_1: axis 0 0 1 -> 0 1 1; origin xyz=0 -0.35 0.7 rpy=0 0 0 -> xyz=0 0.35 0.7 rpy=0 0 0
- joint 1_2: axis 1 0 1 -> 0 1 1; origin xyz=0 -0.18012029744042013 0.4918620234154919 rpy=0 0 0 -> xyz=0 0.5998551847634835 0.8045694845140354 rpy=0 0 0
- joint 2_3: axis 1 0 0 -> 0 1 1; origin xyz=0 -0.7860225796338303 0.7748980921186417 rpy=0 0 0 -> xyz=0 0.798438940577426 0.7970975626354962 rpy=0 0 0

File: body/body2 4.urdf (robot description, URDF)
Before this commit: robot robot, 9 links, 8 joints
Links:
- removed link 8
- link 1: geometry collision box size=0.4092427925243217 0.5639201301507394 0.5383856696593964; visual box size=0.4092427925243217 0.5639201301507394 0.5383856696593964
- link 2: geometry collision box size=0.5638591384666509 0.9572125911649866 0.9679969186558055; visual box size=0.5638591384666509 0.9572125911649866 0.9679969186558055
- link 3: geometry collision box size=0.3818538196974869 0.3260421720580161 0.9164761276183131; visual box size=0.3818538196974869 0.3260421720580161 0.9164761276183131
- link 4: geometry collision box size=0.37584830395281976 0.4316837934902342 0.22633586446501464; visual box size=0.37584830395281976 0.4316837934902342 0.22633586446501464
- link 5: geometry collision box size=0.3838915449465743 0.854964553667212 0.15902737971998726; visual box size=0.3838915449465743 0.854964553667212 0.15902737971998726
- link 6: geometry collision box size=0.4963055048217496 0.41549171522014816 0.31915254850071706; visual box size=0.4963055048217496 0.41549171522014816 0.31915254850071706
- link 7: geometry collision box size=0.14329141733747497 0.023774922802194953 0.660058845741202; visual box size=0.14329141733747497 0.023774922802194953 0.660058845741202
Joints:
- removed joint 7_8
- joint 0_1: axis 1 0 0 -> 0 1 0
- joint 0_2: axis 0 1 1 -> 1 0 0
- joint 2_3: axis 1 1 0 -> 1 1 1; origin xyz=0 -0.5238954398669781 0.030700276754036526 rpy=0 0 0 -> xyz=0 -0.9572125911649866 0.9679969186558055 rpy=0 0 0
- joint 3_4: axis 0 0 1 -> 0 1 0; origin xyz=0 -0.29860594962301334 0.9679033101508892 rpy=0 0 0 -> xyz=0 -0.3260421720580161 0.9164761276183131 rpy=0 0 0
- joint 4_5: axis 1 1 1 -> 0 1 1; origin xyz=0 -0.9392884321352825 0.7438421186671211 rpy=0 0 0 -> xyz=0 -0.4316837934902342 0.22633586446501464 rpy=0 0 0
- joint 5_6: axis 1 0 0 -> 0 0 1; origin xyz=0 -0.850526660963271 0.5905839712874152 rpy=0 0 0 -> xyz=0 -0.854964553667212 0.15902737971998726 rpy=0 0 0

File: body/body4 3.urdf (robot description, URDF)
Before this commit: robot robot, 8 links, 7 joints
Links:
- link 1: geometry collision box size=0.23047247273079485 0.0782033251045755 0.40107076549286413; visual box size=0.23047247273079485 0.0782033251045755 0.40107076549286413
- link 2: geometry collision box size=0.18447621515420787 0.3614600396390498 0.0668786669697441; visual box size=0.18447621515420787 0.3614600396390498 0.0668786669697441
- link 3: geometry collision box size=0.17564548307796102 0.20876891866685288 0.04392108802403227; visual box size=0.17564548307796102 0.20876891866685288 0.04392108802403227
- link 4: geometry collision box size=0.006272684498982883 0.06086685846026163 0.7792633152106944; visual box size=0.006272684498982883 0.06086685846026163 0.7792633152106944
- link 5: geometry collision box size=0.8355383276164946 0.8372671046774086 0.5652006443590916; visual box size=0.8355383276164946 0.8372671046774086 0.5652006443590916
- link 6: geometry collision box size=0.8987919599055768 0.49116020718177145 0.9357362201159075; visual box size=0.8987919599055768 0.49116020718177145 0.9357362201159075
- link 7: geometry collision box size=0.4974180340567149 0.7815483812998142 0.04790106606058808; visual box size=0.4974180340567149 0.7815483812998142 0.04790106606058808
Joints:
- removed joint 1_2
- added joint 0_2: type revolute, parent 0, child 2, origin xyz=0 -0.35 0.7 rpy=0 0 0, axis 0 1 0, limit lower=-3.14159 upper=3.14159 effort=0.0 velocity=0.0
- joint 0_1: axis 1 0 1 -> 0 0 1
- joint 0_4: origin xyz=0.35 0 0.7 rpy=0 0 0 -> xyz=0 0.35 0.7 rpy=0 0 0
- joint 2_3: axis 0 1 1 -> 0 1 0; origin xyz=-0.030589983033553536 0 0.5414124727934966 rpy=0 0 0 -> xyz=0 -0.3614600396390498 0.0668786669697441 rpy=0 0 0
- joint 4_5: axis 0 1 1 -> 0 1 0; origin xyz=0.23308445025757263 0 0.2187810373376886 rpy=0 0 0 -> xyz=0 0.06086685846026163 0.7792633152106944 rpy=0 0 0
- joint 5_6: axis 1 0 1 -> 1 1 0; origin xyz=0.4161799388943461 0 0.9221885624698875 rpy=0 0 0 -> xyz=0 0.8372671046774086 0.5652006443590916 rpy=0 0 0
- joint 6_7: axis 0 0 1 -> 0 1 0; origin xyz=0.12088995980580641 0 0.7214844075832684 rpy=0 0 0 -> xyz=0 0.49116020718177145 0.9357362201159075 rpy=0 0 0
