Commit message: plot

File: body/body0.urdf (robot description, URDF)
Before this commit: robot robot, 8 links, 7 joints
Links:
- added link 10, mass 1; collision box size=0.11902055707377501 0.24608679063361372 0.8194931666705297; visual box size=0.11902055707377501 0.24608679063361372 0.8194931666705297
- added link 8, mass 1; collision box size=0.9492204766705261 0.35764406505883395 0.4042940811668897; visual box size=0.9492204766705261 0.35764406505883395 0.4042940811668897
- added link 9, mass 1; collision box size=0.5785188290568746 0.009078386819528439 0.04672711869894153; visual box size=0.5785188290568746 0.009078386819528439 0.04672711869894153
- link 1: geometry collision box size=0.2794823660111103 0.9163453718085519 0.7657254516291417; visual box size=0.2794823660111103 0.9163453718085519 0.7657254516291417
- link 2: geometry collision box size=0.6179261849630812 0.44483568613752145 0.13224085421692466; visual box size=0.6179261849630812 0.44483568613752145 0.13224085421692466
- link 3: geometry collision box size=0.9601271002174996 0.16585644239491049 0.16648447729129467; visual box size=0.9601271002174996 0.16585644239491049 0.16648447729129467
- link 4: geometry collision box size=0.1816686685456037 0.9685567743379022 0.19687904392603262; visual box size=0.1816686685456037 0.9685567743379022 0.19687904392603262
- link 5: geometry collision box size=0.36118993472238414 0.1659560571297456 0.14570190954068252; visual box size=0.36118993472238414 0.1659560571297456 0.14570190954068252
- link 6: geometry collision box size=0.5861412585033708 0.5959789505447018 0.7076761524222557; visual box size=0.5861412585033708 0.5959789505447018 0.7076761524222557
- link 7: geometry collision box size=0.48074518663003896 0.31579310584644404 0.48121838623686386; visual box size=0.48074518663003896 0.31579310584644404 0.48121838623686386
Joints:
- removed joint 0_4
- removed joint 4_5
- removed joint 5_6
- added joint 0_5: type revolute, parent 0, child 5, origin xyz=0.35 0 0.7 rpy=0 0 0, axis 1 1 0, limit lower=-3.14159 upper=3.14159 effort=0.0 velocity=0.0
- added joint 0_6: type revolute, parent 0, child 6, origin xyz=0 -0.35 0.7 rpy=0 0 0, axis 1 0 0, limit lower=-3.14159 upper=3.14159 effort=0.0 velocity=0.0
- added joint 3_4: type revolute, parent 3, child 4, origin xyz=-0.9601271002174996 0 0.16648447729129467 rpy=0 0 0, axis 1 1 0, limit lower=-3.14159 upper=3.14159 effort=0.0 velocity=0.0
- added joint 7_8: type revolute, parent 7, child 8, origin xyz=0 -0.31579310584644404 0.48121838623686386 rpy=0 0 0, axis 1 0 0, limit lower=-3.14159 upper=3.14159 effort=0.0 velocity=0.0
- added joint 8_9: type revolute, parent 8, child 9, origin xyz=0 -0.35764406505883395 0.4042940811668897 rpy=0 0 0, axis 1 0 0, limit lower=-3.14159 upper=3.14159 effort=0.0 velocity=0.0
- added joint 9_10: type revolute, parent 9, child 10, origin xyz=0 -0.009078386819528439 0.04672711869894153 rpy=0 0 0, axis 1 0 1, limit lower=-3.14159 upper=3.14159 effort=0.0 velocity=0.0
- joint 0_1: axis 1 0 1 -> 1 1 0
- joint 1_2: axis 0 1 1 -> 1 0 1; origin xyz=-0.6958328667684435 0 0.8018263669964836 rpy=0 0 0 -> xyz=-0.2794823660111103 0 0.7657254516291417 rpy=0 0 0
- joint 2_3: axis 0 1 1 -> 1 0 1; origin xyz=-0.030589983033553536 0 0.5414124727934966 rpy=0 0 0 -> xyz=-0.6179261849630812 0 0.13224085421692466 rpy=0 0 0
- joint 6_7: axis 0 0 1 -> 1 0 0; origin xyz=0.12088995980580641 0 0.7214844075832684 rpy=0 0 0 -> xyz=0 -0.5959789505447018 0.7076761524222557 rpy=0 0 0

File: body/body1.urdf (robot description, URDF)
Before this commit: robot robot, 4 links, 3 joints
Links:
- added link 4, mass 1; collision box size=0.9568854268308546 0.3400733891851615 0.17864939257994905; visual box size=0.9568854268308546 0.3400733891851615 0.17864939257994905
- added link 5, mass 1; collision box size=0.3259049331519225 0.27368510859414175 0.28882651639491064; visual box size=0.3259049331519225 0.27368510859414175 0.28882651639491064
- added link 6, mass 1; collision box size=0.3478845080276999 0.6440630729912358 0.7378273527139065; visual box size=0.3478845080276999 0.6440630729912358 0.7378273527139065
- added link 7, mass 1; collision box size=0.8699112524611612 0.6883369568719272 0.9761221883019409; visual box size=0.8699112524611612 0.6883369568719272 0.9761221883019409
- link 1: geometry collision box size=0.8677989344185498 0.18012029744042013 0.4918620234154919; visual box size=0.8677989344185498 0.18012029744042013 0.4918620234154919
- link 2: geometry collision box size=0.3613262330227255 0.7860225796338303 0.7748980921186417; visual box size=0.3613262330227255 0.7860225796338303 0.7748980921186417
- link 3: geometry collision box size=0.3634317633458549 0.7044695740067031 0.280852055812124; visual box size=0.3634317633458549 0.7044695740067031 0.280852055812124
Joints:
- added joint 0_4: type revolute, parent 0, child 4, origin xyz=0 0.35 0.7 rpy=0 0 0, axis 0 1 0, limit lower=-3.14159 upper=3.14159 effort=0.0 velocity=0.0
- added joint 4_5: type revolute, parent 4, child 5, origin xyz=0 0.3400733891851615 0.17864939257994905 rpy=0 0 0, axis 0 1 0, limit lower=-3.14159 upper=3.14159 effort=0.0 velocity=0.0
- added joint 5_6: type revolute, parent 5, child 6, origin xyz=0 0.27368510859414175 0.28882651639491064 rpy=0 0 0, axis 1 1 0, limit lower=-3.14159 upper=3.14159 effort=0.0 velocity=0.0
- added joint 6_7: type revolute, parent 6, child 7, origin xyz=0 0.6440630729912358 0.7378273527139065 rpy=0 0 0, axis 0 1 1, limit lower=-3.14159 upper=3.14159 effort=0.0 velocity=0.0
- joint 0_1: axis 0 1 1 -> 0 0 1; origin xyz=0 0.35 0.7 rpy=0 0 0 -> xyz=0 -0.35 0.7 rpy=0 0 0
- joint 1_2: axis 0 1 1 -> 1 0 1; origin xyz=0 0.5998551847634835 0.8045694845140354 rpy=0 0 0 -> xyz=0 -0.18012029744042013 0.4918620234154919 rpy=0 0 0
- joint 2_3: axis 0 1 1 -> 1 0 0; origin xyz=0 0.798438940577426 0.7970975626354962 rpy=0 0 0 -> xyz=0 -0.7860225796338303 0.7748980921186417 rpy=0 0 0

File: body/body2.urdf (robot description, URDF)
Before this commit: robot robot, 9 links, 8 joints
Links:
- added link 10, mass 1; collision box size=0.11902055707377501 0.24608679063361372 0.8194931666705297; visual box size=0.11902055707377501 0.24608679063361372 0.8194931666705297
- added link 9, mass 1; collision box size=0.5785188290568746 0.009078386819528439 0.04672711869894153; visual box size=0.5785188290568746 0.009078386819528439 0.04672711869894153
- link 1: geometry collision box size=0.2794823660111103 0.9163453718085519 0.7657254516291417; visual box size=0.2794823660111103 0.9163453718085519 0.7657254516291417
- link 2: geometry collision box size=0.6179261849630812 0.44483568613752145 0.13224085421692466; visual box size=0.6179261849630812 0.44483568613752145 0.13224085421692466
- link 3: geometry collision box size=0.9601271002174996 0.16585644239491049 0.16648447729129467; visual box size=0.9601271002174996 0.16585644239491049 0.16648447729129467
- link 4: geometry collision box size=0.1816686685456037 0.9685567743379022 0.19687904392603262; visual box size=0.1816686685456037 0.9685567743379022 0.19687904392603262
- link 5: geometry collision box size=0.36118993472238414 0.1659560571297456 0.14570190954068252; visual box size=0.36118993472238414 0.1659560571297456 0.14570190954068252
- link 6: geometry collision box size=0.5861412585033708 0.5959789505447018 0.7076761524222557; visual box size=0.5861412585033708 0.5959789505447018 0.7076761524222557
- link 7: geometry collision box size=0.6888553487611566 0.31579310584644404 0.48121838623686386; visual box size=0.6888553487611566 0.31579310584644404 0.48121838623686386
- link 8: geometry collision box size=0.9492204766705261 0.35764406505883395 0.4042940811668897; visual box size=0.9492204766705261 0.35764406505883395 0.4042940811668897
Joints:
- removed joint 0_2
- removed joint 0_7
- removed joint 4_5
- removed joint 5_6
- added joint 0_5: type revolute, parent 0, child 5, origin xyz=0.35 0 0.7 rpy=0 0 0, axis 1 1 0, limit lower=-3.14159 upper=3.14159 effort=0.0 velocity=0.0
- added joint 0_6: type revolute, parent 0, child 6, origin xyz=0 -0.35 0.7 rpy=0 0 0, axis 1 0 0, limit lower=-3.14159 upper=3.14159 effort=0.0 velocity=0.0
- added joint 1_2: type revolute, parent 1, child 2, origin xyz=-0.2794823660111103 0 0.7657254516291417 rpy=0 0 0, axis 1 0 1, limit lower=-3.14159 upper=3.14159 effort=0.0 velocity=0.0
- added joint 6_7: type revolute, parent 6, child 7, origin xyz=0 -0.5959789505447018 0.7076761524222557 rpy=0 0 0, axis 1 0 0, limit lower=-3.14159 upper=3.14159 effort=0.0 velocity=0.0
- added joint 8_9: type revolute, parent 8, child 9, origin xyz=0 -0.35764406505883395 0.4042940811668897 rpy=0 0 0, axis 1 0 0, limit lower=-3.14159 upper=3.14159 effort=0.0 velocity=0.0
- added joint 9_10: type revolute, parent 9, child 10, origin xyz=0 -0.009078386819528439 0.04672711869894153 rpy=0 0 0, axis 1 0 1, limit lower=-3.14159 upper=3.14159 effort=0.0 velocity=0.0
- joint 0_1: axis 1 0 0 -> 1 1 0; origin xyz=0.35 0 0.7 rpy=0 0 0 -> xyz=-0.35 0 0.7 rpy=0 0 0
- joint 2_3: axis 1 1 0 -> 1 0 1; origin xyz=0 -0.5238954398669781 0.030700276754036526 rpy=0 0 0 -> xyz=-0.6179261849630812 0 0.13224085421692466 rpy=0 0 0
- joint 3_4: axis 0 0 1 -> 1 1 0; origin xyz=0 -0.29860594962301334 0.9679033101508892 rpy=0 0 0 -> xyz=-0.9601271002174996 0 0.16648447729129467 rpy=0 0 0
- joint 7_8: axis 0 1 0 -> 1 0 0; origin xyz=0 0.0990253627729546 0.5733827030223086 rpy=0 0 0 -> xyz=0 -0.31579310584644404 0.48121838623686386 rpy=0 0 0

File: body/body3.urdf (robot description, URDF)
Before this commit: robot robot, 10 links, 9 joints
Links:
- removed link 8
- removed link 9
- link 1: geometry collision box size=0.8677989344185498 0.18012029744042013 0.4918620234154919; visual box size=0.8677989344185498 0.18012029744042013 0.4918620234154919
- link 2: geometry collision box size=0.3613262330227255 0.7860225796338303 0.7748980921186417; visual box size=0.3613262330227255 0.7860225796338303 0.7748980921186417
- link 3: geometry collision box size=0.3634317633458549 0.7044695740067031 0.280852055812124; visual box size=0.3634317633458549 0.7044695740067031 0.280852055812124
- link 4: geometry collision box size=0.9568854268308546 0.3400733891851615 0.17864939257994905; visual box size=0.9568854268308546 0.3400733891851615 0.17864939257994905
- link 5: geometry collision box size=0.3259049331519225 0.27368510859414175 0.28882651639491064; visual box size=0.3259049331519225 0.27368510859414175 0.28882651639491064
- link 6: geometry collision box size=0.3478845080276999 0.6440630729912358 0.7378273527139065; visual box size=0.3478845080276999 0.6440630729912358 0.7378273527139065
- link 7: geometry collision box size=0.8699112524611612 0.6883369568719272 0.9761221883019409; visual box size=0.8699112524611612 0.6883369568719272 0.9761221883019409
Joints:
- removed joint 0_9
- removed joint 7_8
- joint 0_1: axis 1 0 1 -> 0 0 1; origin xyz=0.35 0 0.7 rpy=0 0 0 -> xyz=0 -0.35 0.7 rpy=0 0 0
- joint 0_4: axis 1 0 0 -> 0 1 0; origin xyz=0 -0.35 0.7 rpy=0 0 0 -> xyz=0 0.35 0.7 rpy=0 0 0
- joint 1_2: axis 1 0 0 -> 1 0 1; origin xyz=0.18792209207738453 0 0.586792874492806 rpy=0 0 0 -> xyz=0 -0.18012029744042013 0.4918620234154919 rpy=0 0 0
- joint 2_3: axis 0 0 1 -> 1 0 0; origin xyz=0.15894476133589752 0 0.4351028346327276 rpy=0 0 0 -> xyz=0 -0.7860225796338303 0.7748980921186417 rpy=0 0 0
- joint 4_5: axis 1 0 0 -> 0 1 0; origin xyz=0 -0.010506151518672291 0.9825836265504634 rpy=0 0 0 -> xyz=0 0.3400733891851615 0.17864939257994905 rpy=0 0 0
- joint 5_6: axis 1 0 0 -> 1 1 0; origin xyz=0 -0.3985551600379108 0.06419198150479799 rpy=0 0 0 -> xyz=0 0.27368510859414175 0.28882651639491064 rpy=0 0 0
- joint 6_7: axis 1 0 0 -> 0 1 1; origin xyz=0 -0.21519327003609845 0.6178068800115557 rpy=0 0 0 -> xyz=0 0.6440630729912358 0.7378273527139065 rpy=0 0 0

File: body/body4.urdf (robot description, URDF)
Before this commit: robot robot, 4 links, 3 joints
Links:
- added link 10, mass 1; collision box size=0.11902055707377501 0.24608679063361372 0.8194931666705297; visual box size=0.11902055707377501 0.24608679063361372 0.8194931666705297
- added link 4, mass 1; collision box size=0.1816686685456037 0.9685567743379022 0.19687904392603262; visual box size=0.1816686685456037 0.9685567743379022 0.19687904392603262
- added link 5, mass 1; collision box size=0.36118993472238414 0.1659560571297456 0.14570190954068252; visual box size=0.36118993472238414 0.1659560571297456 0.14570190954068252
- added link 6, mass 1; collision box size=0.5861412585033708 0.5959789505447018 0.7076761524222557; visual box size=0.5861412585033708 0.5959789505447018 0.7076761524222557
- added link 7, mass 1; collision box size=0.6888553487611566 0.31579310584644404 0.48121838623686386; visual box size=0.6888553487611566 0.31579310584644404 0.48121838623686386
- added link 8, mass 1; collision box size=0.9492204766705261 0.35764406505883395 0.4042940811668897; visual box size=0.9492204766705261 0.35764406505883395 0.4042940811668897
- added link 9, mass 1; collision box size=0.5785188290568746 0.009078386819528439 0.33937331252621783; visual box size=0.5785188290568746 0.009078386819528439 0.33937331252621783
- link 1: geometry collision box size=0.2794823660111103 0.9163453718085519 0.7657254516291417; visual box size=0.2794823660111103 0.9163453718085519 0.7657254516291417
- link 2: geometry collision box size=0.6179261849630812 0.44483568613752145 0.13224085421692466; visual box size=0.6179261849630812 0.44483568613752145 0.13224085421692466
- link 3: geometry collision box size=0.9601271002174996 0.16585644239491049 0.16648447729129467; visual box size=0.9601271002174996 0.16585644239491049 0.16648447729129467
Joints:
- added joint 0_5: type revolute, parent 0, child 5, origin xyz=0.35 0 0.7 rpy=0 0 0, axis 1 1 0, limit lower=-3.14159 upper=3.14159 effort=0.0 velocity=0.0
- added joint 0_6: type revolute, parent 0, child 6, origin xyz=0 -0.35 0.7 rpy=0 0 0, axis 1 0 0, limit lower=-3.14159 upper=3.14159 effort=0.0 velocity=0.0
- added joint 3_4: type revolute, parent 3, child 4, origin xyz=-0.9601271002174996 0 0.16648447729129467 rpy=0 0 0, axis 1 1 0, limit lower=-3.14159 upper=3.14159 effort=0.0 velocity=0.0
- added joint 6_7: type revolute, parent 6, child 7, origin xyz=0 -0.5959789505447018 0.7076761524222557 rpy=0 0 0, axis 1 0 0, limit lower=-3.14159 upper=3.14159 effort=0.0 velocity=0.0
- added joint 7_8: type revolute, parent 7, child 8, origin xyz=0 -0.31579310584644404 0.48121838623686386 rpy=0 0 0, axis 1 0 0, limit lower=-3.14159 upper=3.14159 effort=0.0 velocity=0.0
- added joint 8_9: type revolute, parent 8, child 9, origin xyz=0 -0.35764406505883395 0.4042940811668897 rpy=0 0 0, axis 1 0 0, limit lower=-3.14159 upper=3.14159 effort=0.0 velocity=0.0
- added joint 9_10: type revolute, parent 9, child 10, origin xyz=0 -0.009078386819528439 0.33937331252621783 rpy=0 0 0, axis 1 0 1, limit lower=-3.14159 upper=3.14159 effort=0.0 velocity=0.0
- joint 0_1: axis 1 0 0 -> 1 1 0; origin xyz=0 0.35 0.7 rpy=0 0 0 -> xyz=-0.35 0 0.7 rpy=0 0 0
- joint 1_2: axis 1 0 0 -> 1 0 1; origin xyz=0 0.8289343809851581 0.39779731306487276 rpy=0 0 0 -> xyz=-0.2794823660111103 0 0.7657254516291417 rpy=0 0 0
- joint 2_3: origin xyz=0 0.17757811046169503 0.3172416351802618 rpy=0 0 0 -> xyz=-0.6179261849630812 0 0.13224085421692466 rpy=0 0 0

File: body/body5.urdf (robot description, URDF)
Before this commit: robot robot, 8 links, 7 joints
Links:
- link 1: geometry collision box size=0.8677989344185498 0.18012029744042013 0.4918620234154919; visual box size=0.8677989344185498 0.18012029744042013 0.4918620234154919
- link 2: geometry collision box size=0.3613262330227255 0.7860225796338303 0.7748980921186417; visual box size=0.3613262330227255 0.7860225796338303 0.7748980921186417
- link 3: geometry collision box size=0.3634317633458549 0.7044695740067031 0.280852055812124; visual box size=0.3634317633458549 0.7044695740067031 0.280852055812124
- link 4: geometry collision box size=0.9568854268308546 0.3400733891851615 0.17864939257994905; visual box size=0.9568854268308546 0.3400733891851615 0.17864939257994905
- link 5: geometry collision box size=0.3259049331519225 0.27368510859414175 0.28882651639491064; visual box size=0.3259049331519225 0.27368510859414175 0.28882651639491064
- link 6: geometry collision box size=0.3478845080276999 0.6440630729912358 0.7378273527139065; visual box size=0.3478845080276999 0.6440630729912358 0.7378273527139065
- link 7: geometry collision box size=0.8699112524611612 0.6883369568719272 0.9761221883019409; visual box size=0.8699112524611612 0.6883369568719272 0.9761221883019409
Joints:
- removed joint 0_2
- removed joint 0_7
- removed joint 3_4
- added joint 0_4: type revolute, parent 0, child 4, origin xyz=0 0.35 0.7 rpy=0 0 0, axis 0 1 0, limit lower=-3.14159 upper=3.14159 effort=0.0 velocity=0.0
- added joint 1_2: type revolute, parent 1, child 2, origin xyz=0 -0.18012029744042013 0.4918620234154919 rpy=0 0 0, axis 1 0 1, limit lower=-3.14159 upper=3.14159 effort=0.0 velocity=0.0
- added joint 6_7: type revolute, parent 6, child 7, origin xyz=0 0.6440630729912358 0.7378273527139065 rpy=0 0 0, axis 0 1 1, limit lower=-3.14159 upper=3.14159 effort=0.0 velocity=0.0
- joint 0_1: axis 0 1 0 -> 0 0 1; origin xyz=0.35 0 0.7 rpy=0 0 0 -> xyz=0 -0.35 0.7 rpy=0 0 0
- joint 2_3: axis 1 1 1 -> 1 0 0; origin xyz=0 -0.9572125911649866 0.9679969186558055 rpy=0 0 0 -> xyz=0 -0.7860225796338303 0.7748980921186417 rpy=0 0 0
- joint 4_5: axis 0 1 1 -> 0 1 0; origin xyz=0 -0.4316837934902342 0.22633586446501464 rpy=0 0 0 -> xyz=0 0.3400733891851615 0.17864939257994905 rpy=0 0 0
- joint 5_6: axis 0 0 1 -> 1 1 0; origin xyz=0 -0.854964553667212 0.15902737971998726 rpy=0 0 0 -> xyz=0 0.27368510859414175 0.28882651639491064 rpy=0 0 0
