Commit message: commit

File: body/body2.urdf (robot description, URDF)
Before this commit: robot robot, 11 links, 10 joints
Links:
- removed link 10
- removed link 9
- link 1: geometry collision box size=0.4456685163423838 0.506309313164471 0.42666502702759324; visual box size=0.4456685163423838 0.506309313164471 0.42666502702759324
- link 2: geometry collision box size=0.45084502714273167 0.5238954398669781 0.030700276754036526; visual box size=0.45084502714273167 0.5238954398669781 0.030700276754036526
- link 3: geometry collision box size=0.058785116206491295 0.29860594962301334 0.9679033101508892; visual box size=0.058785116206491295 0.29860594962301334 0.9679033101508892
- link 4: geometry collision box size=0.31036362735313405 0.9392884321352825 0.7438421186671211; visual box size=0.31036362735313405 0.9392884321352825 0.7438421186671211
- link 5: geometry collision box size=0.5607173210286936 0.850526660963271 0.5905839712874152; visual box size=0.5607173210286936 0.850526660963271 0.5905839712874152
- link 6: geometry collision box size=0.17151709517771863 0.8677810644349934 0.9737752361596916; visual box size=0.17151709517771863 0.8677810644349934 0.9737752361596916
- link 7: geometry collision box size=0.20040745546617267 0.0990253627729546 0.5733827030223086; visual box size=0.20040745546617267 0.0990253627729546 0.5733827030223086
- link 8: geometry collision box size=0.10442422284151531 0.6659575282786826 0.29607267308315155; visual box size=0.10442422284151531 0.6659575282786826 0.29607267308315155
Joints:
- removed joint 0_5
- removed joint 0_6
- removed joint 1_2
- removed joint 6_7
- removed joint 8_9
- removed joint 9_10
- added joint 0_2: type revolute, parent 0, child 2, origin xyz=0 -0.35 0.7 rpy=0 0 0, axis 0 1 1, limit lower=-3.14159 upper=3.14159 effort=0.0 velocity=0.0
- added joint 0_7: type revolute, parent 0, child 7, origin xyz=0 0.35 0.7 rpy=0 0 0, axis 0 0 1, limit lower=-3.14159 upper=3.14159 effort=0.0 velocity=0.0
- added joint 4_5: type revolute, parent 4, child 5, origin xyz=0 -0.9392884321352825 0.7438421186671211 rpy=0 0 0, axis 1 1 1, limit lower=-3.14159 upper=3.14159 effort=0.0 velocity=0.0
- added joint 5_6: type revolute, parent 5, child 6, origin xyz=0 -0.850526660963271 0.5905839712874152 rpy=0 0 0, axis 1 0 0, limit lower=-3.14159 upper=3.14159 effort=0.0 velocity=0.0
- joint 0_1: axis 1 1 0 -> 1 0 0; origin xyz=-0.35 0 0.7 rpy=0 0 0 -> xyz=0.35 0 0.7 rpy=0 0 0
- joint 2_3: axis 1 0 1 -> 1 1 0; origin xyz=-0.6179261849630812 0 0.13224085421692466 rpy=0 0 0 -> xyz=0 -0.5238954398669781 0.030700276754036526 rpy=0 0 0
- joint 3_4: axis 1 1 0 -> 0 0 1; origin xyz=-0.9601271002174996 0 0.16648447729129467 rpy=0 0 0 -> xyz=0 -0.29860594962301334 0.9679033101508892 rpy=0 0 0
- joint 7_8: axis 1 0 0 -> 0 1 0; origin xyz=0 -0.31579310584644404 0.48121838623686386 rpy=0 0 0 -> xyz=0 0.0990253627729546 0.5733827030223086 rpy=0 0 0

File: body/body5.urdf (robot description, URDF)
Before this commit: robot robot, 8 links, 7 joints
Links:
- removed link 6
- removed link 7
- link 1: geometry collision box size=0.6816364556074682 0.7171532633675107 0.3479815079568077; visual box size=0.6816364556074682 0.7171532633675107 0.3479815079568077
- link 2: geometry collision box size=0.52417396740035 0.09040178960519829 0.2551839249465503; visual box size=0.52417396740035 0.09040178960519829 0.2551839249465503
- link 3: geometry collision box size=0.9594388378770715 0.13912615902147096 0.7757572503157156; visual box size=0.9594388378770715 0.13912615902147096 0.7757572503157156
- link 4: geometry collision box size=0.44505873211451163 0.9243078026249281 0.9712075281962813; visual box size=0.44505873211451163 0.9243078026249281 0.9712075281962813
- link 5: geometry collision box size=0.39723997685875156 0.9100841680576449 0.43812894915290224; visual box size=0.39723997685875156 0.9100841680576449 0.43812894915290224
Joints:
- removed joint 0_4
- removed joint 5_6
- removed joint 6_7
- added joint 3_4: type revolute, parent 3, child 4, origin xyz=-0.9594388378770715 0 0.7757572503157156 rpy=0 0 0, axis 1 1 1, limit lower=-3.14159 upper=3.14159 effort=0.0 velocity=0.0
- joint 0_1: axis 0 0 1 -> 1 1 0; origin xyz=0 -0.35 0.7 rpy=0 0 0 -> xyz=-0.35 0 0.7 rpy=0 0 0
- joint 1_2: axis 1 0 1 -> 0 0 1; origin xyz=0 -0.18012029744042013 0.4918620234154919 rpy=0 0 0 -> xyz=-0.6816364556074682 0 0.3479815079568077 rpy=0 0 0
- joint 2_3: axis 1 0 0 -> 0 1 0; origin xyz=0 -0.7860225796338303 0.7748980921186417 rpy=0 0 0 -> xyz=-0.52417396740035 0 0.2551839249465503 rpy=0 0 0
- joint 4_5: axis 0 1 0 -> 1 1 1; origin xyz=0 0.3400733891851615 0.17864939257994905 rpy=0 0 0 -> xyz=-0.44505873211451163 0 0.9712075281962813 rpy=0 0 0
