Commit message: readme

File: body/body1883.urdf (robot description, URDF)
Before this commit: robot robot, 6 links, 5 joints
Links:
- removed link 5
- link 1: geometry collision box size=0.04661346858217019 0.843320339142827 0.8350474212254118; visual box size=0.04661346858217019 0.843320339142827 0.8350474212254118
- link 2: geometry collision box size=0.9730808124776207 0.18294937963584712 0.5790764190210559; visual box size=0.9730808124776207 0.18294937963584712 0.5790764190210559
- link 3: geometry collision box size=0.24141596645460117 0.9074713788816542 0.5355692007995022; visual box size=0.24141596645460117 0.9074713788816542 0.5355692007995022
- link 4: geometry collision box size=0.1968593003562873 0.028400447508653448 0.7332244584062361; visual box size=0.1968593003562873 0.028400447508653448 0.7332244584062361
Joints:
- removed joint 0_2
- removed joint 0_5
- added joint 1_2: type revolute, parent 1, child 2, origin xyz=0 -0.843320339142827 0.8350474212254118 rpy=0 0 0, axis 1 0 0, limit lower=-3.14159 upper=3.14159 effort=0.0 velocity=0.0
- joint 0_1: axis 0 1 0 -> 1 1 1; origin xyz=-0.35 0 0.7 rpy=0 0 0 -> xyz=0 -0.35 0.7 rpy=0 0 0
- joint 2_3: axis 0 1 1 -> 1 0 1; origin xyz=0 -0.14066756704223315 0.771042142786742 rpy=0 0 0 -> xyz=0 -0.18294937963584712 0.5790764190210559 rpy=0 0 0
- joint 3_4: axis 1 0 1 -> 1 1 1; origin xyz=0 -0.6056207876200844 0.675387492843138 rpy=0 0 0 -> xyz=0 -0.9074713788816542 0.5355692007995022 rpy=0 0 0
