Commit message: readme

File: body/body3614.urdf (robot description, URDF)
Before this commit: robot robot, 10 links, 9 joints
Links:
- link 1: geometry collision box size=0.20434474394990176 0.06677322560653898 0.5712163413046109; visual box size=0.20434474394990176 0.06677322560653898 0.5712163413046109
- link 2: geometry collision box size=0.7102784127552225 0.28375240579198935 0.8912814945011249; visual box size=0.7102784127552225 0.28375240579198935 0.8912814945011249
- link 3: geometry collision box size=0.5203192612802345 0.032674747220581946 0.01902667919317269; visual box size=0.5203192612802345 0.032674747220581946 0.01902667919317269
- link 4: geometry collision box size=0.42544407734419154 0.6756003377375025 0.5444763147281303; visual box size=0.42544407734419154 0.6756003377375025 0.5444763147281303
- link 5: geometry collision box size=0.8140323746264132 0.9981599522851606 0.7738334073721997; visual box size=0.8140323746264132 0.9981599522851606 0.7738334073721997
- link 6: geometry collision box size=0.6452068089603276 0.005221673469258281 0.47612167520945226; visual box size=0.6452068089603276 0.005221673469258281 0.47612167520945226
- link 7: geometry collision box size=0.5142837977116697 0.986781958809422 0.4037430704820498; visual box size=0.5142837977116697 0.986781958809422 0.4037430704820498
- link 8: geometry collision box size=0.014156648419942797 0.3518262717957913 0.9878818277899449; visual box size=0.014156648419942797 0.3518262717957913 0.9878818277899449
- link 9: geometry collision box size=0.6450478328166024 0.8970898838125749 0.28250685725828417; visual box size=0.6450478328166024 0.8970898838125749 0.28250685725828417
Joints:
- removed joint 0_7
- removed joint 0_8
- removed joint 8_9
- added joint 0_9: type revolute, parent 0, child 9, origin xyz=0 0.35 0.7 rpy=0 0 0, axis 1 1 1, limit lower=-3.14159 upper=3.14159 effort=0.0 velocity=0.0
- added joint 6_7: type revolute, parent 6, child 7, origin xyz=0 -0.005221673469258281 0.47612167520945226 rpy=0 0 0, axis 0 1 1, limit lower=-3.14159 upper=3.14159 effort=0.0 velocity=0.0
- added joint 7_8: type revolute, parent 7, child 8, origin xyz=0 -0.986781958809422 0.4037430704820498 rpy=0 0 0, axis 1 1 0, limit lower=-3.14159 upper=3.14159 effort=0.0 velocity=0.0
- joint 0_6: axis 0 0 1 -> 1 1 0; origin xyz=0.35 0 0.7 rpy=0 0 0 -> xyz=0 -0.35 0.7 rpy=0 0 0
- joint 1_2: origin xyz=-0.0038304967129093592 0 0.5668284628833831 rpy=0 0 0 -> xyz=-0.20434474394990176 0 0.5712163413046109 rpy=0 0 0
- joint 2_3: axis 1 0 1 -> 0 1 0; origin xyz=-0.3421024224550536 0 0.9675273101090064 rpy=0 0 0 -> xyz=-0.7102784127552225 0 0.8912814945011249 rpy=0 0 0
- joint 3_4: axis 1 1 1 -> 1 0 0; origin xyz=-0.7411576667753312 0 0.829171605593075 rpy=0 0 0 -> xyz=-0.5203192612802345 0 0.01902667919317269 rpy=0 0 0
- joint 4_5: origin xyz=-0.7020120491340093 0 0.8752344059842949 rpy=0 0 0 -> xyz=-0.42544407734419154 0 0.5444763147281303 rpy=0 0 0

File: body/body4336.urdf (robot description, URDF)
Before this commit: robot robot, 6 links, 5 joints
Links:
- link 1: geometry collision box size=0.9450289438845669 0.3928803032247561 0.7597927670002993; visual box size=0.9450289438845669 0.3928803032247561 0.7597927670002993
- link 2: geometry collision box size=0.4081023658584543 0.17478185442679717 0.5595060961453219; visual box size=0.4081023658584543 0.17478185442679717 0.5595060961453219
- link 3: geometry collision box size=0.27105957766023003 0.31927582886663464 0.3891734821433678; visual box size=0.27105957766023003 0.31927582886663464 0.3891734821433678
- link 4: geometry collision box size=0.9846414490037517 0.5413597065496294 0.38628665250155725; visual box size=0.9846414490037517 0.5413597065496294 0.38628665250155725
- link 5: geometry collision box size=0.1290164426772299 0.7657946352964647 0.8179794830524226; visual box size=0.1290164426772299 0.7657946352964647 0.8179794830524226
Joints:
- removed joint 0_5
- added joint 4_5: type revolute, parent 4, child 5, origin xyz=0.9846414490037517 0 0.38628665250155725 rpy=0 0 0, axis 1 0 1, limit lower=-3.14159 upper=3.14159 effort=0.0 velocity=0.0
- joint 0_2: axis 1 1 1 -> 0 1 0; origin xyz=0 -0.35 0.7 rpy=0 0 0 -> xyz=0.35 0 0.7 rpy=0 0 0
- joint 2_3: axis 0 1 1 -> 1 1 0; origin xyz=0 -0.14066756704223315 0.771042142786742 rpy=0 0 0 -> xyz=0.4081023658584543 0 0.5595060961453219 rpy=0 0 0
- joint 3_4: axis 1 0 1 -> 0 1 0; origin xyz=0 -0.6056207876200844 0.675387492843138 rpy=0 0 0 -> xyz=0.27105957766023003 0 0.3891734821433678 rpy=0 0 0
