Commit message: run.py

File: body/body1329.urdf (robot description, URDF)
Before this commit: robot robot, 7 links, 6 joints
Links:
- added link 7, mass 1; collision box size=0.6937382655147536 0.6110035515902715 0.674019983942201; visual box size=0.6937382655147536 0.6110035515902715 0.674019983942201
- added link 8, mass 1; collision box size=0.11745374212114823 0.721120830858009 0.6113236281477744; visual box size=0.11745374212114823 0.721120830858009 0.6113236281477744
- added link 9, mass 1; collision box size=0.6488731319048344 0.8920692618273897 0.7208649653128105; visual box size=0.6488731319048344 0.8920692618273897 0.7208649653128105
- link 1: geometry collision box size=0.0038304967129093592 0.5647054702592181 0.5668284628833831; visual box size=0.0038304967129093592 0.5647054702592181 0.5668284628833831
- link 2: geometry collision box size=0.3421024224550536 0.1437880424720953 0.9675273101090064; visual box size=0.3421024224550536 0.1437880424720953 0.9675273101090064
- link 3: geometry collision box size=0.7411576667753312 0.26210727729902283 0.829171605593075; visual box size=0.7411576667753312 0.26210727729902283 0.829171605593075
- link 4: geometry collision box size=0.7020120491340093 0.5920172622540643 0.8752344059842949; visual box size=0.7020120491340093 0.5920172622540643 0.8752344059842949
- link 5: geometry collision box size=0.13730203781744021 0.05195270405476271 0.7397303384175518; visual box size=0.13730203781744021 0.05195270405476271 0.7397303384175518
- link 6: geometry collision box size=0.04909641869260062 0.9592734693549425 0.3187433928915787; visual box size=0.04909641869260062 0.9592734693549425 0.3187433928915787
Joints:
- removed joint 0_3
- removed joint 5_6
- added joint 0_6: type revolute, parent 0, child 6, origin xyz=0.35 0 0.7 rpy=0 0 0, axis 0 0 1, limit lower=-3.14159 upper=3.14159 effort=0.0 velocity=0.0
- added joint 0_7: type revolute, parent 0, child 7, origin xyz=0 -0.35 0.7 rpy=0 0 0, axis 1 1 1, limit lower=-3.14159 upper=3.14159 effort=0.0 velocity=0.0
- added joint 0_8: type revolute, parent 0, child 8, origin xyz=0 0.35 0.7 rpy=0 0 0, axis 0 0 1, limit lower=-3.14159 upper=3.14159 effort=0.0 velocity=0.0
- added joint 2_3: type revolute, parent 2, child 3, origin xyz=-0.3421024224550536 0 0.9675273101090064 rpy=0 0 0, axis 1 0 1, limit lower=-3.14159 upper=3.14159 effort=0.0 velocity=0.0
- added joint 8_9: type revolute, parent 8, child 9, origin xyz=0 0.721120830858009 0.6113236281477744 rpy=0 0 0, axis 1 0 0, limit lower=-3.14159 upper=3.14159 effort=0.0 velocity=0.0
- joint 0_1: axis 0 1 1 -> 1 1 1; origin xyz=0.35 0 0.7 rpy=0 0 0 -> xyz=-0.35 0 0.7 rpy=0 0 0
- joint 1_2: origin xyz=0.19710371003368676 0 0.15281354088412513 rpy=0 0 0 -> xyz=-0.0038304967129093592 0 0.5668284628833831 rpy=0 0 0
- joint 3_4: axis 1 0 0 -> 1 1 1; origin xyz=0 -0.8193769436752107 0.9460205345354766 rpy=0 0 0 -> xyz=-0.7411576667753312 0 0.829171605593075 rpy=0 0 0
- joint 4_5: axis 1 1 0 -> 1 0 0; origin xyz=0 -0.6215646914709174 0.18693901511158784 rpy=0 0 0 -> xyz=-0.7020120491340093 0 0.8752344059842949 rpy=0 0 0

File: body/body1883.urdf (robot description, URDF)
Before this commit: robot robot, 7 links, 6 joints
Links:
- removed link 6
- link 2: geometry collision box size=0.44206549519156024 0.14066756704223315 0.771042142786742; visual box size=0.44206549519156024 0.14066756704223315 0.771042142786742
- link 3: geometry collision box size=0.43339996101379474 0.6056207876200844 0.675387492843138; visual box size=0.43339996101379474 0.6056207876200844 0.675387492843138
- link 4: geometry collision box size=0.19748712760196974 0.793894941735572 0.674966690099463; visual box size=0.19748712760196974 0.793894941735572 0.674966690099463
- link 5: geometry collision box size=0.32964768003115497 0.3718935946127214 0.17462279126480318; visual box size=0.32964768003115497 0.3718935946127214 0.17462279126480318
Joints:
- removed joint 0_3
- removed joint 0_6
- removed joint 4_5
- added joint 0_5: type revolute, parent 0, child 5, origin xyz=0 0.35 0.7 rpy=0 0 0, axis 1 1 1, limit lower=-3.14159 upper=3.14159 effort=0.0 velocity=0.0
- added joint 2_3: type revolute, parent 2, child 3, origin xyz=0 -0.14066756704223315 0.771042142786742 rpy=0 0 0, axis 0 1 1, limit lower=-3.14159 upper=3.14159 effort=0.0 velocity=0.0
- joint 0_1: axis 1 0 1 -> 0 1 0
- joint 0_2: axis 0 0 1 -> 1 1 1; origin xyz=0.35 0 0.7 rpy=0 0 0 -> xyz=0 -0.35 0.7 rpy=0 0 0
- joint 3_4: axis 0 1 1 -> 1 0 1; origin xyz=0 -0.14066756704223315 0.771042142786742 rpy=0 0 0 -> xyz=0 -0.6056207876200844 0.675387492843138 rpy=0 0 0

File: body/body3285.urdf (robot description, URDF)
Before this commit: robot robot, 9 links, 8 joints
Links:
- removed link 3
- removed link 4
- removed link 5
- removed link 6
- removed link 7
- removed link 8
- link 1: geometry collision box size=0.8029462043611253 0.25022786274203845 0.9592624048128686; visual box size=0.8029462043611253 0.25022786274203845 0.9592624048128686
- link 2: geometry collision box size=0.812722776088469 0.9260479781475539 0.44179500726455545; visual box size=0.812722776088469 0.9260479781475539 0.44179500726455545
Joints:
- removed joint 0_3
- removed joint 0_7
- removed joint 3_4
- removed joint 4_5
- removed joint 5_6
- removed joint 7_8
- joint 0_1: axis 1 0 1 -> 1 0 0; origin xyz=-0.35 0 0.7 rpy=0 0 0 -> xyz=0.35 0 0.7 rpy=0 0 0
- joint 1_2: axis 1 1 0 -> 1 1 1; origin xyz=-0.8561630425294109 0 0.8266850100821808 rpy=0 0 0 -> xyz=0.8029462043611253 0 0.9592624048128686 rpy=0 0 0

File: body/body4211.urdf (robot description, URDF)
Before this commit: robot robot, 5 links, 4 joints
Links:
- added link 5, mass 1; collision box size=0.29701584724089414 0.5998551847634835 0.4461533669966381; visual box size=0.29701584724089414 0.5998551847634835 0.4461533669966381
- added link 6, mass 1; collision box size=0.8610088608533248 0.798438940577426 0.3877899282226017; visual box size=0.8610088608533248 0.798438940577426 0.3877899282226017
- link 1: geometry collision box size=0.8381189500347708 0.44524702398827953 0.03214205870058828; visual box size=0.8381189500347708 0.44524702398827953 0.03214205870058828
- link 2: geometry collision box size=0.7779213529725311 0.7036340433093002 0.7489593458209709; visual box size=0.7779213529725311 0.7036340433093002 0.7489593458209709
- link 3: geometry collision box size=0.5759507062581667 0.3109345449233175 0.609437518264306; visual box size=0.5759507062581667 0.3109345449233175 0.609437518264306
- link 4: geometry collision box size=0.12627597363612753 0.21784257876771995 0.6411097441822928; visual box size=0.12627597363612753 0.21784257876771995 0.6411097441822928
Joints:
- removed joint 2_3
- added joint 0_3: type revolute, parent 0, child 3, origin xyz=0 -0.35 0.7 rpy=0 0 0, axis 0 1 1, limit lower=-3.14159 upper=3.14159 effort=0.0 velocity=0.0
- added joint 4_5: type revolute, parent 4, child 5, origin xyz=0 0.21784257876771995 0.6411097441822928 rpy=0 0 0, axis 0 1 0, limit lower=-3.14159 upper=3.14159 effort=0.0 velocity=0.0
- added joint 5_6: type revolute, parent 5, child 6, origin xyz=0 0.5998551847634835 0.4461533669966381 rpy=0 0 0, axis 0 1 1, limit lower=-3.14159 upper=3.14159 effort=0.0 velocity=0.0
- joint 0_1: axis 1 0 1 -> 1 1 1
- joint 1_2: axis 0 0 1 -> 1 0 0; origin xyz=0.8959277791118226 0 0.2423074349676424 rpy=0 0 0 -> xyz=0.8381189500347708 0 0.03214205870058828 rpy=0 0 0

Commit message: readme

File: body/body1329.urdf (robot description, URDF)
Before this commit: robot robot, 10 links, 9 joints
Links:
- added link 10, mass 1; collision box size=0.48461650514969046 0.2601385947587238 0.11199798963728147; visual box size=0.48461650514969046 0.2601385947587238 0.11199798963728147
- added link 11, mass 1; collision box size=0.5036219109156685 0.4888932756852431 0.9648970399596215; visual box size=0.5036219109156685 0.4888932756852431 0.9648970399596215
- added link 12, mass 1; collision box size=0.09942757041481587 0.3023567543258393 0.009127275335518825; visual box size=0.09942757041481587 0.3023567543258393 0.009127275335518825
- added link 13, mass 1; collision box size=0.48191884293429443 0.032984937129627134 0.2198605733134571; visual box size=0.48191884293429443 0.032984937129627134 0.2198605733134571
- added link 14, mass 1; collision box size=0.46878651317158115 0.669937934416653 0.3012643708859857; visual box size=0.46878651317158115 0.669937934416653 0.3012643708859857
- added link 15, mass 1; collision box size=0.7365572279165892 0.5724843595548945 0.7784539527437297; visual box size=0.7365572279165892 0.5724843595548945 0.7784539527437297
- link 1: geometry collision box size=0.5622636965261801 0.9090661428853595 0.7864095184611026; visual box size=0.5622636965261801 0.9090661428853595 0.7864095184611026
- link 2: geometry collision box size=0.4608438884790995 0.09398989861531226 0.5297007710271594; visual box size=0.4608438884790995 0.09398989861531226 0.5297007710271594
- link 3: geometry collision box size=0.11665471502756686 0.25549993352642664 0.3989006599027948; visual box size=0.11665471502756686 0.25549993352642664 0.3989006599027948
- link 4: geometry collision box size=0.3989738923497974 0.5987197444489328 0.1626400033837353; visual box size=0.3989738923497974 0.5987197444489328 0.1626400033837353
- link 5: geometry collision box size=0.9511974134196001 0.7481692745562536 0.8494863731823896; visual box size=0.9511974134196001 0.7481692745562536 0.8494863731823896
- link 6: geometry collision box size=0.33379905471740934 0.031891434880507497 0.21092491737578556; visual box size=0.33379905471740934 0.031891434880507497 0.21092491737578556
- link 7: geometry collision box size=0.32269580012481414 0.6096110356725748 0.8144409683733833; visual box size=0.32269580012481414 0.6096110356725748 0.8144409683733833
- link 8: geometry collision box size=0.14916790829145898 0.8972180717530853 0.5002637827037587; visual box size=0.14916790829145898 0.8972180717530853 0.5002637827037587
- link 9: geometry collision box size=0.36436095333044294 0.9895337143065168 0.9883276722605159; visual box size=0.36436095333044294 0.9895337143065168 0.9883276722605159
Joints:
- removed joint 0_6
- removed joint 0_7
- removed joint 0_8
- removed joint 3_4
- added joint 0_10: type revolute, parent 0, child 10, origin xyz=0 0.35 0.7 rpy=0 0 0, axis 1 0 1, limit lower=-3.14159 upper=3.14159 effort=0.0 velocity=0.0
- added joint 0_4: type revolute, parent 0, child 4, origin xyz=0 -0.35 0.7 rpy=0 0 0, axis 1 1 0, limit lower=-3.14159 upper=3.14159 effort=0.0 velocity=0.0
- added joint 10_11: type revolute, parent 10, child 11, origin xyz=0 0.2601385947587238 0.11199798963728147 rpy=0 0 0, axis 1 0 0, limit lower=-3.14159 upper=3.14159 effort=0.0 velocity=0.0
- added joint 11_12: type revolute, parent 11, child 12, origin xyz=0 0.4888932756852431 0.9648970399596215 rpy=0 0 0, axis 1 0 0, limit lower=-3.14159 upper=3.14159 effort=0.0 velocity=0.0
- added joint 12_13: type revolute, parent 12, child 13, origin xyz=0 0.3023567543258393 0.009127275335518825 rpy=0 0 0, axis 0 0 1, limit lower=-3.14159 upper=3.14159 effort=0.0 velocity=0.0
- added joint 13_14: type revolute, parent 13, child 14, origin xyz=0 0.032984937129627134 0.2198605733134571 rpy=0 0 0, axis 1 1 0, limit lower=-3.14159 upper=3.14159 effort=0.0 velocity=0.0
- added joint 14_15: type revolute, parent 14, child 15, origin xyz=0 0.669937934416653 0.3012643708859857 rpy=0 0 0, axis 0 1 0, limit lower=-3.14159 upper=3.14159 effort=0.0 velocity=0.0
- added joint 5_6: type revolute, parent 5, child 6, origin xyz=0 -0.7481692745562536 0.8494863731823896 rpy=0 0 0, axis 0 1 0, limit lower=-3.14159 upper=3.14159 effort=0.0 velocity=0.0
- added joint 6_7: type revolute, parent 6, child 7, origin xyz=0 -0.031891434880507497 0.21092491737578556 rpy=0 0 0, axis 0 0 1, limit lower=-3.14159 upper=3.14159 effort=0.0 velocity=0.0
- added joint 7_8: type revolute, parent 7, child 8, origin xyz=0 -0.6096110356725748 0.8144409683733833 rpy=0 0 0, axis 1 1 0, limit lower=-3.14159 upper=3.14159 effort=0.0 velocity=0.0
- joint 1_2: axis 1 1 1 -> 1 0 1; origin xyz=-0.0038304967129093592 0 0.5668284628833831 rpy=0 0 0 -> xyz=-0.5622636965261801 0 0.7864095184611026 rpy=0 0 0
- joint 2_3: axis 1 0 1 -> 1 0 0; origin xyz=-0.3421024224550536 0 0.9675273101090064 rpy=0 0 0 -> xyz=-0.4608438884790995 0 0.5297007710271594 rpy=0 0 0
- joint 4_5: axis 1 0 0 -> 0 0 1; origin xyz=-0.7020120491340093 0 0.8752344059842949 rpy=0 0 0 -> xyz=0 -0.5987197444489328 0.1626400033837353 rpy=0 0 0
- joint 8_9: origin xyz=0 0.721120830858009 0.6113236281477744 rpy=0 0 0 -> xyz=0 -0.8972180717530853 0.5002637827037587 rpy=0 0 0
